File: XLD/Q1_2023/L1.kicad_sch (KiCad schematic)
At the start: 176 parts

Commit message: done
Connections:
- net at L:407.: now also TJI403.; no longer HEMT402. (gnd)
- net at TJI402.: now also L:404.; no longer L:405.
- net at L:403.: now also Coupler401.; no longer TWPA401.
- net at Coupler401.: now also L:404.; no longer L:403.
- net at Coupler402.: now also L:409.; no longer L:410.
- net at L:409.: now also TWPA402.; no longer Coupler402.
- net at TWPA402.: now also L:408.; no longer L:409.
- new net: Eccosorb404., LPF404.
- new net: Eccosorb422., LPF422.
- new net: HEMT402. (gnd), L:407.
- new net: Eccosorb408., LPF408.
- new net: L:405., TJI402.
- new net: L:403., TWPA401.
- new net: Coupler402., L:410.
- new net: Eccosorb402., LPF402.
- new net: Eccosorb418., LPF418.
- new net: Eccosorb420., LPF420.
- new net: Eccosorb412., LPF412.
- new net: Eccosorb407., LPF407.
- new net: Eccosorb401., LPF401.
- new net: Eccosorb411., LPF411.
- new net: Eccosorb416., LPF416.
- new net: Eccosorb415., LPF415.
- new net: Eccosorb419., LPF419.
- new net: Eccosorb414., LPF414.
- new net: Eccosorb423., LPF423.
- new net: Eccosorb410., LPF410.
- new net: Eccosorb403., LPF403.
- new net: ATT473., ATT474.
- new net: Eccosorb406., LPF406.
- new net: Eccosorb417., LPF417.
- new net: Eccosorb421., LPF421.
- new net: Eccosorb405., LPF405.
- new net: Eccosorb409., LPF409.
- new net: Eccosorb413., LPF413.

Commit message: Corrected but path not verified
Connections:
- net at L:407.: now also TJI403.; no longer HEMT402. (gnd)
- net at TJI402.: now also L:404.; no longer L:405.
- net at L:403.: now also Coupler401.; no longer TWPA401.
- net at Coupler401.: now also L:404.; no longer L:403.
- net at Coupler402.: now also L:409.; no longer L:410.
- net at L:409.: now also TWPA402.; no longer Coupler402.
- net at TWPA402.: now also L:408.; no longer L:409.
- new net: Eccosorb404., LPF404.
- new net: Eccosorb422., LPF422.
- new net: HEMT402. (gnd), L:407.
- new net: Eccosorb408., LPF408.
- new net: L:405., TJI402.
- new net: L:403., TWPA401.
- new net: Coupler402., L:410.
- new net: Eccosorb402., LPF402.
- new net: Eccosorb418., LPF418.
- new net: Eccosorb420., LPF420.
- new net: Eccosorb412., LPF412.
- new net: Eccosorb407., LPF407.
- new net: Eccosorb401., LPF401.
- new net: Eccosorb411., LPF411.
- new net: Eccosorb416., LPF416.
- new net: Eccosorb415., LPF415.
- new net: Eccosorb419., LPF419.
- new net: Eccosorb414., LPF414.
- new net: Eccosorb423., LPF423.
- new net: Eccosorb410., LPF410.
- new net: Eccosorb403., LPF403.
- new net: ATT473., ATT474.
- new net: Eccosorb406., LPF406.
- new net: Eccosorb417., LPF417.
- new net: Eccosorb421., LPF421.
- new net: Eccosorb405., LPF405.
- new net: Eccosorb409., LPF409.
- new net: Eccosorb413., LPF413.

Commit message: filter fixed'
Parts:
- renumbered ATT457 to ATT?, ATT497 to ATT?, ATT465 to ATT?, ATT462 to ATT?, ATT490 to ATT?, ATT475 to ATT?, ATT491 to ATT?, ATT476 to ATT?, ATT480 to ATT?, ATT488 to ATT?, ATT466 to ATT?, ATT486 to ATT?, ATT495 to ATT?, ATT482 to ATT?, ATT478 to ATT?, ATT483 to ATT?, ATT481 to ATT?, ATT484 to ATT?, ATT498 to ATT?, ATT467 to ATT?, ATT469 to ATT?, ATT473 to ATT?, ATT487 to ATT?, ATT471 to ATT?, ATT493 to ATT?, ATT496 to ATT?, ATT463 to ATT?, ATT460 to ATT?, ATT468 to ATT?, ATT499 to ATT?, ATT472 to ATT?, ATT477 to ATT?, ATT494 to ATT?, ATT474 to ATT?, ATT492 to ATT?, ATT470 to ATT?, ATT458 to ATT?, ATT456 to ATT?, ATT489 to ATT?, ATT461 to ATT?, ATT479 to ATT?, ATT459 to ATT?, ATT464 to ATT?, ATT485 to ATT?, Coupler402 to Coupler?, Coupler401 to Coupler?, Eccosorb404 to Eccosorb?, Eccosorb422 to Eccosorb?, Eccosorb402 to Eccosorb?, Eccosorb418 to Eccosorb?, Eccosorb420 to Eccosorb?, Eccosorb412 to Eccosorb?, Eccosorb407 to Eccosorb?, Eccosorb401 to Eccosorb?, Eccosorb411 to Eccosorb?, Eccosorb416 to Eccosorb?, Eccosorb419 to Eccosorb?, Eccosorb414 to Eccosorb?, Eccosorb410 to Eccosorb?, Eccosorb403 to Eccosorb?, Eccosorb406 to Eccosorb?, Eccosorb417 to Eccosorb?, Eccosorb423 to Eccosorb?, Eccosorb409 to Eccosorb?, Eccosorb408 to Eccosorb?, Eccosorb421 to Eccosorb?, Eccosorb415 to Eccosorb?, Eccosorb413 to Eccosorb?, Eccosorb405 to Eccosorb?, HEMT402 to HEMT?, HEMT401 to HEMT?, L:435 to L:?, L:444 to L:?, L:414 to L:?, L:439 to L:?, L:436 to L:?, L:425 to L:?, L:405 to L:?, L:432 to L:?, L:403 to L:?, L:410 to L:?, L:447 to L:?, L:409 to L:?, L:441 to L:?, L:416 to L:?, L:445 to L:?, L:433 to L:?, L:404 to L:?, L:413 to L:?, L:427 to L:?, L:442 to L:?, L:440 to L:?, L:418 to L:?, L:411 to L:?, L:424 to L:?, L:408 to L:?, L:419 to L:?, L:438 to L:?, L:428 to L:?, L:407 to L:?, L:430 to L:?, L:417 to L:?, L:402 to L:?, L:429 to L:?, L:443 to L:?, L:422 to L:?, L:420 to L:?, L:446 to L:?, L:401 to L:?, L:431 to L:?, L:423 to L:?, L:448 to L:?, L:415 to L:?, L:412 to L:?, L:434 to L:?, L:426 to L:?, L:437 to L:?, L:406 to L:?, L:421 to L:?, LPF408 to LPF?, LPF422 to LPF?, LPF418 to LPF?, LPF407 to LPF?, LPF411 to LPF?, LPF402 to LPF?, LPF415 to LPF?, LPF423 to LPF?, LPF412 to LPF?, LPF404 to LPF?, LPF410 to LPF?, LPF414 to LPF?, LPF401 to LPF?, LPF421 to LPF?, LPF405 to LPF?, LPF420 to LPF?, LPF417 to LPF?, LPF413 to LPF?, LPF419 to LPF?, LPF403 to LPF?, LPF409 to LPF?, LPF416 to LPF?, LPF406 to LPF?, LX-X409 to LX-X?, LX-X406 to LX-X?, LX-X422 to LX-X?, LX-X417 to LX-X?, LX-X424 to LX-X?, LX-X411 to LX-X?, LX-X407 to LX-X?, LX-X415 to LX-X?, LX-X414 to LX-X?, LX-X408 to LX-X?, LX-X405 to LX-X?, LX-X423 to LX-X?, LX-X416 to LX-X?, LX-X401 to LX-X?, LX-X412 to LX-X?, LX-X403 to LX-X?, LX-X419 to LX-X?, LX-X421 to LX-X?, LX-X418 to LX-X?, LX-X420 to LX-X?, LX-X404 to LX-X?, LX-X413 to LX-X?, LX-X425 to LX-X?, LX-X410 to LX-X?, LX-X402 to LX-X?, LX401 to LX?, TJI404 to TJI?, TJI401 to TJI?, TJI403 to TJI?, TJI402 to TJI?, TWPA401 to TWPA?, TWPA402 to TWPA?, Ω?401 to Ω?, Ω?402 to Ω?
Connections:
- net at L:?.: now also TJI?.; no longer HEMT?. (gnd)
- net at TJI?.: now also L:?.; no longer L:?.
- net at L:?.: now also Coupler?.; no longer TWPA?.
- net at Coupler?.: now also L:?.; no longer L:?. (x2)
- net at L:?.: now also TWPA?.; no longer Coupler?.
- net at TWPA?.: now also L:?.; no longer L:?.
- new net: Eccosorb?., LPF?. (x23)
- new net: HEMT?. (gnd), L:?.
- new net: L:?., TJI?.
- new net: L:?., TWPA?.
- new net: Coupler?., L:?.
- new net: ATT?., ATT?.
