File: XLD/Q1_2023/L2.kicad_sch (KiCad schematic)
At the start: 61 parts

Commit message: done
Connections:
- net at L:212.: now also TJI206.; no longer Coupler201.
- net at TJI206.: now also L:213.; no longer L:212.
- net at TJI209.: no longer L:216.
- net at TJI205.: now also L:210.; no longer L:209.
- net at L:210.: now also TWPA201.; no longer TJI205.
- net at TWPA201.: now also L:211.; no longer L:210.
- new net: L:202., TJI201.
- new net: Coupler201., L:212.
- new net: L:208., TJI204.
- new net: L:215., TJI208.
- new net: L:214., TJI207.
- new net: L:206., TJI203.
- new net: L:216., TJI209.
- new net: L:209., TJI205.
- new net: L:204., TJI202.

Commit message: Corrected but path not verified
Connections:
- net at L:212.: now also TJI206.; no longer Coupler201.
- net at TJI206.: now also L:213.; no longer L:212.
- net at TJI209.: no longer L:216.
- net at TJI205.: now also L:210.; no longer L:209.
- net at L:210.: now also TWPA201.; no longer TJI205.
- net at TWPA201.: now also L:211.; no longer L:210.
- new net: L:202., TJI201.
- new net: Coupler201., L:212.
- new net: L:208., TJI204.
- new net: L:215., TJI208.
- new net: L:214., TJI207.
- new net: L:206., TJI203.
- new net: L:216., TJI209.
- new net: L:209., TJI205.
- new net: L:204., TJI202.

Commit message: filter fixed'
Parts:
- renumbered ATT216 to ATT?, ATT201 to ATT?, ATT209 to ATT?, ATT205 to ATT?, ATT210 to ATT?, ATT207 to ATT?, ATT211 to ATT?, ATT213 to ATT?, ATT220 to ATT?, ATT215 to ATT?, ATT204 to ATT?, ATT217 to ATT?, ATT203 to ATT?, ATT214 to ATT?, ATT212 to ATT?, ATT208 to ATT?, ATT202 to ATT?, ATT219 to ATT?, ATT218 to ATT?, ATT206 to ATT?, Coupler201 to Coupler?, HEMT205 to HEMT?, HEMT206 to HEMT?, HEMT208 to HEMT?, HEMT201 to HEMT?, HEMT207 to HEMT?, HEMT202 to HEMT?, HEMT204 to HEMT?, HEMT203 to HEMT?, L:212 to L:?, L:207 to L:?, L:215 to L:?, L:205 to L:?, L:203 to L:?, L:216 to L:?, L:209 to L:?, L:202 to L:?, L:206 to L:?, L:210 to L:?, L:211 to L:?, L:201 to L:?, L:204 to L:?, L:214 to L:?, L:208 to L:?, L:213 to L:?, LX-X202 to LX-X?, LX-X203 to LX-X?, LX-X205 to LX-X?, LX-X204 to LX-X?, LX-X201 to LX-X?, LX201 to LX?, TJI201 to TJI?, TJI204 to TJI?, TJI208 to TJI?, TJI207 to TJI?, TJI203 to TJI?, TJI205 to TJI?, TJI206 to TJI?, TJI202 to TJI?, TJI209 to TJI?, TWPA201 to TWPA?
Connections:
- net at L:?.: now also TJI?.; no longer Coupler?.
- net at TJI?.: now also L:?.; no longer L:?. (x2)
- net at TJI?.: no longer L:?.
- net at L:?.: now also TWPA?.; no longer TJI?.
- net at TWPA?.: now also L:?.; no longer L:?.
- new net: L:?., TJI?. (x8)
- new net: Coupler?., L:?.
