File: XLD/Q1_2023/L3.kicad_sch (KiCad schematic)
At the start: 298 parts

Commit message: done
Connections:
- net at Eccosorb313.: now also LPF313.; no longer L:327.
- net at Eccosorb318.: now also L:337.; no longer LPF318.
- net at Eccosorb320.: now also L:341.; no longer LPF320.
- net at Eccosorb323.: now also L:348.; no longer LPF323.
- net at Eccosorb304.: now also L:308.; no longer LPF304.
- net at Eccosorb312.: now also LPF312.; no longer L:325.
- net at Eccosorb307.: now also LPF307.; no longer L:314.
- net at Eccosorb314.: now also L:329.; no longer LPF314.
- net at Eccosorb303.: now also LPF303.; no longer L:306.
- net at Eccosorb301.: now also LPF301.; no longer L:302.
- net at Eccosorb317.: now also L:335.; no longer LPF317.
- net at Eccosorb322.: now also LPF322.; no longer L:346.
- net at Eccosorb316.: now also LPF316.; no longer L:333.
- net at Eccosorb311.: now also L:323.; no longer LPF311.
- net at Eccosorb324.: now also L:350.; no longer LPF324.
- net at Eccosorb305.: now also LPF305.; no longer L:310.
- net at Eccosorb306.: now also LPF306.; no longer L:312.
- net at Eccosorb319.: now also L:339.; no longer LPF319.
- net at Eccosorb310.: now also L:321.; no longer LPF310.
- net at Eccosorb321.: now also L:344.; no longer LPF321.
- net at Eccosorb302.: now also L:304.; no longer LPF302.
- net at Eccosorb308.: now also LPF308.; no longer L:316.
- net at Eccosorb309.: now also LPF309.; no longer L:318.
- net at Eccosorb325.: now also LPF325.; no longer L:354.
- new net: Eccosorb313., L:327.
- new net: Eccosorb318., LPF318.
- new net: Eccosorb320., LPF320.
- new net: Eccosorb323., LPF323.
- new net: Eccosorb304., LPF304.
- new net: Eccosorb312., L:325.
- new net: Eccosorb307., L:314.
- new net: Eccosorb314., LPF314.
- new net: Eccosorb303., L:306.
- new net: Eccosorb301., L:302.
- new net: Eccosorb317., LPF317.
- new net: Eccosorb322., L:346.
- new net: Eccosorb316., L:333.
- new net: Eccosorb311., LPF311.
- new net: Eccosorb324., LPF324.
- new net: Eccosorb326., LPF326.
- new net: Eccosorb305., L:310.
- new net: Eccosorb306., L:312.
- new net: Eccosorb319., LPF319.
- new net: Eccosorb310., LPF310.
- new net: Eccosorb321., LPF321.
- new net: Eccosorb302., LPF302.
- new net: Eccosorb308., L:316.
- new net: Eccosorb309., L:318.
- new net: Eccosorb315., LPF315.
- new net: Eccosorb325., L:354.

Commit message: Corrected but path not verified
Connections:
- net at Eccosorb313.: now also LPF313.; no longer L:327.
- net at Eccosorb318.: now also L:337.; no longer LPF318.
- net at Eccosorb320.: now also L:341.; no longer LPF320.
- net at Eccosorb323.: now also L:348.; no longer LPF323.
- net at Eccosorb304.: now also L:308.; no longer LPF304.
- net at Eccosorb312.: now also LPF312.; no longer L:325.
- net at Eccosorb307.: now also LPF307.; no longer L:314.
- net at Eccosorb314.: now also L:329.; no longer LPF314.
- net at Eccosorb303.: now also LPF303.; no longer L:306.
- net at Eccosorb301.: now also LPF301.; no longer L:302.
- net at Eccosorb317.: now also L:335.; no longer LPF317.
- net at Eccosorb322.: now also LPF322.; no longer L:346.
- net at Eccosorb316.: now also LPF316.; no longer L:333.
- net at Eccosorb311.: now also L:323.; no longer LPF311.
- net at Eccosorb324.: now also L:350.; no longer LPF324.
- net at Eccosorb305.: now also LPF305.; no longer L:310.
- net at Eccosorb306.: now also LPF306.; no longer L:312.
- net at Eccosorb319.: now also L:339.; no longer LPF319.
- net at Eccosorb310.: now also L:321.; no longer LPF310.
- net at Eccosorb321.: now also L:344.; no longer LPF321.
- net at Eccosorb302.: now also L:304.; no longer LPF302.
- net at Eccosorb308.: now also LPF308.; no longer L:316.
- net at Eccosorb309.: now also LPF309.; no longer L:318.
- net at Eccosorb325.: now also LPF325.; no longer L:354.
- new net: Eccosorb313., L:327.
- new net: Eccosorb318., LPF318.
- new net: Eccosorb320., LPF320.
- new net: Eccosorb323., LPF323.
- new net: Eccosorb304., LPF304.
- new net: Eccosorb312., L:325.
- new net: Eccosorb307., L:314.
- new net: Eccosorb314., LPF314.
- new net: Eccosorb303., L:306.
- new net: Eccosorb301., L:302.
- new net: Eccosorb317., LPF317.
- new net: Eccosorb322., L:346.
- new net: Eccosorb316., L:333.
- new net: Eccosorb311., LPF311.
- new net: Eccosorb324., LPF324.
- new net: Eccosorb326., LPF326.
- new net: Eccosorb305., L:310.
- new net: Eccosorb306., L:312.
- new net: Eccosorb319., LPF319.
- new net: Eccosorb310., LPF310.
- new net: Eccosorb321., LPF321.
- new net: Eccosorb302., LPF302.
- new net: Eccosorb308., L:316.
- new net: Eccosorb309., L:318.
- new net: Eccosorb315., LPF315.
- new net: Eccosorb325., L:354.

Commit message: filter fixed'
Parts:
- LPF?: renamed from LPF318; value F‐30‐8000‐R -> F-30-8000-R; symbol Quantum Computing:F‐30‐8000‐R -> Quantum Computing:F-30-8000-R
- LPF?: renamed from LPF320; value F‐30‐8000‐R -> F-30-8000-R; symbol Quantum Computing:F‐30‐8000‐R -> Quantum Computing:F-30-8000-R
- LPF?: renamed from LPF304; value F‐30‐8000‐R -> F-30-8000-R; symbol Quantum Computing:F‐30‐8000‐R -> Quantum Computing:F-30-8000-R
- LPF?: renamed from LPF323; value F‐30‐8000‐R -> F-30-8000-R; symbol Quantum Computing:F‐30‐8000‐R -> Quantum Computing:F-30-8000-R
- LPF?: renamed from LPF322; value F‐30‐8000‐R -> F-30-8000-R; symbol Quantum Computing:F‐30‐8000‐R -> Quantum Computing:F-30-8000-R
- LPF?: renamed from LPF324; value F‐30‐8000‐R -> F-30-8000-R; symbol Quantum Computing:F‐30‐8000‐R -> Quantum Computing:F-30-8000-R
- LPF?: renamed from LPF307; value F‐30‐8000‐R -> F-30-8000-R; symbol Quantum Computing:F‐30‐8000‐R -> Quantum Computing:F-30-8000-R
- LPF?: renamed from LPF301; value F‐30‐8000‐R -> F-30-8000-R; symbol Quantum Computing:F‐30‐8000‐R -> Quantum Computing:F-30-8000-R
- LPF?: renamed from LPF316; value F‐30‐8000‐R -> F-30-8000-R; symbol Quantum Computing:F‐30‐8000‐R -> Quantum Computing:F-30-8000-R
- LPF?: renamed from LPF319; value F‐30‐8000‐R -> F-30-8000-R; symbol Quantum Computing:F‐30‐8000‐R -> Quantum Computing:F-30-8000-R
- LPF?: renamed from LPF321; value F‐30‐8000‐R -> F-30-8000-R; symbol Quantum Computing:F‐30‐8000‐R -> Quantum Computing:F-30-8000-R
- LPF?: renamed from LPF302; value F‐30‐8000‐R -> F-30-8000-R; symbol Quantum Computing:F‐30‐8000‐R -> Quantum Computing:F-30-8000-R
- LPF?: renamed from LPF308; value F‐30‐8000‐R -> F-30-8000-R; symbol Quantum Computing:F‐30‐8000‐R -> Quantum Computing:F-30-8000-R
- LPF?: renamed from LPF317; value F‐30‐8000‐R -> F-30-8000-R; symbol Quantum Computing:F‐30‐8000‐R -> Quantum Computing:F-30-8000-R
- LPF?: renamed from LPF326; value F‐30‐8000‐R -> F-30-8000-R; symbol Quantum Computing:F‐30‐8000‐R -> Quantum Computing:F-30-8000-R
- LPF?: renamed from LPF303; value F‐30‐8000‐R -> F-30-8000-R; symbol Quantum Computing:F‐30‐8000‐R -> Quantum Computing:F-30-8000-R
- LPF?: renamed from LPF305; value F‐30‐8000‐R -> F-30-8000-R; symbol Quantum Computing:F‐30‐8000‐R -> Quantum Computing:F-30-8000-R
- LPF?: renamed from LPF306; value F‐30‐8000‐R -> F-30-8000-R; symbol Quantum Computing:F‐30‐8000‐R -> Quantum Computing:F-30-8000-R
- LPF?: renamed from LPF309; value F‐30‐8000‐R -> F-30-8000-R; symbol Quantum Computing:F‐30‐8000‐R -> Quantum Computing:F-30-8000-R
- LPF?: renamed from LPF315; value F‐30‐8000‐R -> F-30-8000-R; symbol Quantum Computing:F‐30‐8000‐R -> Quantum Computing:F-30-8000-R
- LPF?: renamed from LPF325; value F‐30‐8000‐R -> F-30-8000-R; symbol Quantum Computing:F‐30‐8000‐R -> Quantum Computing:F-30-8000-R
- renumbered ATT405 to ATT?, ATT445 to ATT?, ATT367 to ATT?, ATT410 to ATT?, ATT418 to ATT?, ATT358 to ATT?, ATT425 to ATT?, ATT370 to ATT?, ATT326 to ATT?, ATT395 to ATT?, ATT391 to ATT?, ATT448 to ATT?, ATT335 to ATT?, ATT381 to ATT?, ATT437 to ATT?, ATT320 to ATT?, ATT342 to ATT?, ATT349 to ATT?, ATT400 to ATT?, ATT331 to ATT?, ATT364 to ATT?, ATT374 to ATT?, ATT338 to ATT?, ATT431 to ATT?, ATT397 to ATT?, ATT373 to ATT?, ATT401 to ATT?, ATT310 to ATT?, ATT398 to ATT?, ATT419 to ATT?, ATT382 to ATT?, ATT451 to ATT?, ATT351 to ATT?, ATT350 to ATT?, ATT422 to ATT?, ATT389 to ATT?, ATT355 to ATT?, ATT413 to ATT?, ATT325 to ATT?, ATT347 to ATT?, ATT426 to ATT?, ATT452 to ATT?, ATT309 to ATT?, ATT406 to ATT?, ATT449 to ATT?, ATT328 to ATT?, ATT359 to ATT?, ATT346 to ATT?, ATT415 to ATT?, ATT392 to ATT?, ATT399 to ATT?, ATT318 to ATT?, ATT428 to ATT?, ATT375 to ATT?, ATT334 to ATT?, ATT317 to ATT?, ATT409 to ATT?, ATT324 to ATT?, ATT450 to ATT?, ATT307 to ATT?, ATT341 to ATT?, ATT357 to ATT?, ATT372 to ATT?, ATT453 to ATT?, ATT396 to ATT?, ATT336 to ATT?, ATT430 to ATT?, ATT354 to ATT?, ATT366 to ATT?, ATT348 to ATT?, ATT380 to ATT?, ATT365 to ATT?, ATT446 to ATT?, ATT332 to ATT?, ATT417 to ATT?, ATT388 to ATT?, ATT379 to ATT?, ATT404 to ATT?, ATT305 to ATT?, ATT436 to ATT?, ATT383 to ATT?, ATT352 to ATT?, ATT403 to ATT?, ATT356 to ATT?, ATT442 to ATT?, ATT454 to ATT?, ATT333 to ATT?, ATT377 to ATT?, ATT439 to ATT?, ATT408 to ATT?, ATT361 to ATT?, ATT312 to ATT?, ATT302 to ATT?, ATT378 to ATT?, ATT323 to ATT?, ATT438 to ATT?, ATT363 to ATT?, ATT322 to ATT?, ATT308 to ATT?, ATT390 to ATT?, ATT432 to ATT?, ATT414 to ATT?, ATT344 to ATT?, ATT315 to ATT?, ATT306 to ATT?, ATT353 to ATT?, ATT394 to ATT?, ATT314 to ATT?, ATT412 to ATT?, ATT360 to ATT?, ATT429 to ATT?, ATT424 to ATT?, ATT303 to ATT?, ATT369 to ATT?, ATT384 to ATT?, ATT411 to ATT?, ATT440 to ATT?, ATT385 to ATT?, ATT337 to ATT?, ATT371 to ATT?, ATT434 to ATT?, ATT329 to ATT?, ATT301 to ATT?, ATT343 to ATT?, ATT423 to ATT?, ATT330 to ATT?, ATT433 to ATT?, ATT402 to ATT?, ATT339 to ATT?, ATT313 to ATT?, ATT427 to ATT?, ATT420 to ATT?, ATT340 to ATT?, ATT455 to ATT?, ATT316 to ATT?, ATT345 to ATT?, ATT444 to ATT?, ATT304 to ATT?, ATT435 to ATT?, ATT387 to ATT?, ATT368 to ATT?, ATT327 to ATT?, ATT319 to ATT?, ATT321 to ATT?, ATT362 to ATT?, ATT443 to ATT?, ATT311 to ATT?, ATT416 to ATT?, ATT376 to ATT?, ATT393 to ATT?, ATT386 to ATT?, ATT421 to ATT?, ATT407 to ATT?, ATT447 to ATT?, ATT441 to ATT?, Eccosorb323 to Eccosorb?, Eccosorb304 to Eccosorb?, Eccosorb307 to Eccosorb?, Eccosorb314 to Eccosorb?, Eccosorb301 to Eccosorb?, Eccosorb303 to Eccosorb?, Eccosorb317 to Eccosorb?, Eccosorb316 to Eccosorb?, Eccosorb324 to Eccosorb?, Eccosorb326 to Eccosorb?, Eccosorb305 to Eccosorb?, Eccosorb322 to Eccosorb?, Eccosorb306 to Eccosorb?, Eccosorb312 to Eccosorb?, Eccosorb321 to Eccosorb?, Eccosorb311 to Eccosorb?, Eccosorb315 to Eccosorb?, Eccosorb313 to Eccosorb?, Eccosorb310 to Eccosorb?, Eccosorb325 to Eccosorb?, Eccosorb309 to Eccosorb?, Eccosorb320 to Eccosorb?, Eccosorb318 to Eccosorb?, Eccosorb308 to Eccosorb?, Eccosorb319 to Eccosorb?, Eccosorb302 to Eccosorb?, L:327 to L:?, L:353 to L:?, L:349 to L:?, L:325 to L:?, L:338 to L:?, L:336 to L:?, L:306 to L:?, L:303 to L:?, L:351 to L:?, L:311 to L:?, L:346 to L:?, L:355 to L:?, L:340 to L:?, L:341 to L:?, L:302 to L:?, L:333 to L:?, L:314 to L:?, L:324 to L:?, L:334 to L:?, L:332 to L:?, L:308 to L:?, L:356 to L:?, L:317 to L:?, L:313 to L:?, L:345 to L:?, L:309 to L:?, L:339 to L:?, L:350 to L:?, L:307 to L:?, L:316 to L:?, L:330 to L:?, L:318 to L:?, L:326 to L:?, L:337 to L:?, L:310 to L:?, L:321 to L:?, L:328 to L:?, L:335 to L:?, L:301 to L:?, L:354 to L:?, L:342 to L:?, L:315 to L:?, L:348 to L:?, L:344 to L:?, L:343 to L:?, L:320 to L:?, L:352 to L:?, L:329 to L:?, L:312 to L:?, L:347 to L:?, L:331 to L:?, L:305 to L:?, L:319 to L:?, L:304 to L:?, L:323 to L:?, L:322 to L:?, LPF311 to LPF?, LPF310 to LPF?, LPF314 to LPF?, LPF313 to LPF?, LPF312 to LPF?, LX-X313 to LX-X?, LX-X301 to LX-X?, LX-X303 to LX-X?, LX-X315 to LX-X?, LX-X326 to LX-X?, LX-X322 to LX-X?, LX-X308 to LX-X?, LX-X310 to LX-X?, LX-X312 to LX-X?, LX-X304 to LX-X?, LX-X330 to LX-X?, LX-X306 to LX-X?, LX-X327 to LX-X?, LX-X314 to LX-X?, LX-X317 to LX-X?, LX-X316 to LX-X?, LX-X319 to LX-X?, LX-X305 to LX-X?, LX-X323 to LX-X?, LX-X307 to LX-X?, LX-X318 to LX-X?, LX-X302 to LX-X?, LX-X324 to LX-X?, LX-X331 to LX-X?, LX-X311 to LX-X?, LX-X320 to LX-X?, LX-X329 to LX-X?, LX-X328 to LX-X?, LX-X325 to LX-X?, LX-X309 to LX-X?, LX-X321 to LX-X?, LX301 to LX?, Ω?301 to Ω?, Ω?302 to Ω?, Ω?303 to Ω?
Connections:
- net at Eccosorb?.: now also LPF?.; no longer L:?. (x12)
- net at Eccosorb?.: now also L:?.; no longer LPF?. (x12)
- new net: Eccosorb?., L:?. (x12)
- new net: Eccosorb?., LPF?. (x14)
