File: XLD/Q1_2023/L4.kicad_sch (KiCad schematic)
At the start: 298 parts

Commit message: done
Connections:
- net at Eccosorb532.: now also L:548.; no longer LPF523.
- net at Eccosorb501.: now also L:502.; no longer LPF501.
- net at Eccosorb502.: now also LPF502.; no longer L:504.
- net at Eccosorb521.: now also Ω?502.; no longer LPF512.
- net at Eccosorb504.: now also L:508.; no longer LPF504.
- net at Eccosorb526.: now also L:536.; no longer LPF517.
- net at Eccosorb531.: now also LPF522.; no longer L:546.
- net at Eccosorb503.: now also LPF503.; no longer L:506.
- net at Eccosorb505.: now also LPF505.; no longer L:510.
- net at Eccosorb523.: now also LPF514.; no longer L:530.
- net at Eccosorb528.: now also LPF519.; no longer L:540.
- net at Eccosorb522.: now also L:528.; no longer LPF513.
- net at Eccosorb527.: now also LPF518.; no longer L:538.
- net at Eccosorb524.: now also L:532.; no longer LPF515.
- net at Eccosorb529.: now also L:542.; no longer LPF520.
- net at Eccosorb525.: now also LPF516.; no longer L:534.
- net at Eccosorb530.: now also LPF521.; no longer L:544.
- new net: Eccosorb532., LPF523.
- new net: Eccosorb501., LPF501.
- new net: Eccosorb502., L:504.
- new net: Eccosorb517., LPF508.
- new net: Eccosorb521., LPF512.
- new net: Eccosorb504., LPF504.
- new net: Eccosorb518., LPF509.
- new net: Eccosorb526., LPF517.
- new net: Eccosorb531., L:546.
- new net: Eccosorb503., L:506.
- new net: Eccosorb505., L:510.
- new net: Eccosorb523., L:530.
- new net: Eccosorb528., L:540.
- new net: Eccosorb519., LPF510.
- new net: Eccosorb522., LPF513.
- new net: Eccosorb527., L:538.
- new net: Eccosorb524., LPF515.
- new net: Eccosorb516., LPF507.
- new net: Eccosorb529., LPF520.
- new net: Eccosorb515., LPF506.
- new net: Eccosorb525., L:534.
- new net: Eccosorb530., L:544.

Commit message: Corrected but path not verified
Connections:
- net at Eccosorb532.: now also L:548.; no longer LPF523.
- net at Eccosorb501.: now also L:502.; no longer LPF501.
- net at Eccosorb502.: now also LPF502.; no longer L:504.
- net at Eccosorb521.: now also Ω?502.; no longer LPF512.
- net at Eccosorb504.: now also L:508.; no longer LPF504.
- net at Eccosorb526.: now also L:536.; no longer LPF517.
- net at Eccosorb531.: now also LPF522.; no longer L:546.
- net at Eccosorb503.: now also LPF503.; no longer L:506.
- net at Eccosorb505.: now also LPF505.; no longer L:510.
- net at Eccosorb523.: now also LPF514.; no longer L:530.
- net at Eccosorb528.: now also LPF519.; no longer L:540.
- net at Eccosorb522.: now also L:528.; no longer LPF513.
- net at Eccosorb527.: now also LPF518.; no longer L:538.
- net at Eccosorb524.: now also L:532.; no longer LPF515.
- net at Eccosorb529.: now also L:542.; no longer LPF520.
- net at Eccosorb525.: now also LPF516.; no longer L:534.
- net at Eccosorb530.: now also LPF521.; no longer L:544.
- new net: Eccosorb532., LPF523.
- new net: Eccosorb501., LPF501.
- new net: Eccosorb502., L:504.
- new net: Eccosorb517., LPF508.
- new net: Eccosorb521., LPF512.
- new net: Eccosorb504., LPF504.
- new net: Eccosorb518., LPF509.
- new net: Eccosorb526., LPF517.
- new net: Eccosorb531., L:546.
- new net: Eccosorb503., L:506.
- new net: Eccosorb505., L:510.
- new net: Eccosorb523., L:530.
- new net: Eccosorb528., L:540.
- new net: Eccosorb519., LPF510.
- new net: Eccosorb522., LPF513.
- new net: Eccosorb527., L:538.
- new net: Eccosorb524., LPF515.
- new net: Eccosorb516., LPF507.
- new net: Eccosorb529., LPF520.
- new net: Eccosorb515., LPF506.
- new net: Eccosorb525., L:534.
- new net: Eccosorb530., L:544.

Commit message: filter fixed'
Parts:
- LPF?: renamed from LPF523; value F‐30‐8000‐R -> F-30-8000-R; symbol Quantum Computing:F‐30‐8000‐R -> Quantum Computing:F-30-8000-R
- LPF?: renamed from LPF517; value F‐30‐8000‐R -> F-30-8000-R; symbol Quantum Computing:F‐30‐8000‐R -> Quantum Computing:F-30-8000-R
- LPF?: renamed from LPF513; value F‐30‐8000‐R -> F-30-8000-R; symbol Quantum Computing:F‐30‐8000‐R -> Quantum Computing:F-30-8000-R
- LPF?: renamed from LPF522; value F‐30‐8000‐R -> F-30-8000-R; symbol Quantum Computing:F‐30‐8000‐R -> Quantum Computing:F-30-8000-R
- LPF?: renamed from LPF520; value F‐30‐8000‐R -> F-30-8000-R; symbol Quantum Computing:F‐30‐8000‐R -> Quantum Computing:F-30-8000-R
- LPF?: renamed from LPF515; value F‐30‐8000‐R -> F-30-8000-R; symbol Quantum Computing:F‐30‐8000‐R -> Quantum Computing:F-30-8000-R
- LPF?: renamed from LPF514; value F‐30‐8000‐R -> F-30-8000-R; symbol Quantum Computing:F‐30‐8000‐R -> Quantum Computing:F-30-8000-R
- LPF?: renamed from LPF519; value F‐30‐8000‐R -> F-30-8000-R; symbol Quantum Computing:F‐30‐8000‐R -> Quantum Computing:F-30-8000-R
- LPF?: renamed from LPF516; value F‐30‐8000‐R -> F-30-8000-R; symbol Quantum Computing:F‐30‐8000‐R -> Quantum Computing:F-30-8000-R
- LPF?: renamed from LPF518; value F‐30‐8000‐R -> F-30-8000-R; symbol Quantum Computing:F‐30‐8000‐R -> Quantum Computing:F-30-8000-R
- LPF?: renamed from LPF521; value F‐30‐8000‐R -> F-30-8000-R; symbol Quantum Computing:F‐30‐8000‐R -> Quantum Computing:F-30-8000-R
- renumbered ATT595 to ATT?, ATT606 to ATT?, ATT532 to ATT?, ATT543 to ATT?, ATT551 to ATT?, ATT602 to ATT?, ATT503 to ATT?, ATT639 to ATT?, ATT640 to ATT?, ATT632 to ATT?, ATT510 to ATT?, ATT567 to ATT?, ATT507 to ATT?, ATT523 to ATT?, ATT592 to ATT?, ATT611 to ATT?, ATT560 to ATT?, ATT525 to ATT?, ATT511 to ATT?, ATT513 to ATT?, ATT504 to ATT?, ATT570 to ATT?, ATT558 to ATT?, ATT561 to ATT?, ATT526 to ATT?, ATT653 to ATT?, ATT548 to ATT?, ATT564 to ATT?, ATT559 to ATT?, ATT538 to ATT?, ATT645 to ATT?, ATT594 to ATT?, ATT627 to ATT?, ATT524 to ATT?, ATT521 to ATT?, ATT589 to ATT?, ATT599 to ATT?, ATT536 to ATT?, ATT604 to ATT?, ATT517 to ATT?, ATT590 to ATT?, ATT506 to ATT?, ATT658 to ATT?, ATT546 to ATT?, ATT566 to ATT?, ATT637 to ATT?, ATT644 to ATT?, ATT626 to ATT?, ATT617 to ATT?, ATT641 to ATT?, ATT598 to ATT?, ATT537 to ATT?, ATT575 to ATT?, ATT659 to ATT?, ATT522 to ATT?, ATT562 to ATT?, ATT633 to ATT?, ATT541 to ATT?, ATT574 to ATT?, ATT509 to ATT?, ATT528 to ATT?, ATT648 to ATT?, ATT651 to ATT?, ATT621 to ATT?, ATT612 to ATT?, ATT643 to ATT?, ATT533 to ATT?, ATT631 to ATT?, ATT624 to ATT?, ATT654 to ATT?, ATT577 to ATT?, ATT565 to ATT?, ATT625 to ATT?, ATT652 to ATT?, ATT531 to ATT?, ATT515 to ATT?, ATT656 to ATT?, ATT660 to ATT?, ATT529 to ATT?, ATT573 to ATT?, ATT613 to ATT?, ATT584 to ATT?, ATT545 to ATT?, ATT549 to ATT?, ATT563 to ATT?, ATT534 to ATT?, ATT601 to ATT?, ATT512 to ATT?, ATT587 to ATT?, ATT615 to ATT?, ATT547 to ATT?, ATT646 to ATT?, ATT581 to ATT?, ATT623 to ATT?, ATT527 to ATT?, ATT596 to ATT?, ATT608 to ATT?, ATT642 to ATT?, ATT540 to ATT?, ATT582 to ATT?, ATT622 to ATT?, ATT605 to ATT?, ATT583 to ATT?, ATT650 to ATT?, ATT544 to ATT?, ATT571 to ATT?, ATT516 to ATT?, ATT597 to ATT?, ATT600 to ATT?, ATT535 to ATT?, ATT603 to ATT?, ATT508 to ATT?, ATT501 to ATT?, ATT619 to ATT?, ATT502 to ATT?, ATT520 to ATT?, ATT636 to ATT?, ATT586 to ATT?, ATT649 to ATT?, ATT550 to ATT?, ATT635 to ATT?, ATT505 to ATT?, ATT629 to ATT?, ATT579 to ATT?, ATT542 to ATT?, ATT620 to ATT?, ATT568 to ATT?, ATT569 to ATT?, ATT634 to ATT?, ATT607 to ATT?, ATT514 to ATT?, ATT647 to ATT?, ATT539 to ATT?, ATT519 to ATT?, ATT580 to ATT?, ATT553 to ATT?, ATT657 to ATT?, ATT518 to ATT?, ATT616 to ATT?, ATT591 to ATT?, ATT585 to ATT?, ATT655 to ATT?, ATT554 to ATT?, ATT614 to ATT?, ATT610 to ATT?, ATT555 to ATT?, ATT578 to ATT?, ATT630 to ATT?, ATT572 to ATT?, ATT588 to ATT?, ATT628 to ATT?, ATT609 to ATT?, ATT593 to ATT?, ATT557 to ATT?, ATT638 to ATT?, ATT530 to ATT?, ATT552 to ATT?, ATT576 to ATT?, ATT618 to ATT?, ATT556 to ATT?, Eccosorb532 to Eccosorb?, Eccosorb502 to Eccosorb?, Eccosorb517 to Eccosorb?, Eccosorb507 to Eccosorb?, Eccosorb518 to Eccosorb?, Eccosorb510 to Eccosorb?, Eccosorb519 to Eccosorb?, Eccosorb526 to Eccosorb?, Eccosorb514 to Eccosorb?, Eccosorb505 to Eccosorb?, Eccosorb527 to Eccosorb?, Eccosorb504 to Eccosorb?, Eccosorb524 to Eccosorb?, Eccosorb522 to Eccosorb?, Eccosorb511 to Eccosorb?, Eccosorb509 to Eccosorb?, Eccosorb506 to Eccosorb?, Eccosorb531 to Eccosorb?, Eccosorb523 to Eccosorb?, Eccosorb520 to Eccosorb?, Eccosorb529 to Eccosorb?, Eccosorb516 to Eccosorb?, Eccosorb508 to Eccosorb?, Eccosorb525 to Eccosorb?, Eccosorb528 to Eccosorb?, Eccosorb530 to Eccosorb?, Eccosorb521 to Eccosorb?, Eccosorb501 to Eccosorb?, Eccosorb515 to Eccosorb?, Eccosorb503 to Eccosorb?, Eccosorb513 to Eccosorb?, Eccosorb512 to Eccosorb?, L:515 to L:?, L:533 to L:?, L:501 to L:?, L:511 to L:?, L:548 to L:?, L:546 to L:?, L:506 to L:?, L:510 to L:?, L:524 to L:?, L:530 to L:?, L:518 to L:?, L:509 to L:?, L:519 to L:?, L:503 to L:?, L:508 to L:?, L:540 to L:?, L:529 to L:?, L:545 to L:?, L:541 to L:?, L:522 to L:?, L:502 to L:?, L:516 to L:?, L:537 to L:?, L:520 to L:?, L:507 to L:?, L:531 to L:?, L:512 to L:?, L:526 to L:?, L:538 to L:?, L:547 to L:?, L:517 to L:?, L:534 to L:?, L:513 to L:?, L:535 to L:?, L:504 to L:?, L:539 to L:?, L:542 to L:?, L:525 to L:?, L:528 to L:?, L:544 to L:?, L:514 to L:?, L:543 to L:?, L:521 to L:?, L:523 to L:?, L:505 to L:?, L:527 to L:?, L:536 to L:?, L:532 to L:?, LPF501 to LPF?, LPF512 to LPF?, LPF504 to LPF?, LPF509 to LPF?, LPF511 to LPF?, LPF503 to LPF?, LPF508 to LPF?, LPF507 to LPF?, LPF506 to LPF?, LPF505 to LPF?, LPF502 to LPF?, LPF510 to LPF?, LX-X519 to LX-X?, LX-X517 to LX-X?, LX-X516 to LX-X?, LX-X507 to LX-X?, LX-X506 to LX-X?, LX-X514 to LX-X?, LX-X509 to LX-X?, LX-X526 to LX-X?, LX-X504 to LX-X?, LX-X503 to LX-X?, LX-X520 to LX-X?, LX-X505 to LX-X?, LX-X531 to LX-X?, LX-X518 to LX-X?, LX-X512 to LX-X?, LX-X511 to LX-X?, LX-X501 to LX-X?, LX-X525 to LX-X?, LX-X521 to LX-X?, LX-X527 to LX-X?, LX-X529 to LX-X?, LX-X515 to LX-X?, LX-X528 to LX-X?, LX-X508 to LX-X?, LX-X524 to LX-X?, LX-X523 to LX-X?, LX-X532 to LX-X?, LX-X510 to LX-X?, LX-X513 to LX-X?, LX-X502 to LX-X?, LX-X522 to LX-X?, LX-X530 to LX-X?, LX501 to LX?, Ω?501 to Ω?, Ω?502 to Ω?
Connections:
- net at Eccosorb?.: now also L:?.; no longer LPF?. (x7)
- net at Eccosorb?.: now also LPF?.; no longer L:?. (x9)
- net at Eccosorb?.: now also Ω?.; no longer LPF?.
- new net: Eccosorb?., LPF?. (x13)
- new net: Eccosorb?., L:?. (x9)
