File: XLD/Q1_2023/qblox_192_168_0_20.kicad_sch (KiCad schematic)
At the start: 12 parts

Commit message: done
Parts:
- removed QCM_RF603, QCM_RF604: QBlox_QCM_RF, symbol Quantum Computing:QBlox_QCM_RF
Connections:
- net 20_mod12_o1 is gone; now on an unnamed net: QCM_RF604. (o2)
- net 20_mod12_o2 is gone; now on an unnamed net: QCM_RF604. (o2)
- net 20_mod14_o1 is gone; now on an unnamed net: QRM_RF601. (o4)
- net 20_mod14_o2 is gone; now on an unnamed net: QRM_RF601. (o4)
- net 20_mod14_o3 is gone; now on an unnamed net: QRM_RF601. (o4)
- net 20_mod14_o4 is gone; now on an unnamed net: QRM_RF601. (o4)
- net 20_mod19_o1 is gone; now on an unnamed net: QRM_RF601. (o4)
- net 20_mod19_o2 is gone; now on an unnamed net: QRM_RF601. (o4)
- net 20_mod19_o3 is gone; now on an unnamed net: QRM_RF601. (o4)
- net 20_mod19_o4 is gone; now on an unnamed net: QRM_RF601. (o4)
- net 20_ro_out_mod16_mod18 is gone; now on net 20_ro_out_mod12_mod16: SC601.
- net 20_mod18_i1: now reaches QRM_RF601. (o1)
- net 20_mod18_i1: no longer SC602.
- net at IP602. (9): now also QRM_RF601. (o1); no longer QRM_RF601. (o1)
- net 20_ro_out_mod12_mod16: now reaches SC601.
- net 20_ro_out_mod12_mod16: no longer QRM_RF601. (o1)
- net at QCM602. (o4): now also IP602. (9)
- net at QCM_RF604. (o2): now also SC601.; no longer IP602. (9)
- net 20_mod16_i1: now reaches QRM_RF601. (o1)
- net 20_mod16_i1: no longer IP602. (9)
- net 20_ro_in_mod16_mod18 renamed 20_ro_out_mod12_mod18
- net 20_ro_out_mod12_mod18: no longer QRM_RF601. (o1)
- new net: QRM_RF601. (o1), SC602.
- new net: QCM_RF604. (o2), SC602.
- new net: IP602. (9), QRM_RF601. (o1)
- new net: IP602. (9), QCM_RF604. (o2)
- new net: IP602. (9), QCM601. (Trig)
- new net: QRM_RF601. (o1), SC601.
- no-connect marks 7 -> 15

Commit message: Corrected but path not verified
Connections:
- net at QRM_RF601. (o4): now also IP602. (9) (x2)
- net at IP602. (9): now also QRM_RF601. (o1); no longer QRM_RF601. (o4)
- net at QCM_RF604. (o2): now also SC601.; no longer SC602.
- net at QCM602. (o4): now also IP602. (9)
- new net: QRM_RF601. (o1), SC602.
- new net: QCM_RF604. (o2), SC602.
- new net: IP602. (9), QRM_RF601. (o1)
- new net: IP602. (9), QCM_RF604. (o2)
- new net: IP602. (9), QCM601. (Trig)
- new net: QRM_RF601. (o1), SC601.

Commit message: filter fixed'
Connections:
- net at QRM_RF601. (o4): now also IP602. (9) (x2)
- net at IP602. (9): now also QRM_RF601. (o1); no longer QRM_RF601. (o4)
- net at QCM_RF604. (o2): now also SC601.; no longer SC602.
- net at QCM602. (o4): now also IP602. (9)
- new net: QRM_RF601. (o1), SC602.
- new net: QCM_RF604. (o2), SC602.
- new net: IP602. (9), QRM_RF601. (o1)
- new net: IP602. (9), QCM_RF604. (o2)
- new net: IP602. (9), QCM601. (Trig)
- new net: QRM_RF601. (o1), SC601.
Changed lines of the file:
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@@
         )
         (path "/9924af8b-9fcb-4325-a1dc-18dd2c4184d7/01ac70ae-656e-4c1c-b9e0-89039088ad17"
-          (reference "QCM803") (unit 1)
+          (reference "QCM?") (unit 1)
         )
       )
@@
         )
         (path "/9924af8b-9fcb-4325-a1dc-18dd2c4184d7/01ac70ae-656e-4c1c-b9e0-89039088ad17"
-          (reference "QRM_RF802") (unit 1)
+          (reference "QRM_RF?") (unit 1)
         )
       )
@@
         )
         (path "/9924af8b-9fcb-4325-a1dc-18dd2c4184d7/01ac70ae-656e-4c1c-b9e0-89039088ad17"
-          (reference "QCM802") (unit 1)
+          (reference "QCM?") (unit 1)
         )
       )
@@
         )
         (path "/9924af8b-9fcb-4325-a1dc-18dd2c4184d7/01ac70ae-656e-4c1c-b9e0-89039088ad17"
-          (reference "QRM801") (unit 1)
+          (reference "QRM?") (unit 1)
         )
       )
@@
         )
         (path "/9924af8b-9fcb-4325-a1dc-18dd2c4184d7/01ac70ae-656e-4c1c-b9e0-89039088ad17"
-          (reference "QCM_RF803") (unit 1)
+          (reference "QCM_RF?") (unit 1)
         )
       )
@@
         )
         (path "/9924af8b-9fcb-4325-a1dc-18dd2c4184d7/01ac70ae-656e-4c1c-b9e0-89039088ad17"
-          (reference "QCM801") (unit 1)
+          (reference "QCM?") (unit 1)
         )
       )
@@
         )
         (path "/9924af8b-9fcb-4325-a1dc-18dd2c4184d7/01ac70ae-656e-4c1c-b9e0-89039088ad17"
-          (reference "QRM_RF801") (unit 1)
-        )
-      )
+          (reference "QRM_RF?") (unit 1)
+        )
+      )
