File: XLD/Q1_2023/qblox_192_168_0_6.kicad_sch (KiCad schematic)
At the start: 11 parts

Commit message: done
Connections:
- net at IP601. (9): now also QCM_RF602. (o2); no longer QCM603. (o4)
- new net: IP601. (9), QCM603. (o4)
- new net: IP601. (9), QCM602. (o4)
- new net: IP601. (9), QCM_RF601. (o2)
- new net: IP601. (9), QCM_RF603. (o2)
- new net: IP601. (9), QRM_RF602. (o1)
- new net: IP601. (9), QRM_RF601. (o1)
- new net: IP601. (9), QCM601. (Trig)
Changed lines of the file:
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@@
     (pin "")
     (instances
-      (project "KiCad 25qF"
+      (project "Q1_2023"
         (path "/9924af8b-9fcb-4325-a1dc-18dd2c4184d7/2b9d3711-dc59-4b0f-99b7-021db4c5fe7b"
           (reference "QCM603") (unit 1)
@@
     (pin "")
     (instances
-      (project "KiCad 25qF"
+      (project "Q1_2023"
         (path "/9924af8b-9fcb-4325-a1dc-18dd2c4184d7/2b9d3711-dc59-4b0f-99b7-021db4c5fe7b"
           (reference "QCM602") (unit 1)
@@
     (pin "")
     (instances
-      (project "KiCad 25qF"
+      (project "Q1_2023"
         (path "/9924af8b-9fcb-4325-a1dc-18dd2c4184d7/2b9d3711-dc59-4b0f-99b7-021db4c5fe7b"
           (reference "QCM_RF601") (unit 1)
@@
     (pin "")
     (instances
-      (project "KiCad 25qF"
+      (project "Q1_2023"
         (path "/9924af8b-9fcb-4325-a1dc-18dd2c4184d7/2b9d3711-dc59-4b0f-99b7-021db4c5fe7b"
           (reference "QCM_RF603") (unit 1)
@@
     (pin "")
     (instances
-      (project "KiCad 25qF"
+      (project "Q1_2023"
         (path "/9924af8b-9fcb-4325-a1dc-18dd2c4184d7/2b9d3711-dc59-4b0f-99b7-021db4c5fe7b"
           (reference "SC601") (unit 1)
@@
     (pin "")
     (instances
-      (project "KiCad 25qF"
+      (project "Q1_2023"
         (path "/9924af8b-9fcb-4325-a1dc-18dd2c4184d7/2b9d3711-dc59-4b0f-99b7-021db4c5fe7b"
           (reference "IP601") (unit 1)
@@
     (pin "")
     (instances
-      (project "KiCad 25qF"
+      (project "Q1_2023"
         (path "/9924af8b-9fcb-4325-a1dc-18dd2c4184d7/2b9d3711-dc59-4b0f-99b7-021db4c5fe7b"
           (reference "QRM_RF602") (unit 1)
@@
     (pin "")
     (instances
-      (project "KiCad 25qF"
+      (project "Q1_2023"
         (path "/9924af8b-9fcb-4325-a1dc-18dd2c4184d7/2b9d3711-dc59-4b0f-99b7-021db4c5fe7b"
           (reference "QRM_RF601") (unit 1)
@@
     (pin "")
     (instances
-      (project "KiCad 25qF"
+      (project "Q1_2023"
         (path "/9924af8b-9fcb-4325-a1dc-18dd2c4184d7/2b9d3711-dc59-4b0f-99b7-021db4c5fe7b"
           (reference "SC602") (unit 1)
@@
     (pin "")
     (instances
-      (project "KiCad 25qF"
+      (project "Q1_2023"
         (path "/9924af8b-9fcb-4325-a1dc-18dd2c4184d7/2b9d3711-dc59-4b0f-99b7-021db4c5fe7b"
           (reference "QCM601") (unit 1)
@@
     (pin "")
     (instances
-      (project "KiCad 25qF"
+      (project "Q1_2023"
         (path "/9924af8b-9fcb-4325-a1dc-18dd2c4184d7/2b9d3711-dc59-4b0f-99b7-021db4c5fe7b"
           (reference "QCM_RF602") (unit 1)

Commit message: Corrected but path not verified
Connections:
- net at IP601. (9): now also QCM_RF602. (o2); no longer QCM603. (o4)
- new net: IP601. (9), QCM603. (o4)
- new net: IP601. (9), QCM602. (o4)
- new net: IP601. (9), QCM_RF601. (o2)
- new net: IP601. (9), QCM_RF603. (o2)
- new net: IP601. (9), QRM_RF602. (o1)
- new net: IP601. (9), QRM_RF601. (o1)
- new net: IP601. (9), QCM601. (Trig)

Commit message: filter fixed'
Parts:
- renumbered QCM603 to QCM?, QCM602 to QCM?, QCM601 to QCM?, QCM_RF601 to QCM_RF?, QCM_RF603 to QCM_RF?, QCM_RF602 to QCM_RF?, QRM_RF602 to QRM_RF?, QRM_RF601 to QRM_RF?
Connections:
- net at IP601. (9): now also QCM_RF?. (o2); no longer QCM?. (o4)
- new net: IP601. (9), QCM?. (o4) (x2)
- new net: IP601. (9), QCM_RF?. (o2) (x2)
- new net: IP601. (9), QRM_RF?. (o1) (x2)
- new net: IP601. (9), QCM?. (Trig)
Changed lines of the file:
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@@
   (symbol (lib_id "Quantum Computing:QBlox_QCM") (at 201.93 137.795 0) (unit 1)
     (in_bom yes) (on_board no) (dnp no) (fields_autoplaced)
-    (property "Reference" "QCM603" (at 200.025 139.827 0)
+    (property "Reference" "QCM?" (at 200.025 139.827 0)
       (effects (font (size 1.27 1.27)) (justify left))
     )
@@
       (project "Q1_2023"
         (path "/9924af8b-9fcb-4325-a1dc-18dd2c4184d7/2b9d3711-dc59-4b0f-99b7-021db4c5fe7b"
-          (reference "QCM603") (unit 1)
+          (reference "QCM?") (unit 1)
         )
         (path "/9924af8b-9fcb-4325-a1dc-18dd2c4184d7/01ac70ae-656e-4c1c-b9e0-89039088ad17"
@@
   (symbol (lib_id "Quantum Computing:QBlox_QCM") (at 142.875 137.795 0) (unit 1)
     (in_bom yes) (on_board no) (dnp no) (fields_autoplaced)
-    (property "Reference" "QCM602" (at 140.97 139.827 0)
+    (property "Reference" "QCM?" (at 140.97 139.827 0)
       (effects (font (size 1.27 1.27)) (justify left))
     )
@@
       (project "Q1_2023"
         (path "/9924af8b-9fcb-4325-a1dc-18dd2c4184d7/2b9d3711-dc59-4b0f-99b7-021db4c5fe7b"
-          (reference "QCM602") (unit 1)
+          (reference "QCM?") (unit 1)
         )
         (path "/9924af8b-9fcb-4325-a1dc-18dd2c4184d7/01ac70ae-656e-4c1c-b9e0-89039088ad17"
@@
   (symbol (lib_id "Quantum Computing:QBlox_QCM_RF") (at 162.56 137.795 0) (unit 1)
     (in_bom yes) (on_board no) (dnp no) (fields_autoplaced)
-    (property "Reference" "QCM_RF601" (at 160.655 139.827 0)
+    (property "Reference" "QCM_RF?" (at 160.655 139.827 0)
       (effects (font (size 1.27 1.27)) (justify left))
     )
@@
       (project "Q1_2023"
         (path "/9924af8b-9fcb-4325-a1dc-18dd2c4184d7/2b9d3711-dc59-4b0f-99b7-021db4c5fe7b"
-          (reference "QCM_RF601") (unit 1)
+          (reference "QCM_RF?") (unit 1)
         )
         (path "/9924af8b-9fcb-4325-a1dc-18dd2c4184d7/01ac70ae-656e-4c1c-b9e0-89039088ad17"
@@
   (symbol (lib_id "Quantum Computing:QBlox_QCM_RF") (at 260.985 137.795 0) (unit 1)
     (in_bom yes) (on_board no) (dnp no) (fields_autoplaced)
-    (property "Reference" "QCM_RF603" (at 259.08 139.827 0)
+    (property "Reference" "QCM_RF?" (at 259.08 139.827 0)
       (effects (font (size 1.27 1.27)) (justify left))
     )
@@
       (project "Q1_2023"
         (path "/9924af8b-9fcb-4325-a1dc-18dd2c4184d7/2b9d3711-dc59-4b0f-99b7-021db4c5fe7b"
-          (reference "QCM_RF603") (unit 1)
+          (reference "QCM_RF?") (unit 1)
         )
         (path "/9924af8b-9fcb-4325-a1dc-18dd2c4184d7/01ac70ae-656e-4c1c-b9e0-89039088ad17"
@@
   (symbol (lib_id "Quantum Computing:QBlox_QRM_RF") (at 339.725 137.795 0) (unit 1)
     (in_bom yes) (on_board no) (dnp no) (fields_autoplaced)
-    (property "Reference" "QRM_RF602" (at 337.82 139.827 0)
+    (property "Reference" "QRM_RF?" (at 337.82 139.827 0)
       (effects (font (size 1.27 1.27)) (justify left))
     )
@@
       (project "Q1_2023"
         (path "/9924af8b-9fcb-4325-a1dc-18dd2c4184d7/2b9d3711-dc59-4b0f-99b7-021db4c5fe7b"
-          (reference "QRM_RF602") (unit 1)
+          (reference "QRM_RF?") (unit 1)
         )
         (path "/9924af8b-9fcb-4325-a1dc-18dd2c4184d7/01ac70ae-656e-4c1c-b9e0-89039088ad17"
@@
   (symbol (lib_id "Quantum Computing:QBlox_QRM_RF") (at 300.355 137.795 0) (unit 1)
     (in_bom yes) (on_board no) (dnp no) (fields_autoplaced)
-    (property "Reference" "QRM_RF601" (at 298.45 139.827 0)
+    (property "Reference" "QRM_RF?" (at 298.45 139.827 0)
       (effects (font (size 1.27 1.27)) (justify left))
     )
@@
       (project "Q1_2023"
         (path "/9924af8b-9fcb-4325-a1dc-18dd2c4184d7/2b9d3711-dc59-4b0f-99b7-021db4c5fe7b"
-          (reference "QRM_RF601") (unit 1)
+          (reference "QRM_RF?") (unit 1)
         )
         (path "/9924af8b-9fcb-4325-a1dc-18dd2c4184d7/01ac70ae-656e-4c1c-b9e0-89039088ad17"
@@
   (symbol (lib_id "Quantum Computing:QBlox_CTRL") (at 102.235 137.795 0) (unit 1)
     (in_bom yes) (on_board no) (dnp no) (fields_autoplaced)
-    (property "Reference" "QCM601" (at 100.33 139.827 0)
+    (property "Reference" "QCM?" (at 100.33 139.827 0)
       (effects (font (size 1.27 1.27)) (justify left))
     )
@@
       (project "Q1_2023"
         (path "/9924af8b-9fcb-4325-a1dc-18dd2c4184d7/2b9d3711-dc59-4b0f-99b7-021db4c5fe7b"
-          (reference "QCM601") (unit 1)
+          (reference "QCM?") (unit 1)
         )
         (path "/9924af8b-9fcb-4325-a1dc-18dd2c4184d7/01ac70ae-656e-4c1c-b9e0-89039088ad17"
@@
   (symbol (lib_id "Quantum Computing:QBlox_QCM_RF") (at 182.245 137.795 0) (unit 1)
     (in_bom yes) (on_board no) (dnp no) (fields_autoplaced)
-    (property "Reference" "QCM_RF602" (at 180.34 139.827 0)
+    (property "Reference" "QCM_RF?" (at 180.34 139.827 0)
       (effects (font (size 1.27 1.27)) (justify left))
     )
@@
       (project "Q1_2023"
         (path "/9924af8b-9fcb-4325-a1dc-18dd2c4184d7/2b9d3711-dc59-4b0f-99b7-021db4c5fe7b"
-          (reference "QCM_RF602") (unit 1)
-        )
-        (path "/9924af8b-9fcb-4325-a1dc-18dd2c4184d7/01ac70ae-656e-4c1c-b9e0-89039088ad17"
+          (reference "QCM_RF?") (unit 1)
+        )
+        (path "/9924af8b-9fcb-4325-a1dc-18dd2c4184d7/01ac70ae-656e-4c1c-b9e0-89039088ad17"
