File: XLD/Q2_2023/L1.kicad_sch (KiCad schematic)
At the start: 176 parts

Commit message: mend
Connections:
- net at L:?.: now also TJI?.; no longer HEMT?. (gnd)
- net at TJI?.: now also L:?.; no longer L:?.
- net at L:?.: now also Coupler?.; no longer TWPA?.
- net at Coupler?.: now also L:?.; no longer L:?. (x2)
- net at L:?.: now also TWPA?.; no longer Coupler?.
- net at TWPA?.: now also L:?.; no longer L:?.
- new net: Eccosorb?., LPF?. (x23)
- new net: HEMT?. (gnd), L:?.
- new net: L:?., TJI?.
- new net: L:?., TWPA?.
- new net: Coupler?., L:?.
- new net: ATT?., ATT?.

Commit message: more updates
Connections:
- net L3-10: no longer Coupler?.20dB
- net L3-16: no longer Coupler?.20dB
- net at L:?.: now also TJI?.; no longer HEMT?. (gnd)
- net at TJI?.: now also L:?.; no longer L:?.
- net at L:?.: now also Coupler?.; no longer TWPA?.
- net at Coupler?.: now also L:?.; no longer L:?. (x2)
- net at L:?.: now also TWPA?.; no longer Coupler?.
- net at TWPA?.: no longer L:?. (x2)
- new net: Eccosorb?., LPF?. (x23)
- new net: HEMT?. (gnd), L:?.
- new net: L:?., TJI?.
- new net: L:?., TWPA?.
- new net: Coupler?., L:?.
- new net: ATT?., ATT?.
- now unconnected: TWPA?.
Other:
- moved on the sheet: TWPA?
Changed lines of the file:
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@@
     )
     (property "Value" "SMA-SMP" (at 621.665 262.89 0)
-      (effects (font (size 0.64 0.64)))
+      (effects (font (size 1 1)))
     )
     (property "Footprint" "" (at 621.03 262.89 0)
@@
     )
     (property "Value" "SMA-SMP" (at 525.145 262.89 0)
-      (effects (font (size 0.64 0.64)))
+      (effects (font (size 1 1)))
     )
     (property "Footprint" "" (at 524.51 262.89 0)
@@
     )
     (property "Value" "SMA-SMP" (at 380.365 262.89 0)
-      (effects (font (size 0.64 0.64)))
+      (effects (font (size 1 1)))
     )
     (property "Footprint" "" (at 379.73 262.89 0)
@@
     )
     (property "Value" "SMA-SMA" (at 90.805 267.97 0)
-      (effects (font (size 0.64 0.64)))
+      (effects (font (size 1 1)))
     )
     (property "Footprint" "" (at 90.17 267.97 0)
@@
     )
     (property "Value" "SMA-SMP" (at 476.885 262.89 0)
-      (effects (font (size 0.64 0.64)))
+      (effects (font (size 1 1)))
     )
     (property "Footprint" "" (at 476.25 262.89 0)
@@
     )
     (property "Value" "SMA-SMA_small" (at 90.805 219.075 0)
-      (effects (font (size 0.64 0.64)))
+      (effects (font (size 1 1)))
     )
     (property "Footprint" "" (at 90.17 219.075 0)
@@
     )
     (property "Value" "SMA-SMA" (at 114.935 240.03 0)
-      (effects (font (size 0.64 0.64)))
+      (effects (font (size 1 1)))
     )
     (property "Footprint" "" (at 114.3 240.03 0)
@@
     )
     (property "Value" "SMA-SMA_small" (at 114.935 219.075 0)
-      (effects (font (size 0.64 0.64)))
+      (effects (font (size 1 1)))
     )
     (property "Footprint" "" (at 114.3 219.075 0)
@@
     )
     (property "Value" "SMA-SMA" (at 90.805 240.03 0)
-      (effects (font (size 0.64 0.64)))
+      (effects (font (size 1 1)))
     )
     (property "Footprint" "" (at 90.17 240.03 0)
@@
     )
     (property "Value" "SMA-SMP" (at 404.495 262.89 0)
-      (effects (font (size 0.64 0.64)))
+      (effects (font (size 1 1)))
     )
     (property "Footprint" "" (at 403.86 262.89 0)
@@
     )
     (property "Value" "SMA-SMP" (at 597.535 262.89 0)
-      (effects (font (size 0.64 0.64)))
+      (effects (font (size 1 1)))
     )
     (property "Footprint" "" (at 596.9 262.89 0)
@@
     )
     (property "Value" "SMA-SMP" (at 573.405 262.89 0)
-      (effects (font (size 0.64 0.64)))
+      (effects (font (size 1 1)))
     )
     (property "Footprint" "" (at 572.77 262.89 0)
@@
     )
     (property "Value" "SMA-SMA" (at 114.935 267.97 0)
-      (effects (font (size 0.64 0.64)))
+      (effects (font (size 1 1)))
     )
     (property "Footprint" "" (at 114.3 267.97 0)
@@
     )
     (property "Value" "SMA-SMA" (at 114.935 201.93 0)
-      (effects (font (size 0.64 0.64)))
+      (effects (font (size 1 1)))
     )
     (property "Footprint" "" (at 114.3 201.93 0)
@@
     )
     (property "Value" "SMA-SMP" (at 549.275 263.525 0)
-      (effects (font (size 0.64 0.64)))
+      (effects (font (size 1 1)))
     )
     (property "Footprint" "" (at 548.64 263.525 0)
@@
     )
     (property "Value" "SMA-SMA" (at 114.935 170.18 0)
-      (effects (font (size 0.64 0.64)))
+      (effects (font (size 1 1)))
     )
     (property "Footprint" "" (at 114.3 170.18 0)
@@
     )
     (property "Value" "SMA-SMP" (at 452.755 262.89 0)
-      (effects (font (size 0.64 0.64)))
+      (effects (font (size 1 1)))
     )
     (property "Footprint" "" (at 452.12 262.89 0)
@@
     )
     (property "Value" "SMA-SMA" (at 90.805 201.93 0)
-      (effects (font (size 0.64 0.64)))
+      (effects (font (size 1 1)))
     )
     (property "Footprint" "" (at 90.17 201.93 0)
@@
     )
     (property "Value" "SMA-SMP" (at 645.795 262.89 0)
-      (effects (font (size 0.64 0.64)))
+      (effects (font (size 1 1)))
     )
     (property "Footprint" "" (at 645.16 262.89 0)
@@
     )
     (property "Value" "SMA-SMP" (at 356.235 262.89 0)
-      (effects (font (size 0.64 0.64)))
+      (effects (font (size 1 1)))
     )
     (property "Footprint" "" (at 355.6 262.89 0)
@@
     )
     (property "Value" "SMA-SMP" (at 669.925 262.89 0)
-      (effects (font (size 0.64 0.64)))
+      (effects (font (size 1 1)))
     )
     (property "Footprint" "" (at 669.29 262.89 0)
@@
     )
     (property "Value" "SMA-SMP" (at 501.015 262.89 0)
-      (effects (font (size 0.64 0.64)))
+      (effects (font (size 1 1)))
     )
     (property "Footprint" "" (at 500.38 262.89 0)
@@
     )
     (property "Value" "SMA-SMP" (at 332.105 262.89 0)
-      (effects (font (size 0.64 0.64)))
+      (effects (font (size 1 1)))
     )
     (property "Footprint" "" (at 331.47 262.89 0)
