File: XLD/Q2_2023/L2.kicad_sch (KiCad schematic)
At the start: 61 parts

Commit message: mend
Connections:
- net at L:?.: now also TJI?.; no longer Coupler?.
- net at TJI?.: now also L:?.; no longer L:?. (x2)
- net at TJI?.: no longer L:?.
- net at L:?.: now also TWPA?.; no longer TJI?.
- net at TWPA?.: now also L:?.; no longer L:?.
- new net: L:?., TJI?. (x8)
- new net: Coupler?., L:?.

Commit message: more updates
Connections:
- net L3-28: no longer Coupler?.20dB
- net at L:?.: now also TJI?.; no longer Coupler?.
- net at TJI?.: now also L:?.; no longer L:?. (x2)
- net at TJI?.: no longer L:?.
- net at L:?.: no longer TJI?.
- net at TWPA?.: no longer L:?.
- new net: L:?., TJI?. (x8)
- new net: Coupler?., L:?.
Other:
- moved on the sheet: TWPA?
Changed lines of the file:
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@@
     )
     (property "Value" "SMA-SMA" (at 194.945 321.945 0)
-      (effects (font (size 0.64 0.64)))
+      (effects (font (size 1 1)))
     )
     (property "Footprint" "" (at 194.31 321.945 0)
@@
     )
     (property "Value" "SMA-SMA" (at 363.855 252.095 0)
-      (effects (font (size 0.64 0.64)))
+      (effects (font (size 1 1)))
     )
     (property "Footprint" "" (at 363.22 252.095 0)
@@
     )
     (property "Value" "SMA-SMA" (at 484.505 252.095 0)
-      (effects (font (size 0.64 0.64)))
+      (effects (font (size 1 1)))
     )
     (property "Footprint" "" (at 483.87 252.095 0)
@@
     )
     (property "Value" "SMA-SMA" (at 194.945 252.095 0)
-      (effects (font (size 0.64 0.64)))
+      (effects (font (size 1 1)))
     )
     (property "Footprint" "" (at 194.31 252.095 0)
@@
     )
     (property "Value" "SMA-SMA" (at 98.425 249.555 0)
-      (effects (font (size 0.64 0.64)))
+      (effects (font (size 1 1)))
     )
     (property "Footprint" "" (at 97.79 249.555 0)
@@
     )
     (property "Value" "SMA-SMA" (at 146.685 249.555 0)
-      (effects (font (size 0.64 0.64)))
+      (effects (font (size 1 1)))
     )
     (property "Footprint" "" (at 146.05 249.555 0)
@@
     )
     (property "Value" "SMA-SMA" (at 194.945 283.845 0)
-      (effects (font (size 0.64 0.64)))
+      (effects (font (size 1 1)))
     )
     (property "Footprint" "" (at 194.31 283.845 0)
@@
     )
     (property "Value" "SMA-SMA_small" (at 194.945 300.99 0)
-      (effects (font (size 0.64 0.64)))
+      (effects (font (size 1 1)))
     )
     (property "Footprint" "" (at 194.31 300.99 0)
@@
     )
     (property "Value" "SMA-SMA" (at 122.555 250.19 0)
-      (effects (font (size 0.64 0.64)))
+      (effects (font (size 1 1)))
     )
     (property "Footprint" "" (at 121.92 250.19 0)
@@
     )
     (property "Value" "SMA-SMA" (at 243.205 250.825 0)
-      (effects (font (size 0.64 0.64)))
+      (effects (font (size 1 1)))
     )
     (property "Footprint" "" (at 242.57 250.825 0)
@@
     )
     (property "Value" "SMA-SMA" (at 170.815 250.19 0)
-      (effects (font (size 0.64 0.64)))
+      (effects (font (size 1 1)))
     )
     (property "Footprint" "" (at 170.18 250.19 0)
@@
     )
     (property "Value" "SMA-SMP" (at 194.945 350.52 0)
-      (effects (font (size 0.64 0.64)))
+      (effects (font (size 1 1)))
     )
     (property "Footprint" "" (at 194.31 350.52 0)
