File: XLD/Q2_2023/L3.kicad_sch (KiCad schematic)
At the start: 298 parts

Commit message: mend
Connections:
- net at Eccosorb?.: now also LPF?.; no longer L:?. (x12)
- net at Eccosorb?.: now also L:?.; no longer LPF?. (x12)
- new net: Eccosorb?., L:?. (x12)
- new net: Eccosorb?., LPF?. (x14)

Commit message: more updates
Connections:
- net at Eccosorb?.: now also LPF?.; no longer L:?. (x12)
- net at Eccosorb?.: now also L:?.; no longer LPF?. (x12)
- new net: Eccosorb?., L:?. (x12)
- new net: Eccosorb?., LPF?. (x14)
Changed lines of the file:
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@@
     )
     (property "Value" "SMA-SMP" (at 475.615 280.67 0)
-      (effects (font (size 0.64 0.64)))
+      (effects (font (size 1 1)))
     )
     (property "Footprint" "" (at 474.98 280.67 0)
@@
     )
     (property "Value" "SMA-SMP" (at 451.485 280.67 0)
-      (effects (font (size 0.64 0.64)))
+      (effects (font (size 1 1)))
     )
     (property "Footprint" "" (at 450.85 280.67 0)
@@
     )
     (property "Value" "SMA-SMP" (at 210.185 280.67 0)
-      (effects (font (size 0.64 0.64)))
+      (effects (font (size 1 1)))
     )
     (property "Footprint" "" (at 209.55 280.67 0)
@@
     )
     (property "Value" "SMA-SMP" (at 741.045 274.32 0)
-      (effects (font (size 0.64 0.64)))
+      (effects (font (size 1 1)))
     )
     (property "Footprint" "" (at 740.41 274.32 0)
@@
     )
     (property "Value" "SMA-SMA" (at 668.655 279.4 0)
-      (effects (font (size 0.64 0.64)))
+      (effects (font (size 1 1)))
     )
     (property "Footprint" "" (at 668.02 279.4 0)
@@
     )
     (property "Value" "SMA-SMP" (at 161.925 280.67 0)
-      (effects (font (size 0.64 0.64)))
+      (effects (font (size 1 1)))
     )
     (property "Footprint" "" (at 161.29 280.67 0)
@@
     )
     (property "Value" "SMA-SMP" (at 572.135 279.4 0)
-      (effects (font (size 0.64 0.64)))
+      (effects (font (size 1 1)))
     )
     (property "Footprint" "" (at 571.5 279.4 0)
@@
     )
     (property "Value" "SMA-SMP" (at 306.705 280.67 0)
-      (effects (font (size 0.64 0.64)))
+      (effects (font (size 1 1)))
     )
     (property "Footprint" "" (at 306.07 280.67 0)
@@
     )
     (property "Value" "SMA-SMP" (at 234.315 280.67 0)
-      (effects (font (size 0.64 0.64)))
+      (effects (font (size 1 1)))
     )
     (property "Footprint" "" (at 233.68 280.67 0)
@@
     )
     (property "Value" "SMA-SMA" (at 644.525 279.4 0)
-      (effects (font (size 0.64 0.64)))
+      (effects (font (size 1 1)))
     )
     (property "Footprint" "" (at 643.89 279.4 0)
@@
     )
     (property "Value" "SMA-SMP" (at 789.305 275.59 0)
-      (effects (font (size 0.64 0.64)))
+      (effects (font (size 1 1)))
     )
     (property "Footprint" "" (at 788.67 275.59 0)
@@
     )
     (property "Value" "SMA-SMP" (at 330.835 280.67 0)
-      (effects (font (size 0.64 0.64)))
+      (effects (font (size 1 1)))
     )
     (property "Footprint" "" (at 330.2 280.67 0)
@@
     )
     (property "Value" "SMA-SMP" (at 354.965 280.67 0)
-      (effects (font (size 0.64 0.64)))
+      (effects (font (size 1 1)))
     )
     (property "Footprint" "" (at 354.33 280.67 0)
@@
     )
     (property "Value" "SMA-SMA" (at 620.395 283.845 0)
-      (effects (font (size 0.64 0.64)))
+      (effects (font (size 1 1)))
     )
     (property "Footprint" "" (at 619.76 283.845 0)
@@
     )
     (property "Value" "SMA-SMP" (at 258.445 280.67 0)
-      (effects (font (size 0.64 0.64)))
+      (effects (font (size 1 1)))
     )
     (property "Footprint" "" (at 257.81 280.67 0)
@@
     )
     (property "Value" "SMA-SMP" (at 403.225 280.67 0)
-      (effects (font (size 0.64 0.64)))
+      (effects (font (size 1 1)))
     )
     (property "Footprint" "" (at 402.59 280.67 0)
@@
     )
     (property "Value" "SMA-SMP" (at 596.265 279.4 0)
-      (effects (font (size 0.64 0.64)))
+      (effects (font (size 1 1)))
     )
     (property "Footprint" "" (at 595.63 279.4 0)
@@
     )
     (property "Value" "SMA-SMP" (at 861.695 275.59 0)
-      (effects (font (size 0.64 0.64)))
+      (effects (font (size 1 1)))
     )
     (property "Footprint" "" (at 861.06 275.59 0)
@@
     )
     (property "Value" "SMA-SMP" (at 765.175 274.32 0)
-      (effects (font (size 0.64 0.64)))
+      (effects (font (size 1 1)))
     )
     (property "Footprint" "" (at 764.54 274.32 0)
@@
     )
     (property "Value" "SMA-SMA" (at 716.915 280.035 0)
-      (effects (font (size 0.64 0.64)))
+      (effects (font (size 1 1)))
     )
     (property "Footprint" "" (at 716.28 280.035 0)
@@
     )
     (property "Value" "SMA-SMP" (at 499.745 280.67 0)
-      (effects (font (size 0.64 0.64)))
+      (effects (font (size 1 1)))
     )
     (property "Footprint" "" (at 499.11 280.67 0)
@@
     )
     (property "Value" "SMA-SMP" (at 282.575 280.67 0)
-      (effects (font (size 0.64 0.64)))
+      (effects (font (size 1 1)))
     )
     (property "Footprint" "" (at 281.94 280.67 0)
@@
     )
     (property "Value" "SMA-SMP" (at 186.055 280.67 0)
-      (effects (font (size 0.64 0.64)))
+      (effects (font (size 1 1)))
     )
     (property "Footprint" "" (at 185.42 280.67 0)
@@
     )
     (property "Value" "SMA-SMP" (at 427.355 280.67 0)
-      (effects (font (size 0.64 0.64)))
+      (effects (font (size 1 1)))
     )
     (property "Footprint" "" (at 426.72 280.67 0)
