File: XLD/Q2_2023/L4.kicad_sch (KiCad schematic)
At the start: 298 parts

Commit message: mend
Connections:
- net at Eccosorb?.: now also L:?.; no longer LPF?. (x7)
- net at Eccosorb?.: now also LPF?.; no longer L:?. (x9)
- net at Eccosorb?.: now also Ω?.; no longer LPF?.
- new net: Eccosorb?., LPF?. (x13)
- new net: Eccosorb?., L:?. (x9)

Commit message: more updates
Connections:
- net at Eccosorb?.: now also L:?.; no longer LPF?. (x7)
- net at Eccosorb?.: now also LPF?.; no longer L:?. (x9)
- net at Eccosorb?.: now also Ω?.; no longer LPF?.
- new net: Eccosorb?., LPF?. (x13)
- new net: Eccosorb?., L:?. (x9)
Changed lines of the file:
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@@
     )
     (property "Value" "SMA-SMP" (at 909.955 270.51 0)
-      (effects (font (size 0.64 0.64)))
+      (effects (font (size 1 1)))
     )
     (property "Footprint" "" (at 909.32 270.51 0)
@@
     )
     (property "Value" "SMA-SMP" (at 885.825 270.51 0)
-      (effects (font (size 0.64 0.64)))
+      (effects (font (size 1 1)))
     )
     (property "Footprint" "" (at 885.19 270.51 0)
@@
     )
     (property "Value" "SMA-SMP" (at 210.185 275.59 0)
-      (effects (font (size 0.64 0.64)))
+      (effects (font (size 1 1)))
     )
     (property "Footprint" "" (at 209.55 275.59 0)
@@
     )
     (property "Value" "SMA-SMP" (at 258.445 275.59 0)
-      (effects (font (size 0.64 0.64)))
+      (effects (font (size 1 1)))
     )
     (property "Footprint" "" (at 257.81 275.59 0)
@@
     )
     (property "Value" "SMA-SMP" (at 692.785 270.51 0)
-      (effects (font (size 0.64 0.64)))
+      (effects (font (size 1 1)))
     )
     (property "Footprint" "" (at 692.15 270.51 0)
@@
     )
     (property "Value" "SMA-SMP" (at 234.315 275.59 0)
-      (effects (font (size 0.64 0.64)))
+      (effects (font (size 1 1)))
     )
     (property "Footprint" "" (at 233.68 275.59 0)
@@
     )
     (property "Value" "SMA-SMP" (at 813.435 270.51 0)
-      (effects (font (size 0.64 0.64)))
+      (effects (font (size 1 1)))
     )
     (property "Footprint" "" (at 812.8 270.51 0)
@@
     )
     (property "Value" "SMA-SMP" (at 161.925 275.59 0)
-      (effects (font (size 0.64 0.64)))
+      (effects (font (size 1 1)))
     )
     (property "Footprint" "" (at 161.29 275.59 0)
@@
     )
     (property "Value" "SMA-SMP" (at 789.305 270.51 0)
-      (effects (font (size 0.64 0.64)))
+      (effects (font (size 1 1)))
     )
     (property "Footprint" "" (at 788.67 270.51 0)
@@
     )
     (property "Value" "SMA-SMP" (at 741.045 270.51 0)
-      (effects (font (size 0.64 0.64)))
+      (effects (font (size 1 1)))
     )
     (property "Footprint" "" (at 740.41 270.51 0)
@@
     )
     (property "Value" "SMA-SMP" (at 186.055 275.59 0)
-      (effects (font (size 0.64 0.64)))
+      (effects (font (size 1 1)))
     )
     (property "Footprint" "" (at 185.42 275.59 0)
@@
     )
     (property "Value" "SMA-SMP" (at 837.565 270.51 0)
-      (effects (font (size 0.64 0.64)))
+      (effects (font (size 1 1)))
     )
     (property "Footprint" "" (at 836.93 270.51 0)
@@
     )
     (property "Value" "SMA-SMP" (at 668.655 270.51 0)
-      (effects (font (size 0.64 0.64)))
+      (effects (font (size 1 1)))
     )
     (property "Footprint" "" (at 668.02 270.51 0)
@@
     )
     (property "Value" "SMA-SMP" (at 861.695 270.51 0)
-      (effects (font (size 0.64 0.64)))
+      (effects (font (size 1 1)))
     )
     (property "Footprint" "" (at 861.06 270.51 0)
@@
     )
     (property "Value" "SMA-SMP" (at 765.175 270.51 0)
-      (effects (font (size 0.64 0.64)))
+      (effects (font (size 1 1)))
     )
     (property "Footprint" "" (at 764.54 270.51 0)
@@
     )
     (property "Value" "SMA-SMP" (at 716.915 270.51 0)
-      (effects (font (size 0.64 0.64)))
+      (effects (font (size 1 1)))
     )
     (property "Footprint" "" (at 716.28 270.51 0)
