File: XLD/Q2_2023/ZI.kicad_sch (KiCad schematic)
At the start: 0 parts

Commit message: Improvements to library components, title, date
Other:
- company: (none) -> Technology Innovation Institute
- title: (none) -> XLD Setup Q2 2023
Changed lines of the file:
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@@
 (kicad_sch (version 20230121) (generator eeschema)
   (paper "A2")
+  (title_block
+    (title "XLD Setup Q2 2023")
+    (date "2023-06-14")
+    (company "Technology Innovation Institute")
+  )
 )
