File: XLD/Q2_2023/qw25q.kicad_sch (KiCad schematic)
At the start: 423 parts

Commit message: mend
Connections:
- net at Eccosorb?.: now also LPF?.; no longer L:?. (x11)
- net at Eccosorb?.: now also L:?.; no longer LPF?. (x14)
- net at TJI?.: now also L:?. (x2)
- net at TJI?.: no longer L:?. (x2)
- new net: Eccosorb?., L:?. (x11)
- new net: Eccosorb?., LPF?. (x35)
- new net: L:?., TJI?. (x2)
Other:
- moved on the sheet: ATT?, Eccosorb?, HEMT?, L:?, LPF?, LX-X?, LX?, QPU?, TJI?

Commit message: more updates
Connections:
- net L2-1: now also TJI?.
- net L2-2: now also TJI?.
- net L2-3: now also TJI?.
- net L2-4: now also TJI?.
- net at Eccosorb?.: now also LPF?.; no longer L:?. (x11)
- net at Eccosorb?.: now also L:?.; no longer LPF?. (x14)
- new net: Eccosorb?., L:?. (x11)
- new net: Eccosorb?., LPF?. (x35)
- new net: ATT?., HEMT?. (gnd) (x4)
- new net: L:?., TJI?. (x4)
Other:
- note added: "100mK"
- note added: "1K"
- note added: "20mK"
- note added: "300K"
- note added: "4K"
- note added: "50K"
- moved on the sheet: ATT?, Eccosorb?, HEMT?, L:?, LPF?, LX-X?, TJI?

Commit message: update attenuators and pumplines
Parts:
- removed LX?: RF-Feedthrough-32, symbol Quantum Computing:RF-Feedthrough-32
- removed TJI? (x4): LNF-ISISC4_12A, symbol Quantum Computing:LNF-ISISC4_12A
- added ATT1 (x4): Attenuator 0-Cryo, symbol Quantum Computing:Attenuator 0-Cryo
- added ATT322, ATT323, ATT324, ATT325, ATT326: Attenuator 3-Cryo, symbol Quantum Computing:Attenuator 6-Cryo
- added ATT327, ATT328, ATT329, ATT330, ATT331, ATT332, ATT333, ATT334, ATT335, ATT336: Attenuator 1-Cryo, symbol Quantum Computing:Attenuator 6-Cryo
- added ATT337, ATT338, ATT339, ATT340, ATT341, ATT342, ATT343, ATT344, ATT345, ATT346, ATT347, ATT348, ATT349, ATT350, ATT351, ATT352: Attenuator 0-Cryo, symbol Quantum Computing:Attenuator 6-Cryo
- added ATT4 (x4): Attenuator 1-Cryo, symbol Quantum Computing:Attenuator 0-Cryo
- added ATT6 (x4): Attenuator 20-Cryo, symbol Quantum Computing:Attenuator 20-Cryo
- added ATT7 (x4): Attenuator 6-Cryo, symbol Quantum Computing:Attenuator 6-Cryo
- added ATT8 (x4): Attenuator 10-Cryo, symbol Quantum Computing:Attenuator 3-Cryo
- added Coupler1 (x4): QMC-CRYOCOUPLER-20, symbol Quantum Computing:QMC-CRYOCOUPLER-20
- added L:1 (x8), L:2 (x4), L:4 (x4): SMA-SMA, symbol Quantum Computing:SMA-SMA
- added L:3 (x4): SMA-SMA_small, symbol Quantum Computing:SMA-SMA_small
- added L:5 (x4): SMA-SMP, symbol Quantum Computing:SMA-SMP
- added L:6 (x4): COAX-6FT, symbol Quantum Computing:COAX-6FT
- added LO9 (x4): LO_R&S, symbol Quantum Computing:LO_R&S
- added LX-X2 (x4): NbTi-RF-line, symbol Quantum Computing:NbTi-RF-line
- added TJI1 (x4), TJI2 (x4): LNF-ISISC4_12A, symbol Quantum Computing:LNF-ISISC4_12A
- added TWPA1 (x4): SW_TWPA, symbol Quantum Computing:SW_TWPA
- ATT10, ATT12, ATT14, ATT156, ATT158, ATT16, ATT160, ATT162, ATT164, ATT166, ATT168, ATT170, ATT172, ATT18, ATT20, ATT25: renamed from ATT?; value Attenuator 0-Cryo -> Attenuator 3-Cryo
- ATT11, ATT13, ATT15, ATT155, ATT157, ATT159, ATT161, ATT163, ATT165, ATT167, ATT169, ATT17, ATT171, ATT173, ATT174, ATT175, ATT176, ATT177, ATT178, ATT19, ATT21: renamed from ATT?; value Attenuator 20-Cryo -> Attenuator 10-Cryo
- gave numbers to parts that had none: 380
Connections:
- net L1-11: now also ATT346.
- net L1-12: now also ATT345.
- net L1-13: now also ATT344.
- net L1-14: now also ATT343.
- net L1-15: now also ATT342.
- net L1-16: now also ATT341.
- net L1-17: now also ATT340.
- net L1-18: now also ATT339.
- net L1-19: now also ATT338.
- net L1-20: now also ATT337.
- net L1-21: now also ATT322., ATT327., ATT332.
- net L1-22: now also ATT323., ATT328., ATT333.
- net L1-23: now also ATT324., ATT329., ATT334.
- net L1-24: now also ATT325., ATT330., ATT335.
- net L1-25: now also ATT326., ATT331., ATT336.
- net L1-4: now also ATT352.
- net L1-5: now also ATT351.
- net L1-6: now also ATT350.
- net L1-7: now also ATT349.
- net L1-8: now also ATT348.
- net L1-9: now also ATT347.
- net L2-1: now also L:5.
- net L2-2: now also L:5.
- net L2-3: now also L:5.
- net L2-4: now also L:5.
- net L3-1: now also LO9.
- net at Eccosorb56.: now also LPF47.; no longer L:96.
- net at Eccosorb60.: now also LPF51.; no longer L:104.
- net at Eccosorb34.: now also L:5.; no longer LPF25.
- net at Eccosorb84.: now also L:153.; no longer LPF75.
- net at Eccosorb54.: now also LPF45.; no longer L:92.
- net at Eccosorb92.: now also LPF83.; no longer L:170.
- net at Eccosorb59.: now also L:102.; no longer LPF50.
- net at Eccosorb57.: now also L:98.; no longer LPF48.
- net at Eccosorb61.: now also L:106.; no longer LPF52.
- net at Eccosorb53.: now also L:27.; no longer LPF44.
- net at Eccosorb91.: now also L:168.; no longer LPF82.
- net at Eccosorb51.: now also LPF42.; no longer L:9.
- net at Eccosorb50.: now also LPF41.; no longer L:7.
- net at Eccosorb66.: now also LPF57.; no longer L:116.
- net at Eccosorb2.: now also L:3.; no longer LPF2.
- net at Eccosorb65.: now also L:114.; no longer LPF56.
- net at Eccosorb68.: now also L:120.; no longer LPF59.
- net at Eccosorb67.: now also LPF58.; no longer L:118.
- net at Eccosorb55.: now also LPF46.; no longer L:94.
- net at Eccosorb93.: now also L:174.; no longer LPF84.
- net at Eccosorb62.: now also L:108.; no longer LPF53.
- net at Eccosorb52.: now also L:25.; no longer LPF43.
- net at Eccosorb58.: now also L:100.; no longer LPF49.
- net at Eccosorb64.: now also LPF55.; no longer L:112.
- net at Eccosorb63.: now also LPF54.; no longer L:110.
- new net: Eccosorb56., L:96.
- new net: Eccosorb60., L:104.
- new net: Eccosorb34., LPF25.
- new net: ATT329., ATT334.
- new net: Eccosorb84., LPF75.
- new net: Coupler1., L:4. (x4)
- new net: Coupler1., L:3. (x4)
- new net: Eccosorb54., L:92.
- new net: Eccosorb37., LPF28.
- new net: L:4., TJI2. (x4)
- new net: Eccosorb43., LPF34.
- new net: Eccosorb92., L:170.
- new net: Eccosorb33., LPF24.
- new net: Eccosorb59., LPF50.
- new net: Eccosorb57., LPF48.
- new net: Eccosorb39., LPF30.
- new net: ATT331., ATT336.
- new net: L:5., TJI2. (x4)
- new net: Eccosorb61., LPF52.
- new net: L:2., TWPA1. (x4)
- new net: L:3., TWPA1. (x4)
- new net: Eccosorb53., LPF44.
- new net: L:1., TJI1. (x4)
- new net: L:2., TJI1. (x4)
- new net: Eccosorb41., LPF32.
- new net: Eccosorb91., LPF82.
- new net: ATT330., ATT335.
- new net: ATT328., ATT333.
- new net: Eccosorb48., LPF39.
- new net: Eccosorb51., L:9.
- new net: L:6., LX-X2. (x3)
- new net: Eccosorb50., L:7.
- new net: Eccosorb4., LPF4.
- new net: Eccosorb66., L:116.
- new net: Eccosorb44., LPF35.
- new net: Eccosorb2., LPF2.
- new net: Eccosorb40., LPF31.
- new net: Eccosorb46., LPF37.
- new net: Eccosorb65., LPF56.
- new net: Eccosorb68., LPF59.
- new net: Eccosorb67., L:118.
- new net: Eccosorb55., L:94.
- new net: Eccosorb93., LPF84.
- new net: Eccosorb35., LPF26.
- new net: Eccosorb3., LPF3.
- new net: Eccosorb62., LPF53.
- new net: Eccosorb49., LPF40.
- new net: Eccosorb52., LPF43.
- new net: Eccosorb47., LPF38.
- new net: Eccosorb32., LPF23.
- new net: Eccosorb38., LPF29.
- new net: Eccosorb42., LPF33.
- new net: Eccosorb58., LPF49.
- new net: Eccosorb64., L:112.
- new net: Eccosorb5., LPF5.
- new net: Eccosorb63., L:110.
- new net: Eccosorb36., LPF27.
- new net: Eccosorb31., LPF11.
- new net: Eccosorb45., LPF36.
- new net L3-16: ATT1., ATT4., ATT6., ATT7., ATT8., Coupler1.20dB, L:1., L:6., LX-X2.
- new net L3-21: ATT1., ATT4., ATT6., ATT7., ATT8., Coupler1.20dB, L:1., L:6., LO9., LX-X2.
- new net L3-23: ATT1., ATT4., ATT6., ATT7., ATT8., Coupler1.20dB, L:1., L:6., LO9., LX-X2.
- new net L3-24: ATT1., ATT4., ATT6., ATT7., ATT8., Coupler1.20dB, L:1., L:6., LO9., LX-X2.
- no-connect marks 64 -> 0
Other:
- note added: "192.168.0.?"
- note added: "Brass 8inch"
- note added: "ISOLATOR-1"
- note added: "ISOLATOR-2"
- note added: "Short Brass"
- note added: "Steel one"
- moved on the sheet: ATT10, ATT11, ATT12, ATT13, ATT14, ATT15, ATT155, ATT156, ATT157, ATT158, ATT159, ATT16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

Commit message: Improvements to library components, title, date
Parts:
- ATT10, ATT12, ATT14, ATT156, ATT158, ATT16, ATT160, ATT162, ATT164, ATT166, ATT168, ATT170, ATT172, ATT18, ATT20, ATT25: symbol Quantum Computing:Attenuator 0-Cryo -> Quantum Computing:Attenuator 3-Cryo
- ATT103: renamed from ATT17; symbol Quantum Computing:Attenuator 20-Cryo -> Quantum Computing:Attenuator 10-Cryo
- ATT155: renamed from ATT19; symbol Quantum Computing:Attenuator 20-Cryo -> Quantum Computing:Attenuator 10-Cryo
- ATT157: renamed from ATT21; symbol Quantum Computing:Attenuator 20-Cryo -> Quantum Computing:Attenuator 10-Cryo
- ATT159: renamed from ATT155; symbol Quantum Computing:Attenuator 20-Cryo -> Quantum Computing:Attenuator 10-Cryo
- ATT161: renamed from ATT157; symbol Quantum Computing:Attenuator 20-Cryo -> Quantum Computing:Attenuator 10-Cryo
- ATT163: renamed from ATT159; symbol Quantum Computing:Attenuator 20-Cryo -> Quantum Computing:Attenuator 10-Cryo
- ATT165: renamed from ATT161; symbol Quantum Computing:Attenuator 20-Cryo -> Quantum Computing:Attenuator 10-Cryo
- ATT167: renamed from ATT163; symbol Quantum Computing:Attenuator 20-Cryo -> Quantum Computing:Attenuator 10-Cryo
- ATT169: renamed from ATT165; symbol Quantum Computing:Attenuator 20-Cryo -> Quantum Computing:Attenuator 10-Cryo
- ATT171: renamed from ATT167; symbol Quantum Computing:Attenuator 20-Cryo -> Quantum Computing:Attenuator 10-Cryo
- ATT173: renamed from ATT169; symbol Quantum Computing:Attenuator 20-Cryo -> Quantum Computing:Attenuator 10-Cryo
- ATT174: renamed from ATT171; symbol Quantum Computing:Attenuator 20-Cryo -> Quantum Computing:Attenuator 10-Cryo
- ATT175: renamed from ATT173; symbol Quantum Computing:Attenuator 20-Cryo -> Quantum Computing:Attenuator 10-Cryo
- ATT176: renamed from ATT322; symbol Quantum Computing:Attenuator 6-Cryo -> Quantum Computing:Attenuator 3-Cryo
- ATT177: renamed from ATT174; symbol Quantum Computing:Attenuator 20-Cryo -> Quantum Computing:Attenuator 10-Cryo
- ATT178: renamed from ATT323; symbol Quantum Computing:Attenuator 6-Cryo -> Quantum Computing:Attenuator 3-Cryo
- ATT19: renamed from ATT11; symbol Quantum Computing:Attenuator 20-Cryo -> Quantum Computing:Attenuator 10-Cryo
- ATT21: renamed from ATT13; symbol Quantum Computing:Attenuator 20-Cryo -> Quantum Computing:Attenuator 10-Cryo
- ATT298: renamed from ATT175; symbol Quantum Computing:Attenuator 20-Cryo -> Quantum Computing:Attenuator 10-Cryo
- ATT299: renamed from ATT324; symbol Quantum Computing:Attenuator 6-Cryo -> Quantum Computing:Attenuator 3-Cryo
- ATT300: renamed from ATT176; symbol Quantum Computing:Attenuator 20-Cryo -> Quantum Computing:Attenuator 10-Cryo
- ATT301: renamed from ATT325; symbol Quantum Computing:Attenuator 6-Cryo -> Quantum Computing:Attenuator 3-Cryo
- ATT305: renamed from ATT177; symbol Quantum Computing:Attenuator 20-Cryo -> Quantum Computing:Attenuator 10-Cryo
- ATT306: renamed from ATT326; symbol Quantum Computing:Attenuator 6-Cryo -> Quantum Computing:Attenuator 3-Cryo
- ATT310: renamed from ATT178; symbol Quantum Computing:Attenuator 20-Cryo -> Quantum Computing:Attenuator 10-Cryo
- ATT327: renamed from ATT352; symbol Quantum Computing:Attenuator 6-Cryo -> Quantum Computing:Attenuator 0-Cryo
- ATT328: renamed from ATT351; symbol Quantum Computing:Attenuator 6-Cryo -> Quantum Computing:Attenuator 0-Cryo
- ATT329: renamed from ATT350; symbol Quantum Computing:Attenuator 6-Cryo -> Quantum Computing:Attenuator 0-Cryo
- ATT330: renamed from ATT349; symbol Quantum Computing:Attenuator 6-Cryo -> Quantum Computing:Attenuator 0-Cryo
- ATT331: renamed from ATT348; symbol Quantum Computing:Attenuator 6-Cryo -> Quantum Computing:Attenuator 0-Cryo
- ATT332: renamed from ATT347; symbol Quantum Computing:Attenuator 6-Cryo -> Quantum Computing:Attenuator 0-Cryo
- ATT333: renamed from ATT346; symbol Quantum Computing:Attenuator 6-Cryo -> Quantum Computing:Attenuator 0-Cryo
- ATT334: renamed from ATT345; symbol Quantum Computing:Attenuator 6-Cryo -> Quantum Computing:Attenuator 0-Cryo
- ATT335: renamed from ATT344; symbol Quantum Computing:Attenuator 6-Cryo -> Quantum Computing:Attenuator 0-Cryo
- ATT336: renamed from ATT343; symbol Quantum Computing:Attenuator 6-Cryo -> Quantum Computing:Attenuator 0-Cryo
- ATT337: renamed from ATT342; symbol Quantum Computing:Attenuator 6-Cryo -> Quantum Computing:Attenuator 0-Cryo
- ATT338: renamed from ATT341; symbol Quantum Computing:Attenuator 6-Cryo -> Quantum Computing:Attenuator 0-Cryo
- ATT339: renamed from ATT340; symbol Quantum Computing:Attenuator 6-Cryo -> Quantum Computing:Attenuator 0-Cryo
- ATT340: renamed from ATT339; symbol Quantum Computing:Attenuator 6-Cryo -> Quantum Computing:Attenuator 0-Cryo
- ATT341: renamed from ATT338; symbol Quantum Computing:Attenuator 6-Cryo -> Quantum Computing:Attenuator 0-Cryo
- ATT342: renamed from ATT337; symbol Quantum Computing:Attenuator 6-Cryo -> Quantum Computing:Attenuator 0-Cryo
- ATT343: renamed from ATT327; symbol Quantum Computing:Attenuator 6-Cryo -> Quantum Computing:Attenuator 1-Cryo
- ATT344: renamed from ATT332; symbol Quantum Computing:Attenuator 6-Cryo -> Quantum Computing:Attenuator 1-Cryo
- ATT345: renamed from ATT328; symbol Quantum Computing:Attenuator 6-Cryo -> Quantum Computing:Attenuator 1-Cryo
- ATT346: renamed from ATT333; symbol Quantum Computing:Attenuator 6-Cryo -> Quantum Computing:Attenuator 1-Cryo
- ATT347: renamed from ATT329; symbol Quantum Computing:Attenuator 6-Cryo -> Quantum Computing:Attenuator 1-Cryo
- ATT348: renamed from ATT334; symbol Quantum Computing:Attenuator 6-Cryo -> Quantum Computing:Attenuator 1-Cryo
- ATT349: renamed from ATT330; symbol Quantum Computing:Attenuator 6-Cryo -> Quantum Computing:Attenuator 1-Cryo
- ATT350: renamed from ATT335; symbol Quantum Computing:Attenuator 6-Cryo -> Quantum Computing:Attenuator 1-Cryo
- ATT351: renamed from ATT331; symbol Quantum Computing:Attenuator 6-Cryo -> Quantum Computing:Attenuator 1-Cryo
- ATT352: renamed from ATT336; symbol Quantum Computing:Attenuator 6-Cryo -> Quantum Computing:Attenuator 1-Cryo
- ATT4: symbol Quantum Computing:Attenuator 0-Cryo -> Quantum Computing:Attenuator 1-Cryo
- ATT8: symbol Quantum Computing:Attenuator 3-Cryo -> Quantum Computing:Attenuator 10-Cryo
- ATT98: renamed from ATT15; symbol Quantum Computing:Attenuator 20-Cryo -> Quantum Computing:Attenuator 10-Cryo
- CBL30: renamed from L:2; value COAX-6FT -> Minicircuits-6FT; symbol Quantum Computing:COAX-6FT -> Quantum Computing:RF Cable Minicircuits-6FT
- CBL31: renamed from L:55; value COAX-6FT -> Minicircuits-6FT; symbol Quantum Computing:COAX-6FT -> Quantum Computing:RF Cable Minicircuits-6FT
- CBL32: renamed from L:4; value COAX-6FT -> Minicircuits-6FT; symbol Quantum Computing:COAX-6FT -> Quantum Computing:RF Cable Minicircuits-6FT
- CBL33: renamed from L:57; value COAX-6FT -> Minicircuits-6FT; symbol Quantum Computing:COAX-6FT -> Quantum Computing:RF Cable Minicircuits-6FT
- CBL34: renamed from L:6; value COAX-6FT -> Minicircuits-6FT; symbol Quantum Computing:COAX-6FT -> Quantum Computing:RF Cable Minicircuits-6FT
- CBL35: renamed from L:58; value COAX-6FT -> Minicircuits-6FT; symbol Quantum Computing:COAX-6FT -> Quantum Computing:RF Cable Minicircuits-6FT
- CBL36: renamed from L:8; value COAX-6FT -> Minicircuits-6FT; symbol Quantum Computing:COAX-6FT -> Quantum Computing:RF Cable Minicircuits-6FT
- CBL37: renamed from L:59; value COAX-6FT -> Minicircuits-6FT; symbol Quantum Computing:COAX-6FT -> Quantum Computing:RF Cable Minicircuits-6FT
- CBL38: renamed from L:10; value COAX-6FT -> Minicircuits-6FT; symbol Quantum Computing:COAX-6FT -> Quantum Computing:RF Cable Minicircuits-6FT
- CBL39: renamed from L:60; value COAX-6FT -> Minicircuits-6FT; symbol Quantum Computing:COAX-6FT -> Quantum Computing:RF Cable Minicircuits-6FT
- CBL40: renamed from L:26; value COAX-6FT -> Minicircuits-6FT; symbol Quantum Computing:COAX-6FT -> Quantum Computing:RF Cable Minicircuits-6FT
- CBL41: renamed from L:61; value COAX-6FT -> Minicircuits-6FT; symbol Quantum Computing:COAX-6FT -> Quantum Computing:RF Cable Minicircuits-6FT
- CBL42: renamed from L:62; value COAX-6FT -> Minicircuits-6FT; symbol Quantum Computing:COAX-6FT -> Quantum Computing:RF Cable Minicircuits-6FT
- CBL43: renamed from L:63; value COAX-6FT -> Minicircuits-6FT; symbol Quantum Computing:COAX-6FT -> Quantum Computing:RF Cable Minicircuits-6FT
- CBL44: renamed from L:93; value COAX-6FT -> Minicircuits-6FT; symbol Quantum Computing:COAX-6FT -> Quantum Computing:RF Cable Minicircuits-6FT
- CBL45: renamed from L:65; value COAX-6FT -> Minicircuits-6FT; symbol Quantum Computing:COAX-6FT -> Quantum Computing:RF Cable Minicircuits-6FT
- CBL46: renamed from L:95; value COAX-6FT -> Minicircuits-6FT; symbol Quantum Computing:COAX-6FT -> Quantum Computing:RF Cable Minicircuits-6FT
- CBL47: renamed from L:67; value COAX-6FT -> Minicircuits-6FT; symbol Quantum Computing:COAX-6FT -> Quantum Computing:RF Cable Minicircuits-6FT
- CBL48: renamed from L:69; value COAX-6FT -> Minicircuits-6FT; symbol Quantum Computing:COAX-6FT -> Quantum Computing:RF Cable Minicircuits-6FT
- CBL49: renamed from L:97; value COAX-6FT -> Minicircuits-6FT; symbol Quantum Computing:COAX-6FT -> Quantum Computing:RF Cable Minicircuits-6FT
- CBL50: renamed from L:71; value COAX-6FT -> Minicircuits-6FT; symbol Quantum Computing:COAX-6FT -> Quantum Computing:RF Cable Minicircuits-6FT
- CBL51: renamed from L:99; value COAX-6FT -> Minicircuits-6FT; symbol Quantum Computing:COAX-6FT -> Quantum Computing:RF Cable Minicircuits-6FT
- CBL52: renamed from L:72; value COAX-6FT -> Minicircuits-6FT; symbol Quantum Computing:COAX-6FT -> Quantum Computing:RF Cable Minicircuits-6FT
- CBL53: renamed from L:101; value COAX-6FT -> Minicircuits-6FT; symbol Quantum Computing:COAX-6FT -> Quantum Computing:RF Cable Minicircuits-6FT
- CBL54: renamed from L:74; value COAX-6FT -> Minicircuits-6FT; symbol Quantum Computing:COAX-6FT -> Quantum Computing:RF Cable Minicircuits-6FT
- CBL55: renamed from L:103; value COAX-6FT -> Minicircuits-6FT; symbol Quantum Computing:COAX-6FT -> Quantum Computing:RF Cable Minicircuits-6FT
- CBL56: renamed from L:76; value COAX-6FT -> Minicircuits-6FT; symbol Quantum Computing:COAX-6FT -> Quantum Computing:RF Cable Minicircuits-6FT
- CBL57: renamed from L:105; value COAX-6FT -> Minicircuits-6FT; symbol Quantum Computing:COAX-6FT -> Quantum Computing:RF Cable Minicircuits-6FT
- CBL58: renamed from L:78; value COAX-6FT -> Minicircuits-6FT; symbol Quantum Computing:COAX-6FT -> Quantum Computing:RF Cable Minicircuits-6FT
- CBL59: renamed from L:107; value COAX-6FT -> Minicircuits-6FT; symbol Quantum Computing:COAX-6FT -> Quantum Computing:RF Cable Minicircuits-6FT
- CBL60: renamed from L:80; value COAX-6FT -> Minicircuits-6FT; symbol Quantum Computing:COAX-6FT -> Quantum Computing:RF Cable Minicircuits-6FT
- CBL61: renamed from L:109; value COAX-6FT -> Minicircuits-6FT; symbol Quantum Computing:COAX-6FT -> Quantum Computing:RF Cable Minicircuits-6FT
- CBL62: renamed from L:82; value COAX-6FT -> Minicircuits-6FT; symbol Quantum Computing:COAX-6FT -> Quantum Computing:RF Cable Minicircuits-6FT
- CBL63: renamed from L:111; value COAX-6FT -> Minicircuits-6FT; symbol Quantum Computing:COAX-6FT -> Quantum Computing:RF Cable Minicircuits-6FT
- CBL64: renamed from L:84; value COAX-6FT -> Minicircuits-6FT; symbol Quantum Computing:COAX-6FT -> Quantum Computing:RF Cable Minicircuits-6FT
- CBL65: renamed from L:113; value COAX-6FT -> Minicircuits-6FT; symbol Quantum Computing:COAX-6FT -> Quantum Computing:RF Cable Minicircuits-6FT
- CBL66: renamed from L:86; value COAX-6FT -> Minicircuits-6FT; symbol Quantum Computing:COAX-6FT -> Quantum Computing:RF Cable Minicircuits-6FT
- CBL67: renamed from L:115; value COAX-6FT -> Minicircuits-6FT; symbol Quantum Computing:COAX-6FT -> Quantum Computing:RF Cable Minicircuits-6FT
- CBL68: renamed from L:88; value COAX-6FT -> Minicircuits-6FT; symbol Quantum Computing:COAX-6FT -> Quantum Computing:RF Cable Minicircuits-6FT
- CBL69: renamed from L:117; value COAX-6FT -> Minicircuits-6FT; symbol Quantum Computing:COAX-6FT -> Quantum Computing:RF Cable Minicircuits-6FT
- CBL70: renamed from L:90; value COAX-6FT -> Minicircuits-6FT; symbol Quantum Computing:COAX-6FT -> Quantum Computing:RF Cable Minicircuits-6FT
- CBL71: renamed from L:119; value COAX-6FT -> Minicircuits-6FT; symbol Quantum Computing:COAX-6FT -> Quantum Computing:RF Cable Minicircuits-6FT
- CBL72: renamed from L:152; value COAX-6FT -> Minicircuits-6FT; symbol Quantum Computing:COAX-6FT -> Quantum Computing:RF Cable Minicircuits-6FT
- CBL73: renamed from L:167; value COAX-6FT -> Minicircuits-6FT; symbol Quantum Computing:COAX-6FT -> Quantum Computing:RF Cable Minicircuits-6FT
- CBL74: renamed from L:169; value COAX-6FT -> Minicircuits-6FT; symbol Quantum Computing:COAX-6FT -> Quantum Computing:RF Cable Minicircuits-6FT
- CBL75: renamed from L:173; value COAX-6FT -> Minicircuits-6FT; symbol Quantum Computing:COAX-6FT -> Quantum Computing:RF Cable Minicircuits-6FT
- CBL80: renamed from L:121; value COAX-6FT -> Minicircuits-6FT; symbol Quantum Computing:COAX-6FT -> Quantum Computing:RF Cable Minicircuits-6FT
- CBL81: renamed from L:123; value COAX-6FT -> Minicircuits-6FT; symbol Quantum Computing:COAX-6FT -> Quantum Computing:RF Cable Minicircuits-6FT
- CBL82: renamed from L:125; value COAX-6FT -> Minicircuits-6FT; symbol Quantum Computing:COAX-6FT -> Quantum Computing:RF Cable Minicircuits-6FT
- CBL83: renamed from L:127; value COAX-6FT -> Minicircuits-6FT; symbol Quantum Computing:COAX-6FT -> Quantum Computing:RF Cable Minicircuits-6FT
- Coupler1: symbol Quantum Computing:QMC-CRYOCOUPLER-20 -> Quantum Computing:Directional Coupler QMC-CRYOCOUPLER-20
- EF27: renamed from Eccosorb2; symbol Quantum Computing:IR-10GHz -> Quantum Computing:Filter Eccosorb IR-10GHz
- EF28: renamed from Eccosorb3; symbol Quantum Computing:IR-1GHz -> Quantum Computing:Filter Eccosorb IR-1GHz
- EF29: renamed from Eccosorb34; symbol Quantum Computing:IR-10GHz -> Quantum Computing:Filter Eccosorb IR-10GHz
- EF30: renamed from Eccosorb4; symbol Quantum Computing:IR-1GHz -> Quantum Computing:Filter Eccosorb IR-1GHz
- EF31: renamed from Eccosorb50; symbol Quantum Computing:IR-10GHz -> Quantum Computing:Filter Eccosorb IR-10GHz
- EF32: renamed from Eccosorb5; symbol Quantum Computing:IR-1GHz -> Quantum Computing:Filter Eccosorb IR-1GHz
- EF33: renamed from Eccosorb51; symbol Quantum Computing:IR-10GHz -> Quantum Computing:Filter Eccosorb IR-10GHz
- EF34: renamed from Eccosorb31; symbol Quantum Computing:IR-1GHz -> Quantum Computing:Filter Eccosorb IR-1GHz
- EF35: renamed from Eccosorb52; symbol Quantum Computing:IR-10GHz -> Quantum Computing:Filter Eccosorb IR-10GHz
- EF36: renamed from Eccosorb32; symbol Quantum Computing:IR-1GHz -> Quantum Computing:Filter Eccosorb IR-1GHz
- EF37: renamed from Eccosorb53; symbol Quantum Computing:IR-10GHz -> Quantum Computing:Filter Eccosorb IR-10GHz
- EF38: renamed from Eccosorb33; symbol Quantum Computing:IR-1GHz -> Quantum Computing:Filter Eccosorb IR-1GHz
- EF39: renamed from Eccosorb54; symbol Quantum Computing:IR-10GHz -> Quantum Computing:Filter Eccosorb IR-10GHz
- EF40: renamed from Eccosorb35; symbol Quantum Computing:IR-1GHz -> Quantum Computing:Filter Eccosorb IR-1GHz
- EF41: renamed from Eccosorb55; symbol Quantum Computing:IR-10GHz -> Quantum Computing:Filter Eccosorb IR-10GHz
- EF42: renamed from Eccosorb36; symbol Quantum Computing:IR-1GHz -> Quantum Computing:Filter Eccosorb IR-1GHz
- EF43: renamed from Eccosorb56; symbol Quantum Computing:IR-10GHz -> Quantum Computing:Filter Eccosorb IR-10GHz
- EF44: renamed from Eccosorb37; symbol Quantum Computing:IR-1GHz -> Quantum Computing:Filter Eccosorb IR-1GHz
- EF45: renamed from Eccosorb38; symbol Quantum Computing:IR-1GHz -> Quantum Computing:Filter Eccosorb IR-1GHz
- EF46: renamed from Eccosorb57; symbol Quantum Computing:IR-10GHz -> Quantum Computing:Filter Eccosorb IR-10GHz
- EF47: renamed from Eccosorb39; symbol Quantum Computing:IR-1GHz -> Quantum Computing:Filter Eccosorb IR-1GHz
- EF48: renamed from Eccosorb58; symbol Quantum Computing:IR-10GHz -> Quantum Computing:Filter Eccosorb IR-10GHz
- EF49: renamed from Eccosorb40; symbol Quantum Computing:IR-1GHz -> Quantum Computing:Filter Eccosorb IR-1GHz
- EF50: renamed from Eccosorb59; symbol Quantum Computing:IR-10GHz -> Quantum Computing:Filter Eccosorb IR-10GHz
- EF51: renamed from Eccosorb41; symbol Quantum Computing:IR-1GHz -> Quantum Computing:Filter Eccosorb IR-1GHz
- EF52: renamed from Eccosorb60; symbol Quantum Computing:IR-10GHz -> Quantum Computing:Filter Eccosorb IR-10GHz
- EF53: renamed from Eccosorb42; symbol Quantum Computing:IR-1GHz -> Quantum Computing:Filter Eccosorb IR-1GHz
- EF54: renamed from Eccosorb61; symbol Quantum Computing:IR-10GHz -> Quantum Computing:Filter Eccosorb IR-10GHz
- EF55: renamed from Eccosorb43; symbol Quantum Computing:IR-1GHz -> Quantum Computing:Filter Eccosorb IR-1GHz
- EF56: renamed from Eccosorb62; symbol Quantum Computing:IR-10GHz -> Quantum Computing:Filter Eccosorb IR-10GHz
- EF57: renamed from Eccosorb44; symbol Quantum Computing:IR-1GHz -> Quantum Computing:Filter Eccosorb IR-1GHz
- EF58: renamed from Eccosorb63; symbol Quantum Computing:IR-10GHz -> Quantum Computing:Filter Eccosorb IR-10GHz
- EF59: renamed from Eccosorb45; symbol Quantum Computing:IR-1GHz -> Quantum Computing:Filter Eccosorb IR-1GHz
- EF60: renamed from Eccosorb64; symbol Quantum Computing:IR-10GHz -> Quantum Computing:Filter Eccosorb IR-10GHz
- EF61: renamed from Eccosorb46; symbol Quantum Computing:IR-1GHz -> Quantum Computing:Filter Eccosorb IR-1GHz
- EF62: renamed from Eccosorb65; symbol Quantum Computing:IR-10GHz -> Quantum Computing:Filter Eccosorb IR-10GHz
- EF63: renamed from Eccosorb47; symbol Quantum Computing:IR-1GHz -> Quantum Computing:Filter Eccosorb IR-1GHz
- EF64: renamed from Eccosorb66; symbol Quantum Computing:IR-10GHz -> Quantum Computing:Filter Eccosorb IR-10GHz
- EF65: renamed from Eccosorb48; symbol Quantum Computing:IR-1GHz -> Quantum Computing:Filter Eccosorb IR-1GHz
- EF66: renamed from Eccosorb67; symbol Quantum Computing:IR-10GHz -> Quantum Computing:Filter Eccosorb IR-10GHz
- EF67: renamed from Eccosorb49; symbol Quantum Computing:IR-1GHz -> Quantum Computing:Filter Eccosorb IR-1GHz
- EF68: renamed from Eccosorb68; symbol Quantum Computing:IR-10GHz -> Quantum Computing:Filter Eccosorb IR-10GHz
- EF69: renamed from Eccosorb84; symbol Quantum Computing:IR-10GHz -> Quantum Computing:Filter Eccosorb IR-10GHz
- EF70: renamed from Eccosorb91; symbol Quantum Computing:IR-10GHz -> Quantum Computing:Filter Eccosorb IR-10GHz
- EF71: renamed from Eccosorb92; symbol Quantum Computing:IR-10GHz -> Quantum Computing:Filter Eccosorb IR-10GHz
- EF72: renamed from Eccosorb93; symbol Quantum Computing:IR-10GHz -> Quantum Computing:Filter Eccosorb IR-10GHz
- HEMT3: symbol Quantum Computing:LNF-LNC4_8C -> Quantum Computing:Amplifier HEMT LNF-LNC4_8C
- HEMT4: renamed from HEMT1; symbol Quantum Computing:LNF-LNC4_8C -> Quantum Computing:Amplifier HEMT LNF-LNC4_8C
- HEMT5: renamed from HEMT4; symbol Quantum Computing:LNF-LNC4_8C -> Quantum Computing:Amplifier HEMT LNF-LNC4_8C
- HEMT6: renamed from HEMT5; symbol Quantum Computing:LNF-LNC4_8C -> Quantum Computing:Amplifier HEMT LNF-LNC4_8C
- L:1, L:122, L:124, L:126, L:128, L:2, L:4: symbol Quantum Computing:SMA-SMA -> Quantum Computing:RF Cable SMA-SMA
- L:100, L:102, L:104, L:106, L:108, L:110, L:112, L:114, L:116, L:118, L:120, L:153, L:168, L:170, L:174, L:25, L:27, L:3, L:5, L:64, L:66, L:68, L:7, L:70, L:73, L:75, L:77, L:79, L:81, L:83, L:85, L:87, L:89, L:9, L:91, L:92, L:94, L:96, L:98: symbol Quantum Computing:SMA-SMP -> Quantum Computing:RF Cable SMA-SMP
- L:3: value SMA-SMA_small -> SMA-SMA short; symbol Quantum Computing:SMA-SMA_small -> Quantum Computing:RF Cable SMA-SMA_short
- L:6: value COAX-6FT -> Minicircuits-6FT; symbol Quantum Computing:COAX-6FT -> Quantum Computing:RF Cable Minicircuits-6FT
- LPF18: renamed from LPF2; symbol Quantum Computing:F-30-8000-R -> Quantum Computing:Filter Low-Pass F-30-8000-R
- LPF19: renamed from LPF3; symbol Quantum Computing:VLFX-1050+ -> Quantum Computing:Filter Low-Pass VLFX-1050+
- LPF20: renamed from LPF25; symbol Quantum Computing:F-30-8000-R -> Quantum Computing:Filter Low-Pass F-30-8000-R
- LPF21: renamed from LPF4; symbol Quantum Computing:VLFX-1050+ -> Quantum Computing:Filter Low-Pass VLFX-1050+
- LPF22: renamed from LPF41; symbol Quantum Computing:F-30-8000-R -> Quantum Computing:Filter Low-Pass F-30-8000-R
- LPF23: renamed from LPF5; symbol Quantum Computing:VLFX-1050+ -> Quantum Computing:Filter Low-Pass VLFX-1050+
- LPF24: renamed from LPF42; symbol Quantum Computing:F-30-8000-R -> Quantum Computing:Filter Low-Pass F-30-8000-R
- LPF25: renamed from LPF11; symbol Quantum Computing:VLFX-1050+ -> Quantum Computing:Filter Low-Pass VLFX-1050+
- LPF26: renamed from LPF43; symbol Quantum Computing:F-30-8000-R -> Quantum Computing:Filter Low-Pass F-30-8000-R
- LPF27: renamed from LPF23; symbol Quantum Computing:VLFX-1050+ -> Quantum Computing:Filter Low-Pass VLFX-1050+
- LPF28: renamed from LPF44; symbol Quantum Computing:F-30-8000-R -> Quantum Computing:Filter Low-Pass F-30-8000-R
- LPF29: renamed from LPF24; symbol Quantum Computing:VLFX-1050+ -> Quantum Computing:Filter Low-Pass VLFX-1050+
- LPF30: renamed from LPF45; symbol Quantum Computing:F-30-8000-R -> Quantum Computing:Filter Low-Pass F-30-8000-R
- LPF31: renamed from LPF26; symbol Quantum Computing:VLFX-1050+ -> Quantum Computing:Filter Low-Pass VLFX-1050+
- LPF32: renamed from LPF46; symbol Quantum Computing:F-30-8000-R -> Quantum Computing:Filter Low-Pass F-30-8000-R
- LPF33: renamed from LPF27; symbol Quantum Computing:VLFX-1050+ -> Quantum Computing:Filter Low-Pass VLFX-1050+
- LPF34: renamed from LPF47; symbol Quantum Computing:F-30-8000-R -> Quantum Computing:Filter Low-Pass F-30-8000-R
- LPF35: renamed from LPF28; symbol Quantum Computing:VLFX-1050+ -> Quantum Computing:Filter Low-Pass VLFX-1050+
- LPF36: renamed from LPF29; symbol Quantum Computing:VLFX-1050+ -> Quantum Computing:Filter Low-Pass VLFX-1050+
- LPF37: renamed from LPF48; symbol Quantum Computing:F-30-8000-R -> Quantum Computing:Filter Low-Pass F-30-8000-R
- LPF38: renamed from LPF30; symbol Quantum Computing:VLFX-1050+ -> Quantum Computing:Filter Low-Pass VLFX-1050+
- LPF39: renamed from LPF49; symbol Quantum Computing:F-30-8000-R -> Quantum Computing:Filter Low-Pass F-30-8000-R
- LPF40: renamed from LPF31; symbol Quantum Computing:VLFX-1050+ -> Quantum Computing:Filter Low-Pass VLFX-1050+
- LPF41: renamed from LPF50; symbol Quantum Computing:F-30-8000-R -> Quantum Computing:Filter Low-Pass F-30-8000-R
- LPF42: renamed from LPF32; symbol Quantum Computing:VLFX-1050+ -> Quantum Computing:Filter Low-Pass VLFX-1050+
- LPF43: renamed from LPF51; symbol Quantum Computing:F-30-8000-R -> Quantum Computing:Filter Low-Pass F-30-8000-R
- LPF44: renamed from LPF33; symbol Quantum Computing:VLFX-1050+ -> Quantum Computing:Filter Low-Pass VLFX-1050+
- LPF45: renamed from LPF52; symbol Quantum Computing:F-30-8000-R -> Quantum Computing:Filter Low-Pass F-30-8000-R
- LPF46: renamed from LPF34; symbol Quantum Computing:VLFX-1050+ -> Quantum Computing:Filter Low-Pass VLFX-1050+
- LPF47: renamed from LPF53; symbol Quantum Computing:F-30-8000-R -> Quantum Computing:Filter Low-Pass F-30-8000-R
- LPF48: renamed from LPF35; symbol Quantum Computing:VLFX-1050+ -> Quantum Computing:Filter Low-Pass VLFX-1050+
- LPF49: renamed from LPF54; symbol Quantum Computing:F-30-8000-R -> Quantum Computing:Filter Low-Pass F-30-8000-R
- LPF50: renamed from LPF36; symbol Quantum Computing:VLFX-1050+ -> Quantum Computing:Filter Low-Pass VLFX-1050+
- LPF51: renamed from LPF55; symbol Quantum Computing:F-30-8000-R -> Quantum Computing:Filter Low-Pass F-30-8000-R
- LPF52: renamed from LPF37; symbol Quantum Computing:VLFX-1050+ -> Quantum Computing:Filter Low-Pass VLFX-1050+
- LPF53: renamed from LPF56; symbol Quantum Computing:F-30-8000-R -> Quantum Computing:Filter Low-Pass F-30-8000-R
- LPF54: renamed from LPF38; symbol Quantum Computing:VLFX-1050+ -> Quantum Computing:Filter Low-Pass VLFX-1050+
- LPF55: renamed from LPF57; symbol Quantum Computing:F-30-8000-R -> Quantum Computing:Filter Low-Pass F-30-8000-R
- LPF56: renamed from LPF39; symbol Quantum Computing:VLFX-1050+ -> Quantum Computing:Filter Low-Pass VLFX-1050+
- LPF57: renamed from LPF58; symbol Quantum Computing:F-30-8000-R -> Quantum Computing:Filter Low-Pass F-30-8000-R
- LPF58: renamed from LPF40; symbol Quantum Computing:VLFX-1050+ -> Quantum Computing:Filter Low-Pass VLFX-1050+
- LPF59: symbol Quantum Computing:F-30-8000-R -> Quantum Computing:Filter Low-Pass F-30-8000-R
- LPF60: renamed from LPF75; symbol Quantum Computing:F-30-8000-R -> Quantum Computing:Filter Low-Pass F-30-8000-R
- LPF61: renamed from LPF82; symbol Quantum Computing:F-30-8000-R -> Quantum Computing:Filter Low-Pass F-30-8000-R
- LPF62: renamed from LPF83; symbol Quantum Computing:F-30-8000-R -> Quantum Computing:Filter Low-Pass F-30-8000-R
- LPF63: renamed from LPF84; symbol Quantum Computing:F-30-8000-R -> Quantum Computing:Filter Low-Pass F-30-8000-R
- LX-X2: value NbTi-RF-line -> NbTi; symbol Quantum Computing:NbTi-RF-line -> Quantum Computing:RF Line NbTi
- QPU?: value QPU_21q_flux -> QPU QuantWare 25q; symbol Quantum Computing:QPU_21q_flux -> Quantum Computing:QPU QuantWare 25q
- RFL30: renamed from LX-X2; value NbTi-RF-line -> NbTi; symbol Quantum Computing:NbTi-RF-line -> Quantum Computing:RF Line NbTi
- RFL31: renamed from LX-X5; value NbTi-RF-line -> NbTi; symbol Quantum Computing:NbTi-RF-line -> Quantum Computing:RF Line NbTi
- RFL32: renamed from LX-X3; value NbTi-RF-line -> NbTi; symbol Quantum Computing:NbTi-RF-line -> Quantum Computing:RF Line NbTi
- RFL33: renamed from LX-X32; value NbTi-RF-line -> NbTi; symbol Quantum Computing:NbTi-RF-line -> Quantum Computing:RF Line NbTi
- RFL34: renamed from LX-X4; value NbTi-RF-line -> NbTi; symbol Quantum Computing:NbTi-RF-line -> Quantum Computing:RF Line NbTi
- RFL35: renamed from LX-X33; value NbTi-RF-line -> NbTi; symbol Quantum Computing:NbTi-RF-line -> Quantum Computing:RF Line NbTi
- RFL36: renamed from LX-X37; value NbTi-RF-line -> NbTi; symbol Quantum Computing:NbTi-RF-line -> Quantum Computing:RF Line NbTi
- RFL37: renamed from LX-X34; value NbTi-RF-line -> NbTi; symbol Quantum Computing:NbTi-RF-line -> Quantum Computing:RF Line NbTi
- RFL38: renamed from LX-X53; value NbTi-RF-line -> NbTi; symbol Quantum Computing:NbTi-RF-line -> Quantum Computing:RF Line NbTi
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Connections:
- net at EF43.: now also LPF34.; no longer L:96.
- net at EF52.: now also LPF43.; no longer L:104.
- net at EF29.: now also L:5.; no longer LPF20.
- net at EF69.: now also L:153.; no longer LPF60.
- net at Coupler1.: now also L:3.; no longer L:4. (x2)
- net at L:3.: now also TWPA1.; no longer Coupler1.
- net at EF39.: now also LPF30.; no longer L:92.
- net at L:4.: now also Coupler1.; no longer TJI2. (x2)
- net at EF71.: now also LPF62.; no longer L:170.
- net at EF50.: now also L:102.; no longer LPF41.
- net at EF46.: now also L:98.; no longer LPF37.
- net at EF54.: now also L:106.; no longer LPF45.
- net at TJI2.: now also L:4.; no longer L:5.
- net at TWPA1.: now also L:3.; no longer L:2. (x2)
- net at L:3.: now also Coupler1.; no longer TWPA1. (x2)
- net at EF37.: now also L:27.; no longer LPF28.
- net at L:1.: now also TJI1.
- net at TJI1.: now also L:2.; no longer L:1.
- net at L:2.: now also TJI1.; no longer TWPA1. (x2)
- net at TJI1.: now also L:1.; no longer L:2. (x2)
- net at EF70.: now also L:168.; no longer LPF61.
- net at EF33.: now also LPF24.; no longer L:9.
- net at EF31.: now also LPF22.; no longer L:7.
- net at EF64.: now also LPF55.; no longer L:116.
- net at EF27.: now also L:3.; no longer LPF18.
- net at EF62.: now also L:114.; no longer LPF53.
- net at EF68.: now also L:120.; no longer LPF59.
- net at EF66.: now also LPF57.; no longer L:118.
- net at EF41.: now also LPF32.; no longer L:94.
- net at L:4.: now also TJI2.; no longer Coupler1.
- net at EF72.: now also L:174.; no longer LPF63.
- net at L:2.: now also TWPA1.; no longer TJI1.
- net at EF56.: now also L:108.; no longer LPF47.
- net at TJI2.: now also L:5.; no longer L:4.
- net at EF35.: now also L:25.; no longer LPF26.
- net at EF48.: now also L:100.; no longer LPF39.
- net at EF60.: now also LPF51.; no longer L:112.
- net at EF58.: now also LPF49.; no longer L:110.
- new net: EF43., L:96.
- new net: EF52., L:104.
- new net: EF29., LPF20.
- new net: ATT347., ATT348.
- new net: EF69., LPF60.
- new net: Coupler1., L:4. (x2)
- new net: EF39., L:92.
- new net: EF44., LPF35.
- new net: L:4., TJI2.
- new net: EF55., LPF46.
- new net: EF71., L:170.
- new net: EF38., LPF29.
- new net: EF50., LPF41.
- new net: EF46., LPF37.
- new net: EF47., LPF38.
- new net: ATT351., ATT352.
- new net: EF54., LPF45.
- new net: L:5., TJI2.
- new net: L:2., TWPA1. (x3)
- new net: EF37., LPF28.
- new net: EF51., LPF42.
- new net: EF70., LPF61.
- new net: ATT349., ATT350.
- new net: ATT345., ATT346.
- new net: EF65., LPF56.
- new net: EF33., L:9.
- new net: L:6., LX-X2. (x3)
- new net: EF31., L:7.
- new net: EF30., LPF21.
- new net: EF64., L:116.
- new net: EF57., LPF48.
- new net: EF27., LPF18.
- new net: EF49., LPF40.
- new net: EF61., LPF52.
- new net: EF62., LPF53.
- new net: EF68., LPF59.
- new net: EF66., L:118.
- new net: EF41., L:94.
- new net: EF72., LPF63.
- new net: L:2., TJI1.
- new net: EF40., LPF31.
- new net: EF28., LPF19.
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Other:
- note removed: "ISOLATOR-1"
- note removed: "ISOLATOR-2"
- company: (none) -> Technology Innovation Institute
- title: (none) -> XLD Setup Q2 2023

Commit message: correct L2-12 LNA gnd, it was fixed. Changed the IQM5q drive line LP to the correct cut frequency.
Connections:
- net at EF43.: now also LPF34.; no longer L:96.
- net at EF52.: now also LPF43.; no longer L:104.
- net at EF29.: now also L:5.; no longer LPF20.
- net at EF69.: now also L:153.; no longer LPF60.
- net at Coupler1.: now also L:3.; no longer L:4. (x2)
- net at L:3.: now also TWPA1.; no longer Coupler1.
- net at EF39.: now also LPF30.; no longer L:92.
- net at L:4.: now also Coupler1.; no longer TJI2. (x2)
- net at EF71.: now also LPF62.; no longer L:170.
- net at EF50.: now also L:102.; no longer LPF41.
- net at EF46.: now also L:98.; no longer LPF37.
- net at EF54.: now also L:106.; no longer LPF45.
- net at TJI2.: now also L:4.; no longer L:5.
- net at TWPA1.: now also L:3.; no longer L:2. (x2)
- net at L:3.: now also Coupler1.; no longer TWPA1. (x2)
- net at EF37.: now also L:27.; no longer LPF28.
- net at L:1.: now also TJI1.
- net at TJI1.: now also L:2.; no longer L:1.
- net at L:2.: now also TJI1.; no longer TWPA1. (x2)
- net at TJI1.: now also L:1.; no longer L:2. (x2)
- net at EF70.: now also L:168.; no longer LPF61.
- net at EF33.: now also LPF24.; no longer L:9.
- net at EF31.: now also LPF22.; no longer L:7.
- net at EF64.: now also LPF55.; no longer L:116.
- net at EF27.: now also L:3.; no longer LPF18.
- net at EF62.: now also L:114.; no longer LPF53.
- net at EF68.: now also L:120.; no longer LPF59.
- net at EF66.: now also LPF57.; no longer L:118.
- net at EF41.: now also LPF32.; no longer L:94.
- net at L:4.: now also TJI2.; no longer Coupler1.
- net at EF72.: now also L:174.; no longer LPF63.
- net at L:2.: now also TWPA1.; no longer TJI1.
- net at EF56.: now also L:108.; no longer LPF47.
- net at TJI2.: now also L:5.; no longer L:4.
- net at EF35.: now also L:25.; no longer LPF26.
- net at EF48.: now also L:100.; no longer LPF39.
- net at EF60.: now also LPF51.; no longer L:112.
- net at EF58.: now also LPF49.; no longer L:110.
- new net: EF43., L:96.
- new net: EF52., L:104.
- new net: EF29., LPF20.
- new net: ATT347., ATT348.
- new net: EF69., LPF60.
- new net: Coupler1., L:4. (x2)
- new net: EF39., L:92.
- new net: EF44., LPF35.
- new net: L:4., TJI2.
- new net: EF55., LPF46.
- new net: EF71., L:170.
- new net: EF38., LPF29.
- new net: EF50., LPF41.
- new net: EF46., LPF37.
- new net: EF47., LPF38.
- new net: ATT351., ATT352.
- new net: EF54., LPF45.
- new net: L:5., TJI2.
- new net: L:2., TWPA1. (x3)
- new net: EF37., LPF28.
- new net: EF51., LPF42.
- new net: EF70., LPF61.
- new net: ATT349., ATT350.
- new net: ATT345., ATT346.
- new net: EF65., LPF56.
- new net: EF33., L:9.
- new net: L:6., LX-X2. (x3)
- new net: EF31., L:7.
- new net: EF30., LPF21.
- new net: EF64., L:116.
- new net: EF57., LPF48.
- new net: EF27., LPF18.
- new net: EF49., LPF40.
- new net: EF61., LPF52.
- new net: EF62., LPF53.
- new net: EF68., LPF59.
- new net: EF66., L:118.
- new net: EF41., L:94.
- new net: EF72., LPF63.
- new net: L:2., TJI1.
- new net: EF40., LPF31.
- new net: EF28., LPF19.
- new net: EF56., LPF47.
- new net: EF67., LPF58.
- new net: EF35., LPF26.
- new net: EF63., LPF54.
- new net: EF36., LPF27.
- new net: EF45., LPF36.
- new net: EF53., LPF44.
- new net: EF48., LPF39.
- new net: EF60., L:112.
- new net: EF32., LPF23.
- new net: EF58., L:110.
- new net: EF42., LPF33.
- new net: EF34., LPF25.
- new net: EF59., LPF50.
