File: XLD/Q2_2023/qw25q.kicad_sch (KiCad schematic)
At the start: 521 parts

Commit message: updating labels
Connections:
- net at EF43.: now also LPF34.; no longer L:96.
- net at EF52.: now also LPF43.; no longer L:104.
- net at EF29.: now also L:5.; no longer LPF20.
- net at EF69.: now also L:153.; no longer LPF60.
- net at Coupler1.: now also L:3.; no longer L:4. (x2)
- net at L:3.: now also TWPA1.; no longer Coupler1.
- net at EF39.: now also LPF30.; no longer L:92.
- net at L:4.: now also Coupler1.; no longer TJI2. (x2)
- net at EF71.: now also LPF62.; no longer L:170.
- net at EF50.: now also L:102.; no longer LPF41.
- net at EF46.: now also L:98.; no longer LPF37.
- net at EF54.: now also L:106.; no longer LPF45.
- net at TJI2.: now also L:4.; no longer L:5.
- net at TWPA1.: now also L:3.; no longer L:2. (x2)
- net at L:3.: now also Coupler1.; no longer TWPA1. (x2)
- net at EF37.: now also L:27.; no longer LPF28.
- net at L:1.: now also TJI1.
- net at TJI1.: now also L:2.; no longer L:1.
- net at L:2.: now also TJI1.; no longer TWPA1. (x2)
- net at TJI1.: now also L:1.; no longer L:2. (x2)
- net at EF70.: now also L:168.; no longer LPF61.
- net at EF33.: now also LPF24.; no longer L:9.
- net at EF31.: now also LPF22.; no longer L:7.
- net at EF64.: now also LPF55.; no longer L:116.
- net at EF27.: now also L:3.; no longer LPF18.
- net at EF62.: now also L:114.; no longer LPF53.
- net at EF68.: now also L:120.; no longer LPF59.
- net at EF66.: now also LPF57.; no longer L:118.
- net at EF41.: now also LPF32.; no longer L:94.
- net at L:4.: now also TJI2.; no longer Coupler1.
- net at EF72.: now also L:174.; no longer LPF63.
- net at L:2.: now also TWPA1.; no longer TJI1.
- net at EF56.: now also L:108.; no longer LPF47.
- net at TJI2.: now also L:5.; no longer L:4.
- net at EF35.: now also L:25.; no longer LPF26.
- net at EF48.: now also L:100.; no longer LPF39.
- net at EF60.: now also LPF51.; no longer L:112.
- net at EF58.: now also LPF49.; no longer L:110.
- new net: EF43., L:96.
- new net: EF52., L:104.
- new net: EF29., LPF20.
- new net: ATT347., ATT348.
- new net: EF69., LPF60.
- new net: Coupler1., L:4. (x2)
- new net: EF39., L:92.
- new net: EF44., LPF35.
- new net: L:4., TJI2.
- new net: EF55., LPF46.
- new net: EF71., L:170.
- new net: EF38., LPF29.
- new net: EF50., LPF41.
- new net: EF46., LPF37.
- new net: EF47., LPF38.
- new net: ATT351., ATT352.
- new net: EF54., LPF45.
- new net: L:5., TJI2.
- new net: L:2., TWPA1. (x3)
- new net: EF37., LPF28.
- new net: EF51., LPF42.
- new net: EF70., LPF61.
- new net: ATT349., ATT350.
- new net: ATT345., ATT346.
- new net: EF65., LPF56.
- new net: EF33., L:9.
- new net: L:6., LX-X2. (x3)
- new net: EF31., L:7.
- new net: EF30., LPF21.
- new net: EF64., L:116.
- new net: EF57., LPF48.
- new net: EF27., LPF18.
- new net: EF49., LPF40.
- new net: EF61., LPF52.
- new net: EF62., LPF53.
- new net: EF68., LPF59.
- new net: EF66., L:118.
- new net: EF41., L:94.
- new net: EF72., LPF63.
- new net: L:2., TJI1.
- new net: EF40., LPF31.
- new net: EF28., LPF19.
- new net: EF56., LPF47.
- new net: EF67., LPF58.
- new net: EF35., LPF26.
- new net: EF63., LPF54.
- new net: EF36., LPF27.
- new net: EF45., LPF36.
- new net: EF53., LPF44.
- new net: EF48., LPF39.
- new net: EF60., L:112.
- new net: EF32., LPF23.
- new net: EF58., L:110.
- new net: EF42., LPF33.
- new net: EF34., LPF25.
- new net: EF59., LPF50.

Commit message: updatede de line B 5 qubits
Connections:
- net L3-1: no longer LO9.
- net L3-16: now also LO9.
- net at EF43.: now also LPF34.; no longer L:96.
- net at EF52.: now also LPF43.; no longer L:104.
- net at EF29.: now also L:5.; no longer LPF20.
- net at EF69.: now also L:153.; no longer LPF60.
- net at Coupler1.: now also L:3.; no longer L:4. (x2)
- net at L:3.: now also TWPA1.; no longer Coupler1.
- net at EF39.: now also LPF30.; no longer L:92.
- net at L:4.: now also Coupler1.; no longer TJI2. (x2)
- net at EF71.: now also LPF62.; no longer L:170.
- net at EF50.: now also L:102.; no longer LPF41.
- net at EF46.: now also L:98.; no longer LPF37.
- net at EF54.: now also L:106.; no longer LPF45.
- net at TJI2.: now also L:4.; no longer L:5.
- net at TWPA1.: now also L:3.; no longer L:2. (x2)
- net at L:3.: now also Coupler1.; no longer TWPA1. (x2)
- net at EF37.: now also L:27.; no longer LPF28.
- net at L:1.: now also TJI1.
- net at TJI1.: now also L:2.; no longer L:1.
- net at L:2.: now also TJI1.; no longer TWPA1. (x2)
- net at TJI1.: now also L:1.; no longer L:2. (x2)
- net at EF70.: now also L:168.; no longer LPF61.
- net at EF33.: now also LPF24.; no longer L:9.
- net at EF31.: now also LPF22.; no longer L:7.
- net at EF64.: now also LPF55.; no longer L:116.
- net at EF27.: now also L:3.; no longer LPF18.
- net at EF62.: now also L:114.; no longer LPF53.
- net at EF68.: now also L:120.; no longer LPF59.
- net at EF66.: now also LPF57.; no longer L:118.
- net at EF41.: now also LPF32.; no longer L:94.
- net at L:4.: now also TJI2.; no longer Coupler1.
- net at EF72.: now also L:174.; no longer LPF63.
- net at L:2.: now also TWPA1.; no longer TJI1.
- net at EF56.: now also L:108.; no longer LPF47.
- net at TJI2.: now also L:5.; no longer L:4.
- net at EF35.: now also L:25.; no longer LPF26.
- net at EF48.: now also L:100.; no longer LPF39.
- net at EF60.: now also LPF51.; no longer L:112.
- net at EF58.: now also LPF49.; no longer L:110.
- new net: EF43., L:96.
- new net: EF52., L:104.
- new net: EF29., LPF20.
- new net: ATT347., ATT348.
- new net: EF69., LPF60.
- new net: Coupler1., L:4. (x2)
- new net: EF39., L:92.
- new net: EF44., LPF35.
- new net: L:4., TJI2.
- new net: EF55., LPF46.
- new net: EF71., L:170.
- new net: EF38., LPF29.
- new net: EF50., LPF41.
- new net: EF46., LPF37.
- new net: EF47., LPF38.
- new net: ATT351., ATT352.
- new net: EF54., LPF45.
- new net: L:5., TJI2.
- new net: L:2., TWPA1. (x3)
- new net: EF37., LPF28.
- new net: EF51., LPF42.
- new net: EF70., LPF61.
- new net: ATT349., ATT350.
- new net: ATT345., ATT346.
- new net: EF65., LPF56.
- new net: EF33., L:9.
- new net: L:6., LX-X2. (x3)
- new net: EF31., L:7.
- new net: EF30., LPF21.
- new net: EF64., L:116.
- new net: EF57., LPF48.
- new net: EF27., LPF18.
- new net: EF49., LPF40.
- new net: EF61., LPF52.
- new net: EF62., LPF53.
- new net: EF68., LPF59.
- new net: EF66., L:118.
- new net: EF41., L:94.
- new net: EF72., LPF63.
- new net: L:2., TJI1.
- new net: EF40., LPF31.
- new net: EF28., LPF19.
- new net: EF56., LPF47.
- new net: EF67., LPF58.
- new net: EF35., LPF26.
- new net: EF63., LPF54.
- new net: EF36., LPF27.
- new net: EF45., LPF36.
- new net: EF53., LPF44.
- new net: EF48., LPF39.
- new net: EF60., L:112.
- new net: EF32., LPF23.
- new net: EF58., L:110.
- new net: EF42., LPF33.
- new net: EF34., LPF25.
- new net: EF59., LPF50.
- no-connect marks 4 -> 6
Other:
- sheet qm_192_168_0_1 ports: added QM_OPX1_OPX2_INPUT, QM_OPX1_OPX2_OUTPUT; removed QM_1_I9_Q10_OUT, QM_1_IN, QM_2_I9_Q10_OUT
- note added: "192.168.0.31"
- note added: "192.168.0.36"
Changed lines of the file:
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@@
   (junction (at 401.955 142.875) (diameter 0) (color 0 0 0 0)
   )
+  (no_connect (at 788.035 417.195))
+  (no_connect (at 788.035 414.655))
   (no_connect (at 730.885 431.8))
   (no_connect (at 730.885 444.5))
@@
     (stroke (width 0) (type default))
   )
+  (wire (pts (xy 784.987 422.021) (xy 784.987 422.275))
+    (stroke (width 0) (type default))
+  )
   (wire (pts (xy 35.56 26.035) (xy 35.56 29.845))
     (stroke (width 0) (type default))
@@
     (stroke (width 0) (type default))
   )
-  (wire (pts (xy 784.86 422.275) (xy 787.4 422.275))
+  (wire (pts (xy 784.86 422.021) (xy 784.987 422.021))
     (stroke (width 0) (type default))
   )
@@
     (stroke (width 0) (type default))
   )
-  (wire (pts (xy 784.86 419.735) (xy 788.035 419.735))
-    (stroke (width 0) (type default))
-  )
   (bus (pts (xy 802.005 23.495) (xy 777.875 23.495))
     (stroke (width 0) (type default))
@@
     (stroke (width 0) (type default))
   )
+  (wire (pts (xy 784.987 422.275) (xy 787.4 422.275))
+    (stroke (width 0) (type default))
+  )
   (wire (pts (xy 340.36 468.63) (xy 340.36 485.775))
     (stroke (width 0) (type default))
@@
     (effects (font (size 1 1) (color 0 72 72 1)) (justify left bottom))
   )
-  (text "192.168.0.?\n" (at 604.52 387.35 0)
+  (text "192.168.0.31" (at 604.52 387.35 0)
     (effects (font (size 1.27 1.27)) (justify right bottom))
   )
@@
     (effects (font (size 2 2) (color 0 72 72 1)) (justify left bottom))
   )
-  (text "192.168.0.?\n" (at 648.97 387.35 0)
+  (text "192.168.0.36\n" (at 648.97 387.35 0)
     (effects (font (size 1.27 1.27)) (justify right bottom))
   )
@@
     )
   )
-  (global_label "L3-29" (shape input) (at 675.64 374.65 90) (fields_autoplaced)
+  (global_label "L3-29" (shape output) (at 675.64 374.65 90) (fields_autoplaced)
     (effects (font (size 1.27 1.27)) (justify left))
     (property "Intersheetrefs" "${INTERSHEET_REFS}" (at 675.64 365.5152 90)
@@
     )
   )
-  (global_label "L3-24" (shape input) (at 610.235 374.65 90) (fields_autoplaced)
+  (global_label "L3-24" (shape output) (at 610.235 374.65 90) (fields_autoplaced)
     (effects (font (size 1.27 1.27)) (justify left))
     (property "Intersheetrefs" "${INTERSHEET_REFS}" (at 610.235 365.5152 90)
@@
     )
   )
-  (global_label "L3-2" (shape input) (at 730.885 407.035 180) (fields_autoplaced)
+  (global_label "L3-8" (shape input) (at 730.885 407.035 180) (fields_autoplaced)
     (effects (font (size 0.64 0.64)) (justify right))
     (property "Intersheetrefs" "${INTERSHEET_REFS}" (at 726.8912 407.035 0)
@@
     )
   )
-  (global_label "L1-7" (shape input) (at 788.035 414.655 0) (fields_autoplaced)
-    (effects (font (size 0.64 0.64)) (justify left))
-    (property "Intersheetrefs" "${INTERSHEET_REFS}" (at 792.0288 414.655 0)
-      (effects (font (size 1.27 1.27)) (justify left) hide)
-    )
-  )
-  (global_label "L3-1" (shape input) (at 730.885 404.495 180) (fields_autoplaced)
+  (global_label "L3-7" (shape input) (at 730.885 404.495 180) (fields_autoplaced)
     (effects (font (size 0.64 0.64)) (justify right))
     (property "Intersheetrefs" "${INTERSHEET_REFS}" (at 726.8912 404.495 0)
@@
     )
   )
-  (global_label "L1-8" (shape input) (at 788.035 417.195 0) (fields_autoplaced)
-    (effects (font (size 0.64 0.64)) (justify left))
-    (property "Intersheetrefs" "${INTERSHEET_REFS}" (at 792.0288 417.195 0)
-      (effects (font (size 1.27 1.27)) (justify left) hide)
-    )
-  )
   (global_label "L4-23" (shape input) (at 787.4 444.5 0) (fields_autoplaced)
     (effects (font (size 0.64 0.64)) (justify left))
@@
     )
   )
-  (global_label "L3-5" (shape input) (at 788.035 404.495 0) (fields_autoplaced)
+  (global_label "L3-9" (shape input) (at 788.035 404.495 0) (fields_autoplaced)
     (effects (font (size 0.64 0.64)) (justify left))
     (property "Intersheetrefs" "${INTERSHEET_REFS}" (at 792.0288 404.495 0)
@@
     )
   )
-  (global_label "L3-1" (shape input) (at 654.685 374.65 90) (fields_autoplaced)
+  (global_label "L3-16" (shape output) (at 654.685 374.65 90) (fields_autoplaced)
     (effects (font (size 1.27 1.27)) (justify left))
-    (property "Intersheetrefs" "${INTERSHEET_REFS}" (at 654.685 366.7247 90)
+    (property "Intersheetrefs" "${INTERSHEET_REFS}" (at 654.685 365.5152 90)
       (effects (font (size 1.27 1.27)) (justify left) hide)
     )
@@
     )
   )
-  (global_label "L3-26" (shape input) (at 788.035 419.735 0) (fields_autoplaced)
-    (effects (font (size 0.64 0.64)) (justify left))
-    (property "Intersheetrefs" "${INTERSHEET_REFS}" (at 792.6383 419.735 0)
-      (effects (font (size 1.27 1.27)) (justify left) hide)
-    )
-  )
   (global_label "L1-24" (shape input) (at 756.031 401.574 90) (fields_autoplaced)
     (effects (font (size 0.64 0.64)) (justify left))
@@
     )
   )
-  (global_label "L3-23" (shape input) (at 632.46 374.65 90) (fields_autoplaced)
+  (global_label "L3-23" (shape output) (at 632.46 374.65 90) (fields_autoplaced)
     (effects (font (size 1.27 1.27)) (justify left))
     (property "Intersheetrefs" "${INTERSHEET_REFS}" (at 632.46 365.5152 90)
@@
   )
   (symbol (lib_id "Quantum Computing:LO_R&S") (at 654.685 392.43 180) (unit 1)
-    (in_bom yes) (on_board no) (dnp no) (fields_autoplaced)
-    (property "Reference" "LO9" (at 648.97 393.0395 0)
-      (effects (font (size 1.27 1.27)) (justify left))
+    (in_bom yes) (on_board no) (dnp no)
+    (property "Reference" "LO9" (at 643.509 391.16 0)
+      (effects (font (size 1.27 1.27)) (justify right))
     )
-    (property "Value" "LO_R&S" (at 648.97 390.4995 0)
-      (effects (font (size 1.27 1.27)) (justify left))
+    (property "Value" "LO_R&S" (at 641.096 394.589 0)
+      (effects (font (size 1.27 1.27)) (justify right))
     )
     (property "Footprint" "" (at 654.685 392.43 0)
@@
         )
         (path "/9924af8b-9fcb-4325-a1dc-18dd2c4184d7/a7096aa3-4c13-4b44-b9e6-37770984b4aa"
-          (reference "LO21") (unit 1)
+          (reference "LO16") (unit 1)
         )
       )
@@
       (effects (font (size 1.27 1.27)) (justify left top))
     )
-    (pin "QM_1_IN" input (at 732.79 417.195 180)
+    (pin "QM_OPX1_OPX2_INPUT" input (at 732.79 417.195 180)
       (effects (font (size 1.27 1.27)) (justify left))
     )
-    (pin "QM_1_I9_Q10_OUT" input (at 732.79 414.655 180)
+    (pin "QM_OPX1_OPX2_OUTPUT" input (at 732.79 414.655 180)
       (effects (font (size 1.27 1.27)) (justify left))
     )
@@
       (effects (font (size 1.27 1.27)) (justify left))
     )
-    (pin "QM_2_I9_Q10_OUT" input (at 784.86 419.735 0)
-      (effects (font (size 1.27 1.27)) (justify right))
-    )
-    (pin "QM_2_IN" input (at 784.86 422.275 0)
+    (pin "QM_2_IN" input (at 784.86 422.021 0)
       (effects (font (size 1.27 1.27)) (justify right))
     )

Commit message: removed lines for line C in qw25q
Connections:
- net at EF43.: now also LPF34.; no longer L:96.
- net at EF52.: now also LPF43.; no longer L:104.
- net at EF29.: now also L:5.; no longer LPF20.
- net at EF69.: now also L:153.; no longer LPF60.
- net at Coupler1.: now also L:3.; no longer L:4. (x2)
- net at L:3.: now also TWPA1.; no longer Coupler1.
- net at EF39.: now also LPF30.; no longer L:92.
- net at L:4.: now also Coupler1.; no longer TJI2. (x2)
- net at EF71.: now also LPF62.; no longer L:170.
- net at EF50.: now also L:102.; no longer LPF41.
- net at EF46.: now also L:98.; no longer LPF37.
- net at EF54.: now also L:106.; no longer LPF45.
- net at TJI2.: now also L:4.; no longer L:5.
- net at TWPA1.: now also L:3.; no longer L:2. (x2)
- net at L:3.: now also Coupler1.; no longer TWPA1. (x2)
- net at EF37.: now also L:27.; no longer LPF28.
- net at L:1.: now also TJI1.
- net at TJI1.: now also L:2.; no longer L:1.
- net at L:2.: now also TJI1.; no longer TWPA1. (x2)
- net at TJI1.: now also L:1.; no longer L:2. (x2)
- net at EF70.: now also L:168.; no longer LPF61.
- net at EF33.: now also LPF24.; no longer L:9.
- net at EF31.: now also LPF22.; no longer L:7.
- net at EF64.: now also LPF55.; no longer L:116.
- net at EF27.: now also L:3.; no longer LPF18.
- net at EF62.: now also L:114.; no longer LPF53.
- net at EF68.: now also L:120.; no longer LPF59.
- net at EF66.: now also LPF57.; no longer L:118.
- net at EF41.: now also LPF32.; no longer L:94.
- net at L:4.: now also TJI2.; no longer Coupler1.
- net at EF72.: now also L:174.; no longer LPF63.
- net at L:2.: now also TWPA1.; no longer TJI1.
- net at EF56.: now also L:108.; no longer LPF47.
- net at TJI2.: now also L:5.; no longer L:4.
- net at EF35.: now also L:25.; no longer LPF26.
- net at EF48.: now also L:100.; no longer LPF39.
- net at EF60.: now also LPF51.; no longer L:112.
- net at EF58.: now also LPF49.; no longer L:110.
- new net: EF43., L:96.
- new net: EF52., L:104.
- new net: EF29., LPF20.
- new net: ATT347., ATT348.
- new net: EF69., LPF60.
- new net: Coupler1., L:4. (x2)
- new net: EF39., L:92.
- new net: EF44., LPF35.
- new net: L:4., TJI2.
- new net: EF55., LPF46.
- new net: EF71., L:170.
- new net: EF38., LPF29.
- new net: EF50., LPF41.
- new net: EF46., LPF37.
- new net: EF47., LPF38.
- new net: ATT351., ATT352.
- new net: EF54., LPF45.
- new net: L:5., TJI2.
- new net: L:2., TWPA1. (x3)
- new net: EF37., LPF28.
- new net: EF51., LPF42.
- new net: EF70., LPF61.
- new net: ATT349., ATT350.
- new net: ATT345., ATT346.
- new net: EF65., LPF56.
- new net: EF33., L:9.
- new net: L:6., LX-X2. (x3)
- new net: EF31., L:7.
- new net: EF30., LPF21.
- new net: EF64., L:116.
- new net: EF57., LPF48.
- new net: EF27., LPF18.
- new net: EF49., LPF40.
- new net: EF61., LPF52.
- new net: EF62., LPF53.
- new net: EF68., LPF59.
- new net: EF66., L:118.
- new net: EF41., L:94.
- new net: EF72., LPF63.
- new net: L:2., TJI1.
- new net: EF40., LPF31.
- new net: EF28., LPF19.
- new net: EF56., LPF47.
- new net: EF67., LPF58.
- new net: EF35., LPF26.
- new net: EF63., LPF54.
- new net: EF36., LPF27.
- new net: EF45., LPF36.
- new net: EF53., LPF44.
- new net: EF48., LPF39.
- new net: EF60., L:112.
- new net: EF32., LPF23.
- new net: EF58., L:110.
- new net: EF42., LPF33.
- new net: EF34., LPF25.
- new net: EF59., LPF50.
- no-connect marks 6 -> 8
Changed lines of the file:
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@@
   (no_connect (at 730.885 431.8))
   (no_connect (at 730.885 444.5))
+  (no_connect (at 787.4 447.04))
+  (no_connect (at 729.615 463.55))
   (no_connect (at 730.885 441.96))
   (no_connect (at 786.765 435.61))
@@
     )
   )
-  (global_label "L1-17" (shape input) (at 729.615 463.55 180) (fields_autoplaced)
-    (effects (font (size 0.64 0.64)) (justify right))
-    (property "Intersheetrefs" "${INTERSHEET_REFS}" (at 725.0117 463.55 0)
-      (effects (font (size 1.27 1.27)) (justify right) hide)
-    )
-  )
   (global_label "L1-21" (shape input) (at 787.4 469.9 0) (fields_autoplaced)
     (effects (font (size 0.64 0.64)) (justify left))
@@
     )
   )
-  (global_label "L4-24" (shape input) (at 787.4 447.04 0) (fields_autoplaced)
-    (effects (font (size 0.64 0.64)) (justify left))
-    (property "Intersheetrefs" "${INTERSHEET_REFS}" (at 792.0033 447.04 0)
-      (effects (font (size 1.27 1.27)) (justify left) hide)
-    )
-  )
