File: XLD/Q2_2023/qblox_192_168_0_20.kicad_sch (KiCad schematic)
At the start: 10 parts

Commit message: correct L2-12 LNA gnd, it was fixed. Changed the IQM5q drive line LP to the correct cut frequency.
Connections:
- net at QCM6. (o4): now also IP2. (9)
- net at IP2. (9): now also QRM_RF3. (o1); no longer QCM6. (o4)
- net at QCM_RF4. (o2): now also SC3.; no longer SC4.
- net at QCM5. (o4): now also IP2. (9)
- net at QRM1. (o4): now also IP2. (9)
- new net: QRM_RF4. (o1), SC4.
- new net: QCM_RF4. (o2), SC4.
- new net: IP2. (9), QRM_RF4. (o1)
- new net: IP2. (9), QCM_RF4. (o2)
- new net: IP2. (9), QCM4. (Trig)
- new net: QRM_RF3. (o1), SC3.

Commit message: update tii1qb11
Connections:
- net at QCM6. (o4): now also IP2. (9)
- net at IP2. (9): now also QRM_RF3. (o1); no longer QCM6. (o4)
- net at QCM_RF4. (o2): now also SC3.; no longer SC4.
- net at QCM5. (o4): now also IP2. (9)
- net at QRM1. (o4): now also IP2. (9)
- new net: QRM_RF4. (o1), SC4.
- new net: QCM_RF4. (o2), SC4.
- new net: IP2. (9), QRM_RF4. (o1)
- new net: IP2. (9), QCM_RF4. (o2)
- new net: IP2. (9), QCM4. (Trig)
- new net: QRM_RF3. (o1), SC3.
