File: XLD/Q2_2023/qblox_192_168_0_20.kicad_sch (KiCad schematic)
At the start: 10 parts

Commit message: added changes of filter thermalization for flux lines qw25q
Connections:
- net at QCM6. (o4): now also IP2. (9)
- net at IP2. (9): now also QRM_RF3. (o1); no longer QCM6. (o4)
- net at QCM5. (o4): now also IP2. (9)
- net at QRM1. (o4): now also IP2. (9)
- new net: IP2. (9), QRM_RF4. (o1)
- new net: IP2. (9), QCM_RF4. (o2)
- new net: IP2. (9), QCM4. (Trig)

Commit message: added labels to lo3 splitter exits
Connections:
- net at QCM6. (o4): now also IP2. (9)
- net at IP2. (9): now also QRM_RF3. (o1); no longer QCM6. (o4)
- net at QCM5. (o4): now also IP2. (9)
- net at QRM1. (o4): now also IP2. (9)
- new net: IP2. (9), QRM_RF4. (o1)
- new net: IP2. (9), QCM_RF4. (o2)
- new net: IP2. (9), QCM4. (Trig)

Commit message: Updated the labeling for the cables from the splitters to the controller for the local oscillators 3 and 4
Connections:
- net at QCM6. (o4): now also IP2. (9)
- net at IP2. (9): now also QRM_RF3. (o1); no longer QCM6. (o4)
- net at QCM5. (o4): now also IP2. (9)
- net at QRM1. (o4): now also IP2. (9)
- new net: IP2. (9), QRM_RF4. (o1)
- new net: IP2. (9), QCM_RF4. (o2)
- new net: IP2. (9), QCM4. (Trig)

Commit message: corrected the names ans the output lines of the opxs
Connections:
- net at QCM6. (o4): now also IP2. (9)
- net at IP2. (9): now also QRM_RF3. (o1); no longer QCM6. (o4)
- net at QCM5. (o4): now also IP2. (9)
- net at QRM1. (o4): now also IP2. (9)
- new net: IP2. (9), QRM_RF4. (o1)
- new net: IP2. (9), QCM_RF4. (o2)
- new net: IP2. (9), QCM4. (Trig)

Commit message: add lo oscillators to line b con1 con2 con3
Connections:
- net at QCM6. (o4): now also IP2. (9)
- net at IP2. (9): now also QRM_RF3. (o1); no longer QCM6. (o4)
- net at QCM5. (o4): now also IP2. (9)
- net at QRM1. (o4): now also IP2. (9)
- new net: IP2. (9), QRM_RF4. (o1)
- new net: IP2. (9), QCM_RF4. (o2)
- new net: IP2. (9), QCM4. (Trig)

Commit message: partial re-labeling
Connections:
- net at QCM6. (o4): now also IP2. (9)
- net at IP2. (9): now also QRM_RF3. (o1); no longer QCM6. (o4)
- net at QCM5. (o4): now also IP2. (9)
- net at QRM1. (o4): now also IP2. (9)
- new net: IP2. (9), QRM_RF4. (o1)
- new net: IP2. (9), QCM_RF4. (o2)
- new net: IP2. (9), QCM4. (Trig)

Commit message: updating labels
Connections:
- net at QCM6. (o4): now also IP2. (9)
- net at IP2. (9): now also QRM_RF3. (o1); no longer QCM6. (o4)
- net at QCM5. (o4): now also IP2. (9)
- net at QRM1. (o4): now also IP2. (9)
- new net: IP2. (9), QRM_RF4. (o1)
- new net: IP2. (9), QCM_RF4. (o2)
- new net: IP2. (9), QCM4. (Trig)

Commit message: updatede de line B 5 qubits
Connections:
- net at QCM6. (o4): now also IP2. (9)
- net at IP2. (9): now also QRM_RF3. (o1); no longer QCM6. (o4)
- net at QCM5. (o4): now also IP2. (9)
- net at QRM1. (o4): now also IP2. (9)
- new net: IP2. (9), QRM_RF4. (o1)
- new net: IP2. (9), QCM_RF4. (o2)
- new net: IP2. (9), QCM4. (Trig)
