File: XLD/Q2_2023/qblox_192_168_0_6.kicad_sch (KiCad schematic)
At the start: 11 parts

Commit message: correct L2-12 LNA gnd, it was fixed. Changed the IQM5q drive line LP to the correct cut frequency.
Connections:
- net at IP1. (9): now also QCM_RF2. (o2); no longer QCM3. (o4)
- new net: IP1. (9), QCM3. (o4)
- new net: IP1. (9), QCM2. (o4)
- new net: IP1. (9), QCM_RF1. (o2)
- new net: IP1. (9), QCM_RF3. (o2)
- new net: IP1. (9), QRM_RF2. (o1)
- new net: IP1. (9), QRM_RF1. (o1)
- new net: IP1. (9), QCM1. (Trig)

Commit message: update tii1qb11
Connections:
- net at IP1. (9): now also QCM_RF2. (o2); no longer QCM3. (o4)
- new net: IP1. (9), QCM3. (o4)
- new net: IP1. (9), QCM2. (o4)
- new net: IP1. (9), QCM_RF1. (o2)
- new net: IP1. (9), QCM_RF3. (o2)
- new net: IP1. (9), QRM_RF2. (o1)
- new net: IP1. (9), QRM_RF1. (o1)
- new net: IP1. (9), QCM1. (Trig)
