File: XLD/Q2_2023/qblox_192_168_0_6.kicad_sch (KiCad schematic)
At the start: 11 parts

Commit message: mend
Parts:
- renumbered IP601 to IP1, SC601 to SC1, SC602 to SC2
Connections:
- net at IP1. (9): now also QCM_RF2. (o2); no longer QCM3. (o4)
- new net: IP1. (9), QCM3. (o4)
- new net: IP1. (9), QCM2. (o4)
- new net: IP1. (9), QCM_RF1. (o2)
- new net: IP1. (9), QCM_RF3. (o2)
- new net: IP1. (9), QRM_RF2. (o1)
- new net: IP1. (9), QRM_RF1. (o1)
- new net: IP1. (9), QCM1. (Trig)
Changed lines of the file:
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@@
   (symbol (lib_id "Quantum Computing:QBlox_QCM") (at 201.93 137.795 0) (unit 1)
     (in_bom yes) (on_board no) (dnp no) (fields_autoplaced)
-    (property "Reference" "QCM?" (at 200.025 139.827 0)
+    (property "Reference" "QCM3" (at 200.025 139.827 0)
       (effects (font (size 1.27 1.27)) (justify left))
     )
@@
   (symbol (lib_id "Quantum Computing:QBlox_QCM") (at 142.875 137.795 0) (unit 1)
     (in_bom yes) (on_board no) (dnp no) (fields_autoplaced)
-    (property "Reference" "QCM?" (at 140.97 139.827 0)
+    (property "Reference" "QCM2" (at 140.97 139.827 0)
       (effects (font (size 1.27 1.27)) (justify left))
     )
@@
   (symbol (lib_id "Quantum Computing:QBlox_QCM_RF") (at 162.56 137.795 0) (unit 1)
     (in_bom yes) (on_board no) (dnp no) (fields_autoplaced)
-    (property "Reference" "QCM_RF?" (at 160.655 139.827 0)
+    (property "Reference" "QCM_RF1" (at 160.655 139.827 0)
       (effects (font (size 1.27 1.27)) (justify left))
     )
@@
   (symbol (lib_id "Quantum Computing:QBlox_QCM_RF") (at 260.985 137.795 0) (unit 1)
     (in_bom yes) (on_board no) (dnp no) (fields_autoplaced)
-    (property "Reference" "QCM_RF?" (at 259.08 139.827 0)
+    (property "Reference" "QCM_RF3" (at 259.08 139.827 0)
       (effects (font (size 1.27 1.27)) (justify left))
     )
@@
   (symbol (lib_id "Quantum Computing:Splitter_Combiner") (at 304.165 166.37 180) (unit 1)
     (in_bom yes) (on_board no) (dnp no) (fields_autoplaced)
-    (property "Reference" "SC601" (at 304.165 158.75 0)
+    (property "Reference" "SC1" (at 304.165 158.75 0)
       (effects (font (size 1.27 1.27)))
     )
@@
   (symbol (lib_id "Quantum Computing:Qblox_Cluster") (at 300.355 116.84 0) (unit 1)
     (in_bom yes) (on_board yes) (dnp no) (fields_autoplaced)
-    (property "Reference" "IP601" (at 300.355 109.855 0)
+    (property "Reference" "IP1" (at 300.355 109.855 0)
       (effects (font (size 1.27 1.27)))
     )
@@
   (symbol (lib_id "Quantum Computing:QBlox_QRM_RF") (at 339.725 137.795 0) (unit 1)
     (in_bom yes) (on_board no) (dnp no) (fields_autoplaced)
-    (property "Reference" "QRM_RF?" (at 337.82 139.827 0)
+    (property "Reference" "QRM_RF2" (at 337.82 139.827 0)
       (effects (font (size 1.27 1.27)) (justify left))
     )
@@
   (symbol (lib_id "Quantum Computing:QBlox_QRM_RF") (at 300.355 137.795 0) (unit 1)
     (in_bom yes) (on_board no) (dnp no) (fields_autoplaced)
-    (property "Reference" "QRM_RF?" (at 298.45 139.827 0)
+    (property "Reference" "QRM_RF1" (at 298.45 139.827 0)
       (effects (font (size 1.27 1.27)) (justify left))
     )
@@
   (symbol (lib_id "Quantum Computing:Splitter_Combiner") (at 334.645 166.37 180) (unit 1)
     (in_bom yes) (on_board no) (dnp no) (fields_autoplaced)
-    (property "Reference" "SC602" (at 334.645 158.75 0)
+    (property "Reference" "SC2" (at 334.645 158.75 0)
       (effects (font (size 1.27 1.27)))
     )
@@
   (symbol (lib_id "Quantum Computing:QBlox_CTRL") (at 102.235 137.795 0) (unit 1)
     (in_bom yes) (on_board no) (dnp no) (fields_autoplaced)
-    (property "Reference" "QCM?" (at 100.33 139.827 0)
+    (property "Reference" "QCM1" (at 100.33 139.827 0)
       (effects (font (size 1.27 1.27)) (justify left))
     )
@@
   (symbol (lib_id "Quantum Computing:QBlox_QCM_RF") (at 182.245 137.795 0) (unit 1)
     (in_bom yes) (on_board no) (dnp no) (fields_autoplaced)
-    (property "Reference" "QCM_RF?" (at 180.34 139.827 0)
-      (effects (font (size 1.27 1.27)) (justify left))
-    )
+    (property "Reference" "QCM_RF2" (at 180.34 139.827 0)
+      (effects (font (size 1.27 1.27)) (justify left))
+    )

Commit message: more updates
Connections:
- net at IP1. (9): now also QCM_RF2. (o2); no longer QCM3. (o4)
- new net: IP1. (9), QCM3. (o4)
- new net: IP1. (9), QCM2. (o4)
- new net: IP1. (9), QCM_RF1. (o2)
- new net: IP1. (9), QCM_RF3. (o2)
- new net: IP1. (9), QRM_RF2. (o1)
- new net: IP1. (9), QRM_RF1. (o1)
- new net: IP1. (9), QCM1. (Trig)

Commit message: Improvements to library components, title, date
Connections:
- net at IP1. (9): now also QCM_RF2. (o2); no longer QCM3. (o4)
- new net: IP1. (9), QCM3. (o4)
- new net: IP1. (9), QCM2. (o4)
- new net: IP1. (9), QCM_RF1. (o2)
- new net: IP1. (9), QCM_RF3. (o2)
- new net: IP1. (9), QRM_RF2. (o1)
- new net: IP1. (9), QRM_RF1. (o1)
- new net: IP1. (9), QCM1. (Trig)
Other:
- company: (none) -> Technology Innovation Institute
- title: (none) -> XLD Setup Q2 2023
Changed lines of the file:
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@@
 (kicad_sch (version 20230121) (generator eeschema)
   (paper "A2")
+  (title_block
+    (title "XLD Setup Q2 2023")
+    (date "2023-06-14")
+    (company "Technology Innovation Institute")
+  )
   (no_connect (at 98.425 134.62))
   (no_connect (at 98.425 133.35))

Commit message: Correction in line numbers of QW 25Q
We have checked the cables of QW 25Q by connecting the IN and OUT lines to VNA and found that there is are corrections required in the line numbers mentioned in the drawing. Below are the correction made:

QW P14 - In line L3-30 , Out line L2-1
QW P29 - In line L3-26 , Out line L2-2
QW P44 - In line L3-27 , Out line L2-3
QW P59 - In line L3-18 , Out line L2-4

The Coupler pump line L3-21 replaced with L3-29
Connections:
- net at IP1. (9): now also QCM_RF2. (o2); no longer QCM3. (o4)
- new net: IP1. (9), QCM3. (o4)
- new net: IP1. (9), QCM2. (o4)
- new net: IP1. (9), QCM_RF1. (o2)
- new net: IP1. (9), QCM_RF3. (o2)
- new net: IP1. (9), QRM_RF2. (o1)
- new net: IP1. (9), QRM_RF1. (o1)
- new net: IP1. (9), QCM1. (Trig)

Commit message: fix qw5q twpa pump line ip address
Connections:
- net at IP1. (9): now also QCM_RF2. (o2); no longer QCM3. (o4)
- new net: IP1. (9), QCM3. (o4)
- new net: IP1. (9), QCM2. (o4)
- new net: IP1. (9), QCM_RF1. (o2)
- new net: IP1. (9), QCM_RF3. (o2)
- new net: IP1. (9), QRM_RF2. (o1)
- new net: IP1. (9), QRM_RF1. (o1)
- new net: IP1. (9), QCM1. (Trig)

Commit message: various fixes
swap L3-20 with L2-17 in qblox
change ip of Lo18 to 192.168.0.208 (tii1q_b4 twpa pump) and type to ERA
rename LO_ERA_pp to LO_ERA
Connections:
- net at IP1. (9): now also QCM_RF2. (o2); no longer QCM3. (o4)
- new net: IP1. (9), QCM3. (o4)
- new net: IP1. (9), QCM2. (o4)
- new net: IP1. (9), QCM_RF1. (o2)
- new net: IP1. (9), QCM_RF3. (o2)
- new net: IP1. (9), QRM_RF2. (o1)
- new net: IP1. (9), QRM_RF1. (o1)
- new net: IP1. (9), QCM1. (Trig)

Commit message: corrected the output lines for the readout for QW25q
Connections:
- net at IP1. (9): now also QCM_RF2. (o2); no longer QCM3. (o4)
- new net: IP1. (9), QCM3. (o4)
- new net: IP1. (9), QCM2. (o4)
- new net: IP1. (9), QCM_RF1. (o2)
- new net: IP1. (9), QCM_RF3. (o2)
- new net: IP1. (9), QRM_RF2. (o1)
- new net: IP1. (9), QRM_RF1. (o1)
- new net: IP1. (9), QCM1. (Trig)

Commit message: added changes of filter thermalization for flux lines qw25q
Connections:
- net at IP1. (9): now also QCM_RF2. (o2); no longer QCM3. (o4)
- new net: IP1. (9), QCM3. (o4)
- new net: IP1. (9), QCM2. (o4)
- new net: IP1. (9), QCM_RF1. (o2)
- new net: IP1. (9), QCM_RF3. (o2)
- new net: IP1. (9), QRM_RF2. (o1)
- new net: IP1. (9), QRM_RF1. (o1)
- new net: IP1. (9), QCM1. (Trig)
