File: XLD/Q2_2023/qblox_192_168_0_6.kicad_sch (KiCad schematic)
At the start: 11 parts

Commit message: added labels to lo3 splitter exits
Connections:
- net at IP1. (9): now also QCM_RF2. (o2); no longer QCM3. (o4)
- new net: IP1. (9), QCM3. (o4)
- new net: IP1. (9), QCM2. (o4)
- new net: IP1. (9), QCM_RF1. (o2)
- new net: IP1. (9), QCM_RF3. (o2)
- new net: IP1. (9), QRM_RF2. (o1)
- new net: IP1. (9), QRM_RF1. (o1)
- new net: IP1. (9), QCM1. (Trig)

Commit message: Updated the labeling for the cables from the splitters to the controller for the local oscillators 3 and 4
Connections:
- net at IP1. (9): now also QCM_RF2. (o2); no longer QCM3. (o4)
- new net: IP1. (9), QCM3. (o4)
- new net: IP1. (9), QCM2. (o4)
- new net: IP1. (9), QCM_RF1. (o2)
- new net: IP1. (9), QCM_RF3. (o2)
- new net: IP1. (9), QRM_RF2. (o1)
- new net: IP1. (9), QRM_RF1. (o1)
- new net: IP1. (9), QCM1. (Trig)

Commit message: corrected the names ans the output lines of the opxs
Connections:
- net at IP1. (9): now also QCM_RF2. (o2); no longer QCM3. (o4)
- new net: IP1. (9), QCM3. (o4)
- new net: IP1. (9), QCM2. (o4)
- new net: IP1. (9), QCM_RF1. (o2)
- new net: IP1. (9), QCM_RF3. (o2)
- new net: IP1. (9), QRM_RF2. (o1)
- new net: IP1. (9), QRM_RF1. (o1)
- new net: IP1. (9), QCM1. (Trig)

Commit message: add lo oscillators to line b con1 con2 con3
Connections:
- net at IP1. (9): now also QCM_RF2. (o2); no longer QCM3. (o4)
- new net: IP1. (9), QCM3. (o4)
- new net: IP1. (9), QCM2. (o4)
- new net: IP1. (9), QCM_RF1. (o2)
- new net: IP1. (9), QCM_RF3. (o2)
- new net: IP1. (9), QRM_RF2. (o1)
- new net: IP1. (9), QRM_RF1. (o1)
- new net: IP1. (9), QCM1. (Trig)

Commit message: partial re-labeling
Connections:
- net at IP1. (9): now also QCM_RF2. (o2); no longer QCM3. (o4)
- new net: IP1. (9), QCM3. (o4)
- new net: IP1. (9), QCM2. (o4)
- new net: IP1. (9), QCM_RF1. (o2)
- new net: IP1. (9), QCM_RF3. (o2)
- new net: IP1. (9), QRM_RF2. (o1)
- new net: IP1. (9), QRM_RF1. (o1)
- new net: IP1. (9), QCM1. (Trig)

Commit message: updating labels
Connections:
- net at IP1. (9): now also QCM_RF2. (o2); no longer QCM3. (o4)
- new net: IP1. (9), QCM3. (o4)
- new net: IP1. (9), QCM2. (o4)
- new net: IP1. (9), QCM_RF1. (o2)
- new net: IP1. (9), QCM_RF3. (o2)
- new net: IP1. (9), QRM_RF2. (o1)
- new net: IP1. (9), QRM_RF1. (o1)
- new net: IP1. (9), QCM1. (Trig)

Commit message: updatede de line B 5 qubits
Connections:
- net at IP1. (9): now also QCM_RF2. (o2); no longer QCM3. (o4)
- new net: IP1. (9), QCM3. (o4)
- new net: IP1. (9), QCM2. (o4)
- new net: IP1. (9), QCM_RF1. (o2)
- new net: IP1. (9), QCM_RF3. (o2)
- new net: IP1. (9), QRM_RF2. (o1)
- new net: IP1. (9), QRM_RF1. (o1)
- new net: IP1. (9), QCM1. (Trig)

Commit message: removed lines for line C in qw25q
Connections:
- net at IP1. (9): now also QCM_RF2. (o2); no longer QCM3. (o4)
- new net: IP1. (9), QCM3. (o4)
- new net: IP1. (9), QCM2. (o4)
- new net: IP1. (9), QCM_RF1. (o2)
- new net: IP1. (9), QCM_RF3. (o2)
- new net: IP1. (9), QRM_RF2. (o1)
- new net: IP1. (9), QRM_RF1. (o1)
- new net: IP1. (9), QCM1. (Trig)
