File: XLD/Q2_2023/1qs.kicad_sch (KiCad schematic)
At the start: 69 parts

Commit message: correct L2-12 LNA gnd, it was fixed. Changed the IQM5q drive line LP to the correct cut frequency.
Connections:
- net at TWPA4.: now also L:132.; no longer L:133.
- net at L:177.: now also EF74.
- net at EF74.: now also LPF65.; no longer L:177.
- net at TJI14.: now also L:134.; no longer L:135.
- net at L:134.: now also Coupler7.; no longer TJI14.
- net at EF73.: now also L:175.; no longer LPF64.
- net at L:175.: no longer EF73.
- net at L:179.: now also EF75.
- net at EF75.: now also LPF66.; no longer L:179.
- new net: L:133., TWPA4.
- new net: L:140., TJI16.
- new net: L:135., TJI14.
- new net: L:194., TJI13.
- new net: L:6., LX-X2.
- new net: EF73., LPF64.
- new net: L:137., TJI15.

Commit message: update tii1qb11
Connections:
- net at TWPA4.: now also L:132.; no longer L:133.
- net at L:177.: now also EF74.
- net at EF74.: now also LPF65.; no longer L:177.
- net at TJI14.: now also L:134.; no longer L:135.
- net at L:134.: now also Coupler7.; no longer TJI14.
- net at EF73.: now also L:175.; no longer LPF64.
- net at L:175.: no longer EF73.
- net at L:179.: now also EF75.
- net at EF75.: now also LPF66.; no longer L:179.
- new net: L:133., TWPA4.
- new net: L:140., TJI16.
- new net: L:135., TJI14.
- new net: L:194., TJI13.
- new net: L:6., LX-X2.
- new net: EF73., LPF64.
- new net: L:137., TJI15.
Other:
- note added: "D011_225CB"
- note removed: "D011_200nm"
Changed lines of the file:
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@@
     (effects (font (size 1.27 1.27)) (justify left bottom))
   )
-  (text "D011_200nm\n" (at 35.56 388.62 0)
+  (text "D011_225CB\n" (at 35.56 388.62 0)
     (effects (font (size 1.27 1.27)) (justify left bottom))
   )

Commit message: fix qw5q twpa pump line ip address
Connections:
- net at TWPA4.: now also L:132.; no longer L:133.
- net at L:177.: now also EF74.
- net at EF74.: now also LPF65.; no longer L:177.
- net at TJI14.: now also L:134.; no longer L:135.
- net at L:134.: now also Coupler7.; no longer TJI14.
- net at EF73.: now also L:175.; no longer LPF64.
- net at L:175.: no longer EF73.
- net at L:179.: now also EF75.
- net at EF75.: now also LPF66.; no longer L:179.
- new net: L:133., TWPA4.
- new net: L:140., TJI16.
- new net: L:135., TJI14.
- new net: L:194., TJI13.
- new net: L:6., LX-X2.
- new net: EF73., LPF64.
- new net: L:137., TJI15.

Commit message: ip for LO18
Connections:
- net at TWPA4.: now also L:132.; no longer L:133.
- net at L:177.: now also EF74.
- net at EF74.: now also LPF65.; no longer L:177.
- net at TJI14.: now also L:134.; no longer L:135.
- net at L:134.: now also Coupler7.; no longer TJI14.
- net at EF73.: now also L:175.; no longer LPF64.
- net at L:175.: no longer EF73.
- net at L:179.: now also EF75.
- net at EF75.: now also LPF66.; no longer L:179.
- new net: L:133., TWPA4.
- new net: L:140., TJI16.
- new net: L:135., TJI14.
- new net: L:194., TJI13.
- new net: L:6., LX-X2.
- new net: EF73., LPF64.
- new net: L:137., TJI15.
Other:
- note added: "192.168.0.208"
- note removed: "192.168.0.?"
Changed lines of the file:
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@@
     (stroke (width 0) (type default))
   )
-  (text "192.168.0.?\n" (at 172.72 346.71 0)
+  (text "192.168.0.208\n" (at 172.72 346.71 0)
     (effects (font (size 1.27 1.27)) (justify left bottom))
   )
