File: XLD/Q2_2023/1qs.kicad_sch (KiCad schematic)
At the start: 69 parts

Commit message: add lo oscillators to line b con1 con2 con3
Connections:
- net at TWPA4.: now also L:132.; no longer L:133.
- net at L:177.: now also EF74.
- net at EF74.: now also LPF65.; no longer L:177.
- net at TJI14.: now also L:134.; no longer L:135.
- net at L:134.: now also Coupler7.; no longer TJI14.
- net at EF73.: now also L:175.; no longer LPF64.
- net at L:175.: no longer EF73.
- net at L:179.: now also EF75.
- net at EF75.: now also LPF66.; no longer L:179.
- new net: L:133., TWPA4.
- new net: L:140., TJI16.
- new net: L:135., TJI14.
- new net: L:194., TJI13.
- new net: L:6., LX-X2.
- new net: EF73., LPF64.
- new net: L:137., TJI15.

Commit message: partial re-labeling
Connections:
- net at TWPA4.: now also L:132.; no longer L:133.
- net at L:177.: now also EF74.
- net at EF74.: now also LPF65.; no longer L:177.
- net at TJI14.: now also L:134.; no longer L:135.
- net at L:134.: now also Coupler7.; no longer TJI14.
- net at EF73.: now also L:175.; no longer LPF64.
- net at L:175.: no longer EF73.
- net at L:179.: now also EF75.
- net at EF75.: now also LPF66.; no longer L:179.
- new net: L:133., TWPA4.
- new net: L:140., TJI16.
- new net: L:135., TJI14.
- new net: L:194., TJI13.
- new net: L:6., LX-X2.
- new net: EF73., LPF64.
- new net: L:137., TJI15.

Commit message: updating labels
Connections:
- net at TWPA4.: now also L:132.; no longer L:133.
- net at L:177.: now also EF74.
- net at EF74.: now also LPF65.; no longer L:177.
- net at TJI14.: now also L:134.; no longer L:135.
- net at L:134.: now also Coupler7.; no longer TJI14.
- net at EF73.: now also L:175.; no longer LPF64.
- net at L:175.: no longer EF73.
- net at L:179.: now also EF75.
- net at EF75.: now also LPF66.; no longer L:179.
- new net: L:133., TWPA4.
- new net: L:140., TJI16.
- new net: L:135., TJI14.
- new net: L:194., TJI13.
- new net: L:6., LX-X2.
- new net: EF73., LPF64.
- new net: L:137., TJI15.

Commit message: updatede de line B 5 qubits
Connections:
- net at TWPA4.: now also L:132.; no longer L:133.
- net at L:177.: now also EF74.
- net at EF74.: now also LPF65.; no longer L:177.
- net at TJI14.: now also L:134.; no longer L:135.
- net at L:134.: now also Coupler7.; no longer TJI14.
- net at EF73.: now also L:175.; no longer LPF64.
- net at L:175.: no longer EF73.
- net at L:179.: now also EF75.
- net at EF75.: now also LPF66.; no longer L:179.
- new net: L:133., TWPA4.
- new net: L:140., TJI16.
- new net: L:135., TJI14.
- new net: L:194., TJI13.
- new net: L:6., LX-X2.
- new net: EF73., LPF64.
- new net: L:137., TJI15.

Commit message: removed lines for line C in qw25q
Connections:
- net at TWPA4.: now also L:132.; no longer L:133.
- net at L:177.: now also EF74.
- net at EF74.: now also LPF65.; no longer L:177.
- net at TJI14.: now also L:134.; no longer L:135.
- net at L:134.: now also Coupler7.; no longer TJI14.
- net at EF73.: now also L:175.; no longer LPF64.
- net at L:175.: no longer EF73.
- net at L:179.: now also EF75.
- net at EF75.: now also LPF66.; no longer L:179.
- new net: L:133., TWPA4.
- new net: L:140., TJI16.
- new net: L:135., TJI14.
- new net: L:194., TJI13.
- new net: L:6., LX-X2.
- new net: EF73., LPF64.
- new net: L:137., TJI15.
