File: XLD/Q2_2023/iqm5q.kicad_sch (KiCad schematic)
At the start: 130 parts

Commit message: mend
Connections:
- new net: Eccosorb?., LPF?. (x6)
- new net: L:?., TJI?.
Other:
- added sheet ZI (ZI.kicad_sch)
Changed lines of the file:
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@@
+    )
+  )
+  (sheet (at 380.365 316.865) (size 73.66 39.37) (fields_autoplaced)
+    (stroke (width 0.1524) (type solid))
+    (fill (color 0 0 0 0.0000))
+    (property "Sheetname" "ZI" (at 380.365 316.1534 0)
+      (effects (font (size 1.27 1.27)) (justify left bottom))
+    )
+    (property "Sheetfile" "ZI.kicad_sch" (at 380.365 356.8196 0)
+      (effects (font (size 1.27 1.27)) (justify left top))
+    )
+    (instances
+      (project "Q2_2023"
+        (path "/9924af8b-9fcb-4325-a1dc-18dd2c4184d7/148e980e-9f48-4feb-8355-1cd74c17609e" (page "3"))
+      )
     )
   )

Commit message: more updates
Parts:
- removed TJI?: LNF-ISISC4_12A, symbol Quantum Computing:LNF-ISISC4_12A
- added ATT?: Attenuator 1-Cryo, symbol Quantum Computing:Attenuator 0-Cryo
- added ATT?: Attenuator 10-Cryo, symbol Quantum Computing:Attenuator 3-Cryo
- added ATT?: Attenuator 0-Cryo, symbol Quantum Computing:Attenuator 0-Cryo
- added ATT?: Attenuator 20-Cryo, symbol Quantum Computing:Attenuator 20-Cryo
- added ATT?: Attenuator 6-Cryo, symbol Quantum Computing:Attenuator 6-Cryo
- added Coupler?: QMC-CRYOCOUPLER-20, symbol Quantum Computing:QMC-CRYOCOUPLER-20
- added L:? (x3): SMA-SMA, symbol Quantum Computing:SMA-SMA
- added L:?: SMA-SMP, symbol Quantum Computing:SMA-SMP
- added L:?: COAX-6FT, symbol Quantum Computing:COAX-6FT
- added L:?: SMA-SMA_small, symbol Quantum Computing:SMA-SMA_small
- added LX-X?: NbTi-RF-line, symbol Quantum Computing:NbTi-RF-line
- added TJI? (x2): LNF-ISISC4_12A, symbol Quantum Computing:LNF-ISISC4_12A
- added TWPA?: SW_TWPA, symbol Quantum Computing:SW_TWPA
Connections:
- net L2-7: now also L:?.
- new net: Coupler?., L:?. (x2)
- new net: Eccosorb?., LPF?. (x6)
- new net: L:?., TJI?. (x4)
- new net: L:?., TWPA?. (x2)
- new net L3-28: ATT?., ATT?., ATT?., ATT?., ATT?., L:?., L:?., LX-X?.
- new net L3-xx: Coupler?.20dB, L:?.
Other:
- note added: "100mK"
- note added: "1K"
- note added: "20mK"
- note added: "300K"
- note added: "4K"
- note added: "50K"
- note added: "Brass 8inch"
- note added: "ISOLATOR-1"
- note added: "ISOLATOR-2"
- note added: "Short Brass"
- note added: "Steel one"
- note removed: "ISOLATOR-3"
- moved on the sheet: ATT?, Eccosorb?, HEMT?, L:?, LPF?, LX-X?

Commit message: update attenuators and pumplines
Parts:
- added LO9: LO_R&S, symbol Quantum Computing:LO_R&S
- gave numbers to parts that had none: 141
Connections:
- net L3-xx is gone; now on net L3-32: Coupler1.20dB, L:1.
- net at Coupler1.: now also L:3.; no longer L:4.
- net at L:3.: now also TWPA1.; no longer Coupler1.
- net at TJI2.: now also L:4.; no longer L:5.
- net at TJI1.: now also L:56.; no longer L:2.
- net L3-28 renamed L3-32
- net L3-32: now also LO9.
- new net: Coupler1., L:4.
- new net: Eccosorb30., LPF10.
- new net: L:5., TJI2.
- new net: L:2., TJI1.
- new net: Eccosorb29., LPF9.
- new net: Eccosorb1., LPF1.
- new net: Eccosorb28., LPF8.
- new net: Eccosorb27., LPF7.
- new net: Eccosorb26., LPF6.
Other:
- note added: "192.168.0.?"

Commit message: Improvements to library components, title, date
Parts:
- ATT4: symbol Quantum Computing:Attenuator 0-Cryo -> Quantum Computing:Attenuator 1-Cryo
- ATT8: symbol Quantum Computing:Attenuator 3-Cryo -> Quantum Computing:Attenuator 10-Cryo
- CBL14: renamed from L:1; value COAX-6FT -> Minicircuits-6FT; symbol Quantum Computing:COAX-6FT -> Quantum Computing:RF Cable Minicircuits-6FT
- CBL16: renamed from L:11; value COAX-6FT -> Minicircuits-6FT; symbol Quantum Computing:COAX-6FT -> Quantum Computing:RF Cable Minicircuits-6FT
- CBL17: renamed from L:12; value COAX-6FT -> Minicircuits-6FT; symbol Quantum Computing:COAX-6FT -> Quantum Computing:RF Cable Minicircuits-6FT
- CBL18: renamed from L:13; value COAX-6FT -> Minicircuits-6FT; symbol Quantum Computing:COAX-6FT -> Quantum Computing:RF Cable Minicircuits-6FT
- CBL19: renamed from L:14; value COAX-6FT -> Minicircuits-6FT; symbol Quantum Computing:COAX-6FT -> Quantum Computing:RF Cable Minicircuits-6FT
- CBL20: renamed from L:15; value COAX-6FT -> Minicircuits-6FT; symbol Quantum Computing:COAX-6FT -> Quantum Computing:RF Cable Minicircuits-6FT
- CBL21: renamed from L:16; value COAX-6FT -> Minicircuits-6FT; symbol Quantum Computing:COAX-6FT -> Quantum Computing:RF Cable Minicircuits-6FT
- CBL22: renamed from L:17; value COAX-6FT -> Minicircuits-6FT; symbol Quantum Computing:COAX-6FT -> Quantum Computing:RF Cable Minicircuits-6FT
- CBL23: renamed from L:18; value COAX-6FT -> Minicircuits-6FT; symbol Quantum Computing:COAX-6FT -> Quantum Computing:RF Cable Minicircuits-6FT
- CBL24: renamed from L:19; value COAX-6FT -> Minicircuits-6FT; symbol Quantum Computing:COAX-6FT -> Quantum Computing:RF Cable Minicircuits-6FT
- CBL25: renamed from L:20; value COAX-6FT -> Minicircuits-6FT; symbol Quantum Computing:COAX-6FT -> Quantum Computing:RF Cable Minicircuits-6FT
- CBL26: renamed from L:21; value COAX-6FT -> Minicircuits-6FT; symbol Quantum Computing:COAX-6FT -> Quantum Computing:RF Cable Minicircuits-6FT
- CBL27: renamed from L:22; value COAX-6FT -> Minicircuits-6FT; symbol Quantum Computing:COAX-6FT -> Quantum Computing:RF Cable Minicircuits-6FT
- CBL28: renamed from L:23; value COAX-6FT -> Minicircuits-6FT; symbol Quantum Computing:COAX-6FT -> Quantum Computing:RF Cable Minicircuits-6FT
- CBL29: renamed from L:24; value COAX-6FT -> Minicircuits-6FT; symbol Quantum Computing:COAX-6FT -> Quantum Computing:RF Cable Minicircuits-6FT
- Coupler1: symbol Quantum Computing:QMC-CRYOCOUPLER-20 -> Quantum Computing:Directional Coupler QMC-CRYOCOUPLER-20
- EF12: renamed from Eccosorb1; symbol Quantum Computing:IR-10GHz -> Quantum Computing:Filter Eccosorb IR-10GHz
- EF13: renamed from Eccosorb6; symbol Quantum Computing:IR-1GHz -> Quantum Computing:Filter Eccosorb IR-1GHz
- EF14: renamed from Eccosorb7; symbol Quantum Computing:IR-1GHz -> Quantum Computing:Filter Eccosorb IR-1GHz
- EF15: renamed from Eccosorb8; symbol Quantum Computing:IR-1GHz -> Quantum Computing:Filter Eccosorb IR-1GHz
- EF16: renamed from Eccosorb9; symbol Quantum Computing:IR-1GHz -> Quantum Computing:Filter Eccosorb IR-1GHz
- EF17: renamed from Eccosorb10; symbol Quantum Computing:IR-1GHz -> Quantum Computing:Filter Eccosorb IR-1GHz
- EF18: renamed from Eccosorb11; symbol Quantum Computing:IR-1GHz -> Quantum Computing:Filter Eccosorb IR-1GHz
- EF19: renamed from Eccosorb23; symbol Quantum Computing:IR-1GHz -> Quantum Computing:Filter Eccosorb IR-1GHz
- EF20: renamed from Eccosorb24; symbol Quantum Computing:IR-1GHz -> Quantum Computing:Filter Eccosorb IR-1GHz
- EF21: renamed from Eccosorb25; symbol Quantum Computing:IR-1GHz -> Quantum Computing:Filter Eccosorb IR-1GHz
- EF22: renamed from Eccosorb26; symbol Quantum Computing:IR-10GHz-FF -> Quantum Computing:Filter Eccosorb IR-10GHz-FF
- EF23: renamed from Eccosorb27; symbol Quantum Computing:IR-10GHz-FF -> Quantum Computing:Filter Eccosorb IR-10GHz-FF
- EF24: renamed from Eccosorb28; symbol Quantum Computing:IR-10GHz-FF -> Quantum Computing:Filter Eccosorb IR-10GHz-FF
- EF25: renamed from Eccosorb29; symbol Quantum Computing:IR-10GHz-FF -> Quantum Computing:Filter Eccosorb IR-10GHz-FF
- EF26: renamed from Eccosorb30; symbol Quantum Computing:IR-10GHz-FF -> Quantum Computing:Filter Eccosorb IR-10GHz-FF
- HEMT2: renamed from HEMT7; symbol Quantum Computing:LNF-LNC4_8C -> Quantum Computing:Amplifier HEMT LNF-LNC4_8C
- L:1, L:2, L:4, L:56: symbol Quantum Computing:SMA-SMA -> Quantum Computing:RF Cable SMA-SMA
- L:3: value SMA-SMA_small -> SMA-SMA short; symbol Quantum Computing:SMA-SMA_small -> Quantum Computing:RF Cable SMA-SMA_short
- L:5: symbol Quantum Computing:SMA-SMP -> Quantum Computing:RF Cable SMA-SMP
- L:6: value COAX-6FT -> Minicircuits-6FT; symbol Quantum Computing:COAX-6FT -> Quantum Computing:RF Cable Minicircuits-6FT
- LPF12: renamed from LPF1; symbol Quantum Computing:F-30-8000-R -> Quantum Computing:Filter Low-Pass F-30-8000-R
- LPF13: renamed from LPF6; symbol Quantum Computing:F-30-8000-R -> Quantum Computing:Filter Low-Pass F-30-8000-R
- LPF14: renamed from LPF7; symbol Quantum Computing:F-30-8000-R -> Quantum Computing:Filter Low-Pass F-30-8000-R
- LPF15: renamed from LPF8; symbol Quantum Computing:F-30-8000-R -> Quantum Computing:Filter Low-Pass F-30-8000-R
- LPF16: renamed from LPF9; symbol Quantum Computing:F-30-8000-R -> Quantum Computing:Filter Low-Pass F-30-8000-R
- LPF17: renamed from LPF10; symbol Quantum Computing:F-30-8000-R -> Quantum Computing:Filter Low-Pass F-30-8000-R
- LX-X2: value NbTi-RF-line -> NbTi; symbol Quantum Computing:NbTi-RF-line -> Quantum Computing:RF Line NbTi
- QPU?: value QPU_5q_flux_4couplers -> QPU IQM 5q; symbol Quantum Computing:QPU_5q_flux_4couplers -> Quantum Computing:QPU IQM 5q
- RFL14: renamed from LX-X1; value NbTi-RF-line -> NbTi; symbol Quantum Computing:NbTi-RF-line -> Quantum Computing:RF Line NbTi
- RFL16: renamed from LX-X6; value NbTi-RF-line -> NbTi; symbol Quantum Computing:NbTi-RF-line -> Quantum Computing:RF Line NbTi
- RFL17: renamed from LX-X7; value NbTi-RF-line -> NbTi; symbol Quantum Computing:NbTi-RF-line -> Quantum Computing:RF Line NbTi
- RFL18: renamed from LX-X8; value NbTi-RF-line -> NbTi; symbol Quantum Computing:NbTi-RF-line -> Quantum Computing:RF Line NbTi
- RFL19: renamed from LX-X9; value NbTi-RF-line -> NbTi; symbol Quantum Computing:NbTi-RF-line -> Quantum Computing:RF Line NbTi
- RFL20: renamed from LX-X10; value NbTi-RF-line -> NbTi; symbol Quantum Computing:NbTi-RF-line -> Quantum Computing:RF Line NbTi
- RFL21: renamed from LX-X11; value NbTi-RF-line -> NbTi; symbol Quantum Computing:NbTi-RF-line -> Quantum Computing:RF Line NbTi
- RFL22: renamed from LX-X12; value NbTi-RF-line -> NbTi; symbol Quantum Computing:NbTi-RF-line -> Quantum Computing:RF Line NbTi
- RFL23: renamed from LX-X25; value NbTi-RF-line -> NbTi; symbol Quantum Computing:NbTi-RF-line -> Quantum Computing:RF Line NbTi
- RFL24: renamed from LX-X26; value NbTi-RF-line -> NbTi; symbol Quantum Computing:NbTi-RF-line -> Quantum Computing:RF Line NbTi
- RFL25: renamed from LX-X27; value NbTi-RF-line -> NbTi; symbol Quantum Computing:NbTi-RF-line -> Quantum Computing:RF Line NbTi
- RFL26: renamed from LX-X28; value NbTi-RF-line -> NbTi; symbol Quantum Computing:NbTi-RF-line -> Quantum Computing:RF Line NbTi
- RFL27: renamed from LX-X29; value NbTi-RF-line -> NbTi; symbol Quantum Computing:NbTi-RF-line -> Quantum Computing:RF Line NbTi
- RFL28: renamed from LX-X30; value NbTi-RF-line -> NbTi; symbol Quantum Computing:NbTi-RF-line -> Quantum Computing:RF Line NbTi
- RFL29: renamed from LX-X31; value NbTi-RF-line -> NbTi; symbol Quantum Computing:NbTi-RF-line -> Quantum Computing:RF Line NbTi
- TJI1, TJI2: symbol Quantum Computing:LNF-ISISC4_12A -> Quantum Computing:Isolator LNF-ISISC4_12A
- TWPA1: value SW_TWPA -> TWPA SW; symbol Quantum Computing:SW_TWPA -> Quantum Computing:TWPA SW
Connections:
- net at Coupler1.: now also L:3.; no longer L:4.
- net at L:3.: now also TWPA1.; no longer Coupler1.
- net at TJI2.: now also L:4.; no longer L:5.
- net at TJI1.: now also L:56.; no longer L:2.
- new net: Coupler1., L:4.
- new net: EF26., LPF17.
- new net: L:5., TJI2.
- new net: L:2., TJI1.
- new net: EF25., LPF16.
- new net: EF12., LPF12.
- new net: EF24., LPF15.
- new net: EF23., LPF14.
- new net: EF22., LPF13.
Other:
- note removed: "ISOLATOR-1"
- note removed: "ISOLATOR-2"
- company: (none) -> Technology Innovation Institute
- title: (none) -> XLD Setup Q2 2023

Commit message: correct L2-12 LNA gnd, it was fixed. Changed the IQM5q drive line LP to the correct cut frequency.
Connections:
- net at Coupler1.: now also L:3.; no longer L:4.
- net at L:3.: now also TWPA1.; no longer Coupler1.
- net at TJI2.: now also L:4.; no longer L:5.
- net at TJI1.: now also L:56.; no longer L:2.
- new net: Coupler1., L:4.
- new net: EF26., LPF17.
- new net: L:5., TJI2.
- new net: L:2., TJI1.
- new net: EF25., LPF16.
- new net: EF12., LPF12.
- new net: EF24., LPF15.
- new net: EF23., LPF14.
- new net: EF22., LPF13.
- no-connect marks 1 -> 0
Other:
- note removed: "LP 7.2GHz - IR 10GHz"
Changed lines of the file:
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@@
     (company "Technology Innovation Institute")
   )
-  (no_connect (at 132.08 97.155))
   (bus_entry (at 536.575 307.34) (size 2.54 2.54)
     (stroke (width 0) (type default))
@@
     (effects (font (size 2 2) (color 0 194 194 1)) (justify left bottom))
   )
-  (text "LP 7.2GHz - IR 10GHz" (at 274.955 356.235 0)
+  (text "LP 8GHz - IR 10GHz" (at 274.955 356.235 0)
     (effects (font (size 1.27 1.27)) (justify left bottom))
   )

Commit message: update tii1qb11
Connections:
- net at Coupler1.: now also L:3.; no longer L:4.
- net at L:3.: now also TWPA1.; no longer Coupler1.
- net at TJI2.: now also L:4.; no longer L:5.
- net at TJI1.: now also L:56.; no longer L:2.
- new net: Coupler1., L:4.
- new net: EF26., LPF17.
- new net: L:5., TJI2.
- new net: L:2., TJI1.
- new net: EF25., LPF16.
- new net: EF12., LPF12.
- new net: EF24., LPF15.
- new net: EF23., LPF14.
- new net: EF22., LPF13.

Commit message: fix qw5q twpa pump line ip address
Connections:
- net at Coupler1.: now also L:3.; no longer L:4.
- net at L:3.: now also TWPA1.; no longer Coupler1.
- net at TJI2.: now also L:4.; no longer L:5.
- net at TJI1.: now also L:56.; no longer L:2.
- new net: Coupler1., L:4.
- new net: EF26., LPF17.
- new net: L:5., TJI2.
- new net: L:2., TJI1.
- new net: EF25., LPF16.
- new net: EF12., LPF12.
- new net: EF24., LPF15.
- new net: EF23., LPF14.
- new net: EF22., LPF13.

Commit message: ip for LO18
Connections:
- net at Coupler1.: now also L:3.; no longer L:4.
- net at L:3.: now also TWPA1.; no longer Coupler1.
- net at TJI2.: now also L:4.; no longer L:5.
- net at TJI1.: now also L:56.; no longer L:2.
- new net: Coupler1., L:4.
- new net: EF26., LPF17.
- new net: L:5., TJI2.
- new net: L:2., TJI1.
- new net: EF25., LPF16.
- new net: EF12., LPF12.
- new net: EF24., LPF15.
- new net: EF23., LPF14.
- new net: EF22., LPF13.
