File: XLD/Q2_2023/iqm5q.kicad_sch (KiCad schematic)
At the start: 146 parts

Commit message: Updated the labeling for the cables from the splitters to the controller for the local oscillators 3 and 4
Connections:
- net at Coupler1.: now also L:3.; no longer L:4.
- net at L:3.: now also TWPA1.; no longer Coupler1.
- net at TJI2.: now also L:4.; no longer L:5.
- net at TJI1.: now also L:56.; no longer L:2.
- new net: Coupler1., L:4.
- new net: EF26., LPF17.
- new net: L:5., TJI2.
- new net: L:2., TJI1.
- new net: EF25., LPF16.
- new net: EF12., LPF12.
- new net: EF24., LPF15.
- new net: EF23., LPF14.
- new net: EF22., LPF13.

Commit message: corrected the names ans the output lines of the opxs
Connections:
- net at Coupler1.: now also L:3.; no longer L:4.
- net at L:3.: now also TWPA1.; no longer Coupler1.
- net at TJI2.: now also L:4.; no longer L:5.
- net at TJI1.: now also L:56.; no longer L:2.
- new net: Coupler1., L:4.
- new net: EF26., LPF17.
- new net: L:5., TJI2.
- new net: L:2., TJI1.
- new net: EF25., LPF16.
- new net: EF12., LPF12.
- new net: EF24., LPF15.
- new net: EF23., LPF14.
- new net: EF22., LPF13.

Commit message: add lo oscillators to line b con1 con2 con3
Connections:
- net at Coupler1.: now also L:3.; no longer L:4.
- net at L:3.: now also TWPA1.; no longer Coupler1.
- net at TJI2.: now also L:4.; no longer L:5.
- net at TJI1.: now also L:56.; no longer L:2.
- new net: Coupler1., L:4.
- new net: EF26., LPF17.
- new net: L:5., TJI2.
- new net: L:2., TJI1.
- new net: EF25., LPF16.
- new net: EF12., LPF12.
- new net: EF24., LPF15.
- new net: EF23., LPF14.
- new net: EF22., LPF13.

Commit message: partial re-labeling
Connections:
- net at Coupler1.: now also L:3.; no longer L:4.
- net at L:3.: now also TWPA1.; no longer Coupler1.
- net at TJI2.: now also L:4.; no longer L:5.
- net at TJI1.: now also L:56.; no longer L:2.
- new net: Coupler1., L:4.
- new net: EF26., LPF17.
- new net: L:5., TJI2.
- new net: L:2., TJI1.
- new net: EF25., LPF16.
- new net: EF12., LPF12.
- new net: EF24., LPF15.
- new net: EF23., LPF14.
- new net: EF22., LPF13.

Commit message: updating labels
Connections:
- net at Coupler1.: now also L:3.; no longer L:4.
- net at L:3.: now also TWPA1.; no longer Coupler1.
- net at TJI2.: now also L:4.; no longer L:5.
- net at TJI1.: now also L:56.; no longer L:2.
- new net: Coupler1., L:4.
- new net: EF26., LPF17.
- new net: L:5., TJI2.
- new net: L:2., TJI1.
- new net: EF25., LPF16.
- new net: EF12., LPF12.
- new net: EF24., LPF15.
- new net: EF23., LPF14.
- new net: EF22., LPF13.

Commit message: updatede de line B 5 qubits
Connections:
- net at Coupler1.: now also L:3.; no longer L:4.
- net at L:3.: now also TWPA1.; no longer Coupler1.
- net at TJI2.: now also L:4.; no longer L:5.
- net at TJI1.: now also L:56.; no longer L:2.
- new net: Coupler1., L:4.
- new net: EF26., LPF17.
- new net: L:5., TJI2.
- new net: L:2., TJI1.
- new net: EF25., LPF16.
- new net: EF12., LPF12.
- new net: EF24., LPF15.
- new net: EF23., LPF14.
- new net: EF22., LPF13.

Commit message: removed lines for line C in qw25q
Connections:
- net at Coupler1.: now also L:3.; no longer L:4.
- net at L:3.: now also TWPA1.; no longer Coupler1.
- net at TJI2.: now also L:4.; no longer L:5.
- net at TJI1.: now also L:56.; no longer L:2.
- new net: Coupler1., L:4.
- new net: EF26., LPF17.
- new net: L:5., TJI2.
- new net: L:2., TJI1.
- new net: EF25., LPF16.
- new net: EF12., LPF12.
- new net: EF24., LPF15.
- new net: EF23., LPF14.
- new net: EF22., LPF13.
