File: XLD/Q2_2023/qm_192_168_0_1.kicad_sch (KiCad schematic)
At the start: 113 parts, among them T1 Terminator, T10 Terminator, T11 Terminator, T12 Terminator, T13 Terminator, T14 Terminator, T15 Terminator, T16 Terminator, T2 Terminator, T3 Terminator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

Commit message: corrected the output lines for the readout for QW25q
Connections:
- net at Splitter17.: now also Splitter18.; no longer Splitter16.
- net at Splitter18.: no longer Splitter17.
- net at Splitter6.: now also Splitter5.; no longer Splitter8.
- net at Splitter10.: now also Splitter9.; no longer Splitter8.
- net at Splitter22.: no longer Splitter21.
- net at Splitter20.: no longer Splitter21.
- net at Splitter7.: no longer Splitter6.
- net at Splitter5.: no longer Splitter6.
- net at Splitter14.: now also Splitter13.
- net at Splitter13.: now also Splitter12.; no longer Splitter14.
- net at Splitter11.: now also Splitter10.
- net at Splitter12.: no longer Splitter13.
- net at Splitter1.: no longer Splitter2.
- net at Splitter3.: no longer Splitter2.
- net at Splitter4.: now also Splitter3.
- new net: Splitter16., Splitter17.
- new net: Splitter15., Splitter17.
- new net: Splitter6., Splitter8.
- new net: Splitter10., Splitter8.
- new net: Splitter21., Splitter22.
- new net: Splitter20., Splitter21.
- new net: Splitter6., Splitter7.
- new net: Splitter13., Splitter15.
- new net: Splitter1., Splitter2.
- new net: Splitter2., Splitter3.
- now unconnected: Splitter3.

Commit message: added changes of filter thermalization for flux lines qw25q
Connections:
- net at Splitter17.: now also Splitter18.; no longer Splitter16.
- net at Splitter18.: no longer Splitter17.
- net at Splitter6.: now also Splitter5.; no longer Splitter8.
- net at Splitter10.: now also Splitter9.; no longer Splitter8.
- net at Splitter22.: no longer Splitter21.
- net at Splitter20.: no longer Splitter21.
- net at Splitter7.: no longer Splitter6.
- net at Splitter5.: no longer Splitter6.
- net at Splitter14.: now also Splitter13.
- net at Splitter13.: now also Splitter12.; no longer Splitter14.
- net at Splitter11.: now also Splitter10.
- net at Splitter12.: no longer Splitter13.
- net at Splitter1.: no longer Splitter2.
- net at Splitter3.: no longer Splitter2.
- net at Splitter4.: now also Splitter3.
- new net: Splitter16., Splitter17.
- new net: Splitter15., Splitter17.
- new net: Splitter6., Splitter8.
- new net: Splitter10., Splitter8.
- new net: Splitter21., Splitter22.
- new net: Splitter20., Splitter21.
- new net: Splitter6., Splitter7.
- new net: Splitter13., Splitter15.
- new net: Splitter1., Splitter2.
- new net: Splitter2., Splitter3.
- now unconnected: Splitter3.

Commit message: added labels to lo3 splitter exits
Connections:
- net LO_03: no longer MX10. (RF), MX11. (RF), MX13. (RF), MX14. (RF), MX26. (RF), MX27. (RF), MX34. (RF), MX35. (RF)
- net at Splitter17.: now also Splitter18.; no longer Splitter16.
- net at Splitter18.: no longer Splitter17.
- net at Splitter6.: now also Splitter5.; no longer Splitter8.
- net at Splitter10.: now also Splitter9.; no longer Splitter8.
- net at Splitter22.: no longer Splitter21.
- net at Splitter20.: no longer Splitter21.
- net LO3-SP4: now reaches Splitter7.
- net LO3-SP4: now also MX27. (RF), MX34. (RF); no longer Splitter6.
- net LO3-SP2: now reaches Splitter5.
- net LO3-SP2: now also MX11. (RF); no longer Splitter6.
- net at Splitter14.: now also Splitter13.
- net at Splitter13.: now also Splitter12.; no longer Splitter14.
- net LO3-SP8: now reaches Splitter11.
- net LO3-SP8: now also MX14. (RF)
- net at Splitter12.: no longer Splitter13.
- net LO3-SP6: now reaches Splitter9.
- net at Splitter1.: no longer Splitter2.
- net at Splitter3.: no longer Splitter2.
- net at Splitter4.: now also Splitter3.
- new net: Splitter16., Splitter17.
- new net: Splitter15., Splitter17.
- new net: Splitter6., Splitter8.
- new net: Splitter10., Splitter8.
- new net: Splitter21., Splitter22.
- new net: Splitter20., Splitter21.
- new net: Splitter6., Splitter7.
- new net: Splitter10., Splitter11.
- new net: Splitter13., Splitter15.
- new net: Splitter1., Splitter2.
- new net: Splitter2., Splitter3.
- new net LO3-SP1: MX10. (RF), Splitter5.
- new net LO3-SP3: MX26. (RF), Splitter7.
- new net LO3-SP5: MX35. (RF), Splitter9.
- new net LO3-SP7: MX13. (RF), Splitter11.
- now unconnected: Splitter3.
Other:
- moved on the sheet: Splitter10, Splitter11, Splitter5, Splitter6, Splitter7, Splitter9

Commit message: Updated the labeling for the cables from the splitters to the controller for the local oscillators 3 and 4
Connections:
- net LO3-SP2: now also Splitter7.; no longer Splitter5.
- net LO3-SP3: now also MX16. (RF); no longer MX26. (RF)
- net LO3-SP4: now also MX20. (RF), Splitter5.; no longer MX27. (RF), MX34. (RF), Splitter7.
- net LO3-SP5: now also MX17. (RF); no longer MX35. (RF)
- net LO3-SP7: now also MX23. (RF); no longer MX13. (RF)
- net LO3-SP8: no longer MX14. (RF)
- net LO_04: no longer MX16. (RF), MX17. (RF), MX20. (RF), MX23. (RF), MX24. (RF), MX25. (RF), MX32. (RF), MX33. (RF)
- net at Splitter17.: now also Splitter18.; no longer Splitter16.
- net LO4-SP8: now reaches Splitter18.
- net LO4-SP8: no longer Splitter17.
- net LO4-SP6: now reaches Splitter16.
- net at Splitter6.: now also Splitter5.; no longer Splitter8.
- net at Splitter10.: now also Splitter9.; no longer Splitter8.
- net at Splitter22.: no longer Splitter21.
- net at Splitter20.: no longer Splitter21.
- net LO4-SP3: now reaches Splitter14.
- net LO4-SP3: now also MX34. (RF)
- net at Splitter13.: now also Splitter12.; no longer Splitter14.
- net LO4-SP4: now reaches Splitter12.
- net LO4-SP4: now also MX27. (RF); no longer Splitter13.
- net at Splitter1.: no longer Splitter2.
- net at Splitter3.: no longer Splitter2.
- net at Splitter4.: now also Splitter3.
- new net: Splitter16., Splitter17.
- new net: Splitter15., Splitter17.
- new net: Splitter6., Splitter8.
- new net: Splitter10., Splitter8.
- new net: Splitter21., Splitter22.
- new net: Splitter20., Splitter21.
- new net: Splitter6., Splitter7.
- new net: Splitter13., Splitter14.
- new net: Splitter10., Splitter11.
- new net: Splitter13., Splitter15.
- new net: Splitter1., Splitter2.
- new net: Splitter2., Splitter3.
- new net LO4-SP1: MX26. (RF), Splitter12.
- new net LO4-SP2: MX32. (RF), Splitter14.
- new net LO4-SP5: MX33. (RF), Splitter16.
- new net LO4-SP7: MX35. (RF), Splitter18.
- now unconnected: Splitter3.
- no-connect marks 17 -> 25
Other:
- moved on the sheet: LO14, Splitter12, Splitter13, Splitter14, Splitter15, Splitter16, Splitter17, Splitter18

Commit message: connections for qw25q 2 qubit characterization
Parts:
- added Splitter23, Splitter24: ZFRSC_183_S+, symbol Quantum Computing:Splitter ZFRSC_183_S+
Connections:
- net LO3-SP1: no longer MX10. (RF)
- net LO3-SP2: no longer MX11. (RF)
- net LO_01: no longer MX1. (RF)
- net LO_02: now also Splitter24.
- net LO_05: no longer MX7. (RF)
- net LO_08: now also Splitter23.
- net at Splitter17.: now also Splitter18.; no longer Splitter16.
- net at Splitter6.: now also Splitter5.; no longer Splitter8.
- net at Splitter10.: now also Splitter9.; no longer Splitter8.
- net at Splitter22.: no longer Splitter21.
- net at Splitter20.: no longer Splitter21.
- net at Splitter13.: now also Splitter12.; no longer Splitter14.
- net at Splitter1.: no longer Splitter2.
- net at Splitter3.: no longer Splitter2.
- net at Splitter4.: now also Splitter3.
- new net: Splitter16., Splitter17.
- new net: Splitter15., Splitter17.
- new net: Splitter6., Splitter8.
- new net: Splitter10., Splitter8.
- new net: Splitter21., Splitter22.
- new net: Splitter20., Splitter21.
- new net: Splitter6., Splitter7.
- new net: Splitter13., Splitter14.
- new net: Splitter10., Splitter11.
- new net: Splitter13., Splitter15.
- new net: Splitter1., Splitter2.
- new net: Splitter2., Splitter3.
- new net L02_SP1: MX7. (RF), Splitter24.
- new net L02_SP2: MX1. (RF), Splitter24.
- new net L08_SP1: MX10. (RF), Splitter23.
- new net L08_SP2: MX11. (RF), Splitter23.
- now unconnected: Splitter3.
- no-connect marks 25 -> 27
Other:
- moved on the sheet: LO10, LO11, LO12, Splitter1, Splitter2, Splitter3, Splitter4

Commit message: corrected the names ans the output lines of the opxs
Parts:
- renumbered OPX6 to OPX2, OPX3 to OPX4, OPX4 to OPX5, OPX2 to OPX6, OPX5 to OPX7
Connections:
- net LO3-SP3: now also MX13. (RF); no longer MX16. (RF)
- net LO3-SP4: now also MX16. (RF); no longer MX20. (RF)
- net LO3-SP5: now also MX14. (RF); no longer MX17. (RF)
- net LO3-SP7: now also MX17. (RF); no longer MX23. (RF)
- net LO4-SP1: now also MX20. (RF); no longer MX26. (RF)
- net LO4-SP4: now also MX23. (RF); no longer MX27. (RF)
- net at Splitter17.: now also Splitter18.; no longer Splitter16.
- net at Splitter6.: now also Splitter5.; no longer Splitter8.
- net at Splitter10.: now also Splitter9.; no longer Splitter8.
- net at Splitter22.: no longer Splitter21.
- net at Splitter20.: no longer Splitter21.
- net at Splitter13.: now also Splitter12.; no longer Splitter14.
- net at Splitter1.: no longer Splitter2.
- net at Splitter3.: no longer Splitter2.
- net at Splitter4.: now also Splitter3.
- new net: Splitter16., Splitter17.
- new net: Splitter15., Splitter17.
- new net: Splitter6., Splitter8.
- new net: Splitter10., Splitter8.
- new net: Splitter21., Splitter22.
- new net: Splitter20., Splitter21.
- new net: Splitter6., Splitter7.
- new net: Splitter13., Splitter14.
- new net: Splitter10., Splitter11.
- new net: Splitter13., Splitter15.
- new net: Splitter1., Splitter2.
- new net: Splitter2., Splitter3.
- now unconnected: Splitter3.

Commit message: add lo oscillators to line b con1 con2 con3
Parts:
- added Splitter25: ZFRSC_183_S+, symbol Quantum Computing:Splitter ZFRSC_183_S+
- renumbered OPX7 to OPX3
Connections:
- net LO_08 is gone; now on net LO_09: LO12., Splitter23.
- net ERA_01: no longer MX12. (RF)
- net L02_SP1: no longer MX7. (RF)
- net L02_SP2: no longer MX1. (RF)
- net LO4-SP1: no longer MX20. (RF)
- net LO4-SP4: no longer MX23. (RF)
- net LO_01: no longer MX15. (RF), MX2. (RF)
- net LO_06: no longer LO16., Splitter21.
- net at Splitter17.: now also Splitter18.; no longer Splitter16.
- net at Splitter15.: now also Splitter13.; no longer Splitter17.
- net at Splitter8.: now also Splitter10.; no longer Splitter6.
- net at Splitter10.: now also Splitter9.; no longer Splitter8.
- net at Splitter21.: now also Splitter20.; no longer Splitter22.
- net at Splitter20.: no longer Splitter21.
- net at Splitter6.: now also Splitter5.; no longer Splitter7.
- net at Splitter13.: now also Splitter12.; no longer Splitter14.
- net QM_3_5: now reaches OPX3. (LAN)
- net at Splitter1.: no longer Splitter2.
- net at Splitter3.: no longer Splitter2.
- net at Splitter4.: now also Splitter3.
- net L08_SP1 renamed LO_09
- net LO_09: no longer MX10. (RF)
- removed net L08_SP2: MX11. (RF), Splitter23.
- net LO_03 renamed LO3
- net LO3: no longer Splitter8.
- net LO_04 renamed LO4
- net LO4: no longer Splitter15.
- new net: Splitter16., Splitter17.
- new net: Splitter15., Splitter17.
- new net: LO16., Splitter25.
- new net: Splitter6., Splitter8.
- new net: Splitter21., Splitter22.
- new net: Splitter6., Splitter7.
- new net: Splitter13., Splitter14.
- new net: Splitter10., Splitter11.
- new net: Splitter1., Splitter2.
- new net: Splitter2., Splitter3.
- new net L03-SP1: MX1. (RF)
- new net L03-SP2: MX2. (RF)
- new net L04-SP1: MX3. (RF)
- new net L04-SP2: MX7. (RF)
- new net L06_SP1: Splitter25.
- new net L06_SP2: Splitter25.
- new net L07: MX15. (RF)
- new net L09_SP1: MX10. (RF), Splitter23.
- new net L09_SP2: MX11. (RF), Splitter23.
- new net LO6-SP1: MX20. (RF)
- new net LO6-SP2: MX23. (RF)
- new net QM_3_3: OPX3. (LAN)
- new net QM_3_4: OPX3. (LAN)
- now unconnected: Splitter3.
- no-connect marks 27 -> 24
Other:
- moved on the sheet: LO13, LO14, Splitter20, Splitter21, Splitter22

Commit message: partial re-labeling
Parts:
- added Splitter26, Splitter27: ZFRSC_183_S+, symbol Quantum Computing:Splitter ZFRSC_183_S+
Connections:
- net L07 is gone; now on net QM_2_I1_Q2: MX15. (RF)
- net ERA_07: no longer LO4.
- net at Splitter17.: now also Splitter18.; no longer Splitter16.
- net at Splitter15.: now also Splitter13.; no longer Splitter17.
- net at Splitter8.: now also Splitter10.
- net at Splitter6.: now also Splitter5.; no longer Splitter8.
- net at Splitter10.: now also Splitter9.; no longer Splitter8.
- net at Splitter21.: now also Splitter20.
- net at Splitter22.: no longer Splitter21.
- net at Splitter20.: no longer Splitter21.
- net at Splitter13.: now also Splitter12.; no longer Splitter14.
- net at Splitter1.: no longer Splitter2.
- net at Splitter3.: no longer Splitter2.
- net at Splitter4.: now also Splitter3.
- net LO3: no longer names the net of LO13.
- net LO3: now also Splitter26.
- net LO4: no longer names the net of LO14.
- net LO4: now also Splitter27.
- new net: Splitter16., Splitter17.
- new net: Splitter15., Splitter17.
- new net: Splitter6., Splitter8.
- new net: Splitter21., Splitter22.
- new net: Splitter6., Splitter7.
- new net: Splitter13., Splitter14.
- new net: Splitter10., Splitter11.
- new net: Splitter1., Splitter2.
- new net: Splitter2., Splitter3.
- new net ES7: LO4., MX15. (RF)
- new net L03_SP1: Splitter26.
- new net L03_SP2: Splitter26.
- new net L04_SP1: Splitter27.
- new net L04_SP2: Splitter27.
- now unconnected: Splitter3.
- no-connect marks 24 -> 27
Other:
- moved on the sheet: LO13, LO4
