File: XLD/Q2_2023/qw5q_gold.kicad_sch (KiCad schematic)
At the start: 128 parts

Commit message: various fixes
swap L3-20 with L2-17 in qblox
change ip of Lo18 to 192.168.0.208 (tii1q_b4 twpa pump) and type to ERA
rename LO_ERA_pp to LO_ERA
Connections:
- net at Eccosorb2.: now also L:9.; no longer LPF2.
- net at Eccosorb1.: now also L:7.; no longer LPF1.
- net at Eccosorb7.: now also LPF7.; no longer L:19.
- net at Eccosorb10.: now also LPF10.; no longer L:25.
- net at L:3.: now also TWPA1.; no longer Coupler1.
- net at TWPA1.: now also L:2.; no longer L:3.
- net at Eccosorb6.: now also L:17.; no longer LPF6.
- net at TJI1.: now also L:1.; no longer L:2.
- net at Eccosorb5.: now also LPF5.; no longer L:15.
- net at Eccosorb3.: now also L:11.; no longer LPF3.
- net at Eccosorb9.: now also L:23.; no longer LPF9.
- net at TJI2.: now also L:4.; no longer L:5.
- net at Eccosorb11.: now also LPF11.; no longer L:27.
- net at Eccosorb4.: now also L:13.; no longer LPF4.
- net at Eccosorb8.: now also L:21.; no longer LPF8.
- net at L:4.: now also Coupler1.; no longer TJI2.
- new net: Eccosorb2., LPF2.
- new net: Eccosorb1., LPF1.
- new net: Eccosorb7., L:19.
- new net: Eccosorb10., L:25.
- new net: Coupler1., L:3.
- new net: Eccosorb6., LPF6.
- new net: L:2., TJI1.
- new net: Eccosorb5., L:15.
- new net: Eccosorb3., LPF3.
- new net: Eccosorb9., LPF9.
- new net: L:5., TJI2.
- new net: Eccosorb11., L:27.
- new net: Eccosorb4., LPF4.
- new net: Eccosorb8., LPF8.

Commit message: corrected the output lines for the readout for QW25q
Connections:
- net at Eccosorb2.: now also L:9.; no longer LPF2.
- net at Eccosorb1.: now also L:7.; no longer LPF1.
- net at Eccosorb7.: now also LPF7.; no longer L:19.
- net at Eccosorb10.: now also LPF10.; no longer L:25.
- net at L:3.: now also TWPA1.; no longer Coupler1.
- net at TWPA1.: now also L:2.; no longer L:3.
- net at Eccosorb6.: now also L:17.; no longer LPF6.
- net at TJI1.: now also L:1.; no longer L:2.
- net at Eccosorb5.: now also LPF5.; no longer L:15.
- net at Eccosorb3.: now also L:11.; no longer LPF3.
- net at Eccosorb9.: now also L:23.; no longer LPF9.
- net at TJI2.: now also L:4.; no longer L:5.
- net at Eccosorb11.: now also LPF11.; no longer L:27.
- net at Eccosorb4.: now also L:13.; no longer LPF4.
- net at Eccosorb8.: now also L:21.; no longer LPF8.
- net at L:4.: now also Coupler1.; no longer TJI2.
- new net: Eccosorb2., LPF2.
- new net: Eccosorb1., LPF1.
- new net: Eccosorb7., L:19.
- new net: Eccosorb10., L:25.
- new net: Coupler1., L:3.
- new net: Eccosorb6., LPF6.
- new net: L:2., TJI1.
- new net: Eccosorb5., L:15.
- new net: Eccosorb3., LPF3.
- new net: Eccosorb9., LPF9.
- new net: L:5., TJI2.
- new net: Eccosorb11., L:27.
- new net: Eccosorb4., LPF4.
- new net: Eccosorb8., LPF8.

Commit message: added changes of filter thermalization for flux lines qw25q
Connections:
- net at Eccosorb2.: now also L:9.; no longer LPF2.
- net at Eccosorb1.: now also L:7.; no longer LPF1.
- net at Eccosorb7.: now also LPF7.; no longer L:19.
- net at Eccosorb10.: now also LPF10.; no longer L:25.
- net at L:3.: now also TWPA1.; no longer Coupler1.
- net at TWPA1.: now also L:2.; no longer L:3.
- net at Eccosorb6.: now also L:17.; no longer LPF6.
- net at TJI1.: now also L:1.; no longer L:2.
- net at Eccosorb5.: now also LPF5.; no longer L:15.
- net at Eccosorb3.: now also L:11.; no longer LPF3.
- net at Eccosorb9.: now also L:23.; no longer LPF9.
- net at TJI2.: now also L:4.; no longer L:5.
- net at Eccosorb11.: now also LPF11.; no longer L:27.
- net at Eccosorb4.: now also L:13.; no longer LPF4.
- net at Eccosorb8.: now also L:21.; no longer LPF8.
- net at L:4.: now also Coupler1.; no longer TJI2.
- new net: Eccosorb2., LPF2.
- new net: Eccosorb1., LPF1.
- new net: Eccosorb7., L:19.
- new net: Eccosorb10., L:25.
- new net: Coupler1., L:3.
- new net: Eccosorb6., LPF6.
- new net: L:2., TJI1.
- new net: Eccosorb5., L:15.
- new net: Eccosorb3., LPF3.
- new net: Eccosorb9., LPF9.
- new net: L:5., TJI2.
- new net: Eccosorb11., L:27.
- new net: Eccosorb4., LPF4.
- new net: Eccosorb8., LPF8.

Commit message: added labels to lo3 splitter exits
Connections:
- net at Eccosorb2.: now also L:9.; no longer LPF2.
- net at Eccosorb1.: now also L:7.; no longer LPF1.
- net at Eccosorb7.: now also LPF7.; no longer L:19.
- net at Eccosorb10.: now also LPF10.; no longer L:25.
- net at L:3.: now also TWPA1.; no longer Coupler1.
- net at TWPA1.: now also L:2.; no longer L:3.
- net at Eccosorb6.: now also L:17.; no longer LPF6.
- net at TJI1.: now also L:1.; no longer L:2.
- net at Eccosorb5.: now also LPF5.; no longer L:15.
- net at Eccosorb3.: now also L:11.; no longer LPF3.
- net at Eccosorb9.: now also L:23.; no longer LPF9.
- net at TJI2.: now also L:4.; no longer L:5.
- net at Eccosorb11.: now also LPF11.; no longer L:27.
- net at Eccosorb4.: now also L:13.; no longer LPF4.
- net at Eccosorb8.: now also L:21.; no longer LPF8.
- net at L:4.: now also Coupler1.; no longer TJI2.
- new net: Eccosorb2., LPF2.
- new net: Eccosorb1., LPF1.
- new net: Eccosorb7., L:19.
- new net: Eccosorb10., L:25.
- new net: Coupler1., L:3.
- new net: Eccosorb6., LPF6.
- new net: L:2., TJI1.
- new net: Eccosorb5., L:15.
- new net: Eccosorb3., LPF3.
- new net: Eccosorb9., LPF9.
- new net: L:5., TJI2.
- new net: Eccosorb11., L:27.
- new net: Eccosorb4., LPF4.
- new net: Eccosorb8., LPF8.

Commit message: Updated the labeling for the cables from the splitters to the controller for the local oscillators 3 and 4
Connections:
- net at Eccosorb2.: now also L:9.; no longer LPF2.
- net at Eccosorb1.: now also L:7.; no longer LPF1.
- net at Eccosorb7.: now also LPF7.; no longer L:19.
- net at Eccosorb10.: now also LPF10.; no longer L:25.
- net at L:3.: now also TWPA1.; no longer Coupler1.
- net at TWPA1.: now also L:2.; no longer L:3.
- net at Eccosorb6.: now also L:17.; no longer LPF6.
- net at TJI1.: now also L:1.; no longer L:2.
- net at Eccosorb5.: now also LPF5.; no longer L:15.
- net at Eccosorb3.: now also L:11.; no longer LPF3.
- net at Eccosorb9.: now also L:23.; no longer LPF9.
- net at TJI2.: now also L:4.; no longer L:5.
- net at Eccosorb11.: now also LPF11.; no longer L:27.
- net at Eccosorb4.: now also L:13.; no longer LPF4.
- net at Eccosorb8.: now also L:21.; no longer LPF8.
- net at L:4.: now also Coupler1.; no longer TJI2.
- new net: Eccosorb2., LPF2.
- new net: Eccosorb1., LPF1.
- new net: Eccosorb7., L:19.
- new net: Eccosorb10., L:25.
- new net: Coupler1., L:3.
- new net: Eccosorb6., LPF6.
- new net: L:2., TJI1.
- new net: Eccosorb5., L:15.
- new net: Eccosorb3., LPF3.
- new net: Eccosorb9., LPF9.
- new net: L:5., TJI2.
- new net: Eccosorb11., L:27.
- new net: Eccosorb4., LPF4.
- new net: Eccosorb8., LPF8.

Commit message: corrected the names ans the output lines of the opxs
Connections:
- net at Eccosorb2.: now also L:9.; no longer LPF2.
- net at Eccosorb1.: now also L:7.; no longer LPF1.
- net at Eccosorb7.: now also LPF7.; no longer L:19.
- net at Eccosorb10.: now also LPF10.; no longer L:25.
- net at L:3.: now also TWPA1.; no longer Coupler1.
- net at TWPA1.: now also L:2.; no longer L:3.
- net at Eccosorb6.: now also L:17.; no longer LPF6.
- net at TJI1.: now also L:1.; no longer L:2.
- net at Eccosorb5.: now also LPF5.; no longer L:15.
- net at Eccosorb3.: now also L:11.; no longer LPF3.
- net at Eccosorb9.: now also L:23.; no longer LPF9.
- net at TJI2.: now also L:4.; no longer L:5.
- net at Eccosorb11.: now also LPF11.; no longer L:27.
- net at Eccosorb4.: now also L:13.; no longer LPF4.
- net at Eccosorb8.: now also L:21.; no longer LPF8.
- net at L:4.: now also Coupler1.; no longer TJI2.
- new net: Eccosorb2., LPF2.
- new net: Eccosorb1., LPF1.
- new net: Eccosorb7., L:19.
- new net: Eccosorb10., L:25.
- new net: Coupler1., L:3.
- new net: Eccosorb6., LPF6.
- new net: L:2., TJI1.
- new net: Eccosorb5., L:15.
- new net: Eccosorb3., LPF3.
- new net: Eccosorb9., LPF9.
- new net: L:5., TJI2.
- new net: Eccosorb11., L:27.
- new net: Eccosorb4., LPF4.
- new net: Eccosorb8., LPF8.

Commit message: add lo oscillators to line b con1 con2 con3
Connections:
- net at Eccosorb2.: now also L:9.; no longer LPF2.
- net at Eccosorb1.: now also L:7.; no longer LPF1.
- net at Eccosorb7.: now also LPF7.; no longer L:19.
- net at Eccosorb10.: now also LPF10.; no longer L:25.
- net at L:3.: now also TWPA1.; no longer Coupler1.
- net at TWPA1.: now also L:2.; no longer L:3.
- net at Eccosorb6.: now also L:17.; no longer LPF6.
- net at TJI1.: now also L:1.; no longer L:2.
- net at Eccosorb5.: now also LPF5.; no longer L:15.
- net at Eccosorb3.: now also L:11.; no longer LPF3.
- net at Eccosorb9.: now also L:23.; no longer LPF9.
- net at TJI2.: now also L:4.; no longer L:5.
- net at Eccosorb11.: now also LPF11.; no longer L:27.
- net at Eccosorb4.: now also L:13.; no longer LPF4.
- net at Eccosorb8.: now also L:21.; no longer LPF8.
- net at L:4.: now also Coupler1.; no longer TJI2.
- new net: Eccosorb2., LPF2.
- new net: Eccosorb1., LPF1.
- new net: Eccosorb7., L:19.
- new net: Eccosorb10., L:25.
- new net: Coupler1., L:3.
- new net: Eccosorb6., LPF6.
- new net: L:2., TJI1.
- new net: Eccosorb5., L:15.
- new net: Eccosorb3., LPF3.
- new net: Eccosorb9., LPF9.
- new net: L:5., TJI2.
- new net: Eccosorb11., L:27.
- new net: Eccosorb4., LPF4.
- new net: Eccosorb8., LPF8.

Commit message: partial re-labeling
Connections:
- net at Eccosorb2.: now also L:9.; no longer LPF2.
- net at Eccosorb1.: now also L:7.; no longer LPF1.
- net at Eccosorb7.: now also LPF7.; no longer L:19.
- net at Eccosorb10.: now also LPF10.; no longer L:25.
- net at L:3.: now also TWPA1.; no longer Coupler1.
- net at TWPA1.: now also L:2.; no longer L:3.
- net at Eccosorb6.: now also L:17.; no longer LPF6.
- net at TJI1.: now also L:1.; no longer L:2.
- net at Eccosorb5.: now also LPF5.; no longer L:15.
- net at Eccosorb3.: now also L:11.; no longer LPF3.
- net at Eccosorb9.: now also L:23.; no longer LPF9.
- net at TJI2.: now also L:4.; no longer L:5.
- net at Eccosorb11.: now also LPF11.; no longer L:27.
- net at Eccosorb4.: now also L:13.; no longer LPF4.
- net at Eccosorb8.: now also L:21.; no longer LPF8.
- net at L:4.: now also Coupler1.; no longer TJI2.
- new net: Eccosorb2., LPF2.
- new net: Eccosorb1., LPF1.
- new net: Eccosorb7., L:19.
- new net: Eccosorb10., L:25.
- new net: Coupler1., L:3.
- new net: Eccosorb6., LPF6.
- new net: L:2., TJI1.
- new net: Eccosorb5., L:15.
- new net: Eccosorb3., LPF3.
- new net: Eccosorb9., LPF9.
- new net: L:5., TJI2.
- new net: Eccosorb11., L:27.
- new net: Eccosorb4., LPF4.
- new net: Eccosorb8., LPF8.
